File: ESLGSU.kicad_pcb (KiCad board)
At the start: 2 copper layers, 276 parts, among them J1 PJ-080BH, Q1 DMN67D7L-7, Q2 DMN67D7L-7, Q3 DMN67D7L-7, Q4 DMN67D7L-7, Q5 DMN67D7L-7, Q6 DMN67D7L-7, U1 TCA9544A, U10 TPS259474LRPWR, U11 LM73100RPWR, U12 MP28167-A, U13 INA219AxDCN, U14 TPS259474LRPWR, U15 LM73100RPWR, U16 MP28167-A, U17 INA219AxDCN, U18 TPS259474LRPWR, U19 LM73100RPWR, U2 DMT3006LDK, U20 MP28167-A, U21 INA219AxDCN, U22 TPS259474LRPWR, U23 LM73100RPWR, U24 MP28167-A, U26 AP63203WU, U27 AP63205WU, U28 TPS2121, U29 TCAN1051GVDRBRQ, U3 INA219AxDCN, U30 THVD1450DRBR, U31 TXU0304RUTR, U32 TS5A23159RSER, U33 TXU0202DTTR, U34 74LVC2G53GT, U35 TXU0202DTTR, U36 74LVC2G53GT, U37 74LVC2G53GT, U38 TXU0304RUTR, U4 DML3012LDC, U5 LM74700, U6 DMT3006LDK, U7 DML3012LDC, U8 LM74700, U9 INA219AxDCN

Commit message: Finished interfaces work
Parts:
- removed C101, C102: 100n, Capacitor_SMD:C_0603_1608Metric
- removed R96, R99: 0R, Resistor_SMD:R_0603_1608Metric
- added C103: 100p, Capacitor_SMD:C_0402_1005Metric, F.Cu at (199.8, 111.4)
- added C104: 100n, Capacitor_SMD:C_0402_1005Metric, F.Cu at (256.9, 32.9)
- added C105: 100n, Capacitor_SMD:C_0402_1005Metric, F.Cu at (256.9, 35.4)
- added C106: 100n, Capacitor_SMD:C_0402_1005Metric, F.Cu at (256.9, 37.9)
- added C107: 100n, Capacitor_SMD:C_0402_1005Metric, F.Cu at (256.9, 40.4)
- added C110: 100n, Capacitor_SMD:C_0402_1005Metric, F.Cu at (203.8, 111.4)
- added C111: 100n, Capacitor_SMD:C_0402_1005Metric, F.Cu at (203.8, 113.9)
- added R103: 200K, Resistor_SMD:R_0402_1005Metric, F.Cu at (203.8, 116.4)
- added R104: 10K, Resistor_SMD:R_0402_1005Metric, F.Cu at (203.8, 118.9)
- added R105: 10K, Resistor_SMD:R_0402_1005Metric, F.Cu at (203.8, 121.4)
- added R114: 200K, Resistor_SMD:R_0402_1005Metric, F.Cu at (207.8, 111.4)
- added R118: 200K, Resistor_SMD:R_0402_1005Metric, F.Cu at (207.8, 113.9)
- added R119: 200K, Resistor_SMD:R_0402_1005Metric, F.Cu at (207.8, 116.4)
- added RN1: 0R, Resistor_SMD:R_Array_Concave_4x0402, F.Cu at (199.3, 124.5)
- added RN2: 0R, Resistor_SMD:R_Array_Convex_2x0402, F.Cu at (211.3, 111.6)
- added RN3: 0R, Resistor_SMD:R_Array_Concave_4x0402, F.Cu at (259.5, 43.4)
- added RN4: 0R, Resistor_SMD:R_Array_Concave_4x0402, F.Cu at (262.5, 43.4)
- added RN5: 0R, Resistor_SMD:R_Array_Convex_2x0402, F.Cu at (211.3, 114.6)
- added RN6: 0R, Resistor_SMD:R_Array_Convex_2x0402, F.Cu at (211.3, 117.5)
- added RN7: 0R, Resistor_SMD:R_Array_Convex_2x0402, F.Cu at (211.3, 120.5)
- added U39: PCA9306, ESLGSU_Parts_Lib:SOT833-1-XSON8, F.Cu at (199.0, 128.0)
- added U40: TXB0104RUT, ESLGSU_Parts_Lib:T-UQFN-12, F.Cu at (268.7, 47.2)
- added U41: STM32F072VBTx, Package_QFP:LQFP-100_14x14mm_P0.5mm, F.Cu at (185.2, 141.7)
- added U44: TMUX1574RSVR, ESLGSU_Parts_Lib:T-UQFN-16, F.Cu at (276.4, 38.4)
- added U46: TXB0104RUT, ESLGSU_Parts_Lib:T-UQFN-12, F.Cu at (215.0, 128.2)
- added U47: TMUX1574RSVR, ESLGSU_Parts_Lib:T-UQFN-16, F.Cu at (215.0, 124.1)
- C10, C100, C11, C12, C13, C14, C15, C16, C19, C2, C25, C26, C27, C28, C29, C3, C30, C31, C32, C33, C34, C37, C4, C43, C44, C45, C46, C47, C48, C49, C5, C50, C51, C52, C55, C6, C61, C62, C63, C64, C65, C66, C67, C68, C69, C7, C70, C73, C79, C8, C80, C81, C82, C83, C84, C85, C89, C9, C93, C94, C95, C96, C97, C98, C99: footprint Capacitor_SMD:C_0603_1608Metric -> Capacitor_SMD:C_0402_1005Metric
- R1, R10, R11, R12, R14, R15, R16, R17, R18, R19, R2, R20, R21, R22, R23, R24, R25, R26, R27, R28, R29, R31, R32, R33, R34, R35, R36, R37, R38, R39, R4, R40, R41, R42, R43, R44, R45, R46, R47, R48, R49, R5, R50, R51, R52, R54, R55, R56, R57, R58, R59, R6, R60, R61, R62, R63, R64, R65, R66, R67, R69, R7, R70, R71, R72, R73, R74, R75, R76, R77, R78, R79, R8, R80, R81, R82, R83, R84, R85, R86, R87, R88, R89, R9, R90, R91, R92, R93, R94: footprint Resistor_SMD:R_0603_1608Metric -> Resistor_SMD:R_0402_1005Metric
- R100, R95, R97, R98: value 0R -> 200K; footprint Resistor_SMD:R_0603_1608Metric -> Resistor_SMD:R_0402_1005Metric
- U31: value TXU0304RUTR -> TMUX1574RSVR; footprint ESLGSU_Parts_Lib:T-UQFN-12 -> ESLGSU_Parts_Lib:T-UQFN-16
- U32: value TS5A23159RSER -> TMUX1574RSVR; footprint Package_DFN_QFN:Texas_UQFN-10_1.5x2mm_P0.5mm -> ESLGSU_Parts_Lib:T-UQFN-16
- U34: value 74LVC2G53GT -> TMUX1574RSVR; footprint ESLGSU_Parts_Lib:SOT833-1-XSON8 -> ESLGSU_Parts_Lib:T-UQFN-16
- U36: value 74LVC2G53GT -> TXB0104RUT; footprint ESLGSU_Parts_Lib:SOT833-1-XSON8 -> ESLGSU_Parts_Lib:T-UQFN-12
- U37: value 74LVC2G53GT -> STM32H753ZITx; footprint ESLGSU_Parts_Lib:SOT833-1-XSON8 -> Package_QFP:LQFP-144_20x20mm_P0.5mm
- U38: value TXU0304RUTR -> STM32F072VBTx; footprint ESLGSU_Parts_Lib:T-UQFN-12 -> Package_QFP:LQFP-100_14x14mm_P0.5mm
- moved U34 80.2 mm to (276.2, 43.4)
- moved U36 78.3 mm to (270.8, 33.5)
- moved R97 78.3 mm to (272.2, 20.5)
- moved R98 78.3 mm to (272.2, 23.0)
- moved U37 59.0 mm to (210.0, 146.4)
- moved U38 40.9 mm to (191.4, 57.7)
Connections:
- C100 pad 1: GND -> /Main_uC/VBUS
- C100 pad 2: /Main_uC/SYS_3V3 -> GND
- C96 pad 2: Net-(U30-VCC) -> /Main_uC/VBUS
- C97 pad 2: Net-(U32-VCC) -> /Main_uC/VBUS
- R100 pad 1: /Main_uC/SYS_5V -> /Main_uC/UART1_nEN
- R100 pad 2: Net-(U36-Y1) -> /Main_uC/SYS_3V3
- R95 pad 1: /Main_uC/SYS_3V3 -> /Main_uC/RS4851_TXE
- R95 pad 2: Net-(U30-VCC) -> GND
- R97 pad 1: /Main_uC/SYS_3V3 -> /Main_uC/GPIO_A_nEN
- R97 pad 2: Net-(U34-VCC) -> /Main_uC/SYS_3V3
- R98 pad 1: /Main_uC/SYS_5V -> /Main_uC/GPIO_B_nEN
- R98 pad 2: Net-(U34-Y1) -> /Main_uC/SYS_3V3
- U30 pad 2: GND -> /Main_uC/RS4851_TXE
- U30 pad 8: Net-(U30-VCC) -> /Main_uC/VBUS
- U31 pad 1: /Main_uC/SYS_3V3 -> unconnected-(U31-S1B-Pad1)
- U31 pad 10: /Main_uC/SPI1_MOSI -> unconnected-(U31-D4-Pad10)
- U31 pad 11: Net-(U31-OE) -> unconnected-(U31-S4B-Pad11)
- U31 pad 12: Net-(U31-OE) -> unconnected-(U31-S4A-Pad12)
- U31 pad 2: /Main_uC/SPI1_MOSI -> /Main_uC/VBUS
- U31 pad 3: /Main_uC/SPI1_SCK -> Net-(U31-S2A)
- U31 pad 4: GND -> unconnected-(U31-S2B-Pad4)
- U31 pad 5: /Main_uC/SPI1_MISO -> /Main_uC/VBUS
- U31 pad 7: /Main_uC/SPI1_MISO -> unconnected-(U31-D3-Pad7)
- U31 pad 9: /Main_uC/SPI1_SCK -> unconnected-(U31-S3A-Pad9)
- U32 pad 1: /Main_uC/UART1_REV -> Net-(U32-S1B)
- U32 pad 10: Net-(U32-COM1) -> unconnected-(U32-D4-Pad10)
- U32 pad 2: /Main_uC/UART1_RX -> /Main_uC/UART1_TX
- U32 pad 3: GND -> Net-(U32-S1B)
- U32 pad 4: /Main_uC/UART1_TX -> Net-(U32-S1A)
- U32 pad 5: /Main_uC/UART1_REV -> /Main_uC/UART1_RX
- U32 pad 6: Net-(U32-COM2) -> GND
- U32 pad 7: /Main_uC/UART1_RX -> unconnected-(U32-D3-Pad7)
- U32 pad 8: Net-(U32-VCC) -> unconnected-(U32-S3B-Pad8)
- U32 pad 9: /Main_uC/UART1_TX -> unconnected-(U32-S3A-Pad9)
- U33 pad 7: Net-(U30-VCC) -> /Main_uC/VBUS
- U34 pad 1: Net-(U32-VCC) -> Net-(U34-S1B)
- U34 pad 2: /Main_uC/UART1_nEN -> /Main_uC/GPIO_5
- U34 pad 3: GND -> /Main_uC/GPIO_6
- U34 pad 4: GND -> Net-(U34-S2B)
- U34 pad 5: /Main_uC/UART1_5V -> /Main_uC/GPIO_6
- U34 pad 6: Net-(U34-Y1) -> GND
- U34 pad 7: Net-(U34-VCC) -> /Main_uC/GPIO_7
- U34 pad 8: Net-(U34-VCC) -> Net-(U34-S3B)
- U35 pad 1: Net-(U32-COM2) -> Net-(U32-S1B)
- U35 pad 7: Net-(U32-VCC) -> /Main_uC/VBUS
- U35 pad 8: Net-(U32-COM1) -> Net-(U32-S1A)
- U36 pad 1: Net-(U36-Z) -> /Main_uC/SYS_3V3
- U36 pad 2: /Main_uC/SPI1_nEN -> /Main_uC/GPIO_1
- U36 pad 3: GND -> /Main_uC/GPIO_2
- U36 pad 4: GND -> /Main_uC/GPIO_3
- U36 pad 5: /Main_uC/SPI1_5V -> /Main_uC/GPIO_4
- U36 pad 6: Net-(U36-Y1) -> GND
- U36 pad 7: Net-(U36-VCC) -> Net-(U36-B4)
- U36 pad 8: Net-(U36-VCC) -> Net-(U36-B3)
- U37 pad 1: Net-(U36-Z) -> unconnected-(U37-PE2-Pad1)
- U37 pad 2: GND -> unconnected-(U37-PE3-Pad2)
- U37 pad 3: GND -> unconnected-(U37-PE4-Pad3)
- U37 pad 4: GND -> unconnected-(U37-PE5-Pad4)
- U37 pad 5: /Main_uC/SPI1_MM -> unconnected-(U37-PE6-Pad5)
- U37 pad 6: Net-(U37-Y1) -> unconnected-(U37-VBAT-Pad6)
- U37 pad 7: Net-(U31-OE) -> unconnected-(U37-PC13-Pad7)
- U37 pad 8: Net-(U36-VCC) -> unconnected-(U37-PC14-Pad8)
- U38 pad 1: Net-(U37-Y1) -> unconnected-(U38-PE2-Pad1)
- U38 pad 10: /Main_uC/SPI1_MOSI -> unconnected-(U38-PF9-Pad10)
- U38 pad 11: /Main_uC/SYS_3V3 -> unconnected-(U38-PF10-Pad11)
- U38 pad 12: Net-(U37-Y1) -> unconnected-(U38-PF0-Pad12)
- U38 pad 2: /Main_uC/SPI1_MOSI -> unconnected-(U38-PE3-Pad2)
- U38 pad 3: /Main_uC/SPI1_SCK -> unconnected-(U38-PE4-Pad3)
- U38 pad 4: GND -> unconnected-(U38-PE5-Pad4)
- U38 pad 5: /Main_uC/SPI1_MISO -> unconnected-(U38-PE6-Pad5)
- U38 pad 6: GND -> unconnected-(U38-VBAT-Pad6)
- U38 pad 7: /Main_uC/SPI1_MISO -> unconnected-(U38-PC13-Pad7)
- U38 pad 9: /Main_uC/SPI1_SCK -> unconnected-(U38-PC15-Pad9)
Other:
- copper layers 2 -> 6

Commit message: Started some PCB layout work
Parts:
- moved R22 145.0 mm to (35.2, 34.8)
- moved C28 141.3 mm to (40.3, 20.7)
- moved R17 141.3 mm to (40.3, 28.2)
- moved R19 141.3 mm to (40.3, 33.3)
- moved C26 128.6 mm to (39.8, 38.6)
- moved U10 128.6 mm to (44.8, 33.0)
- moved R14 127.1 mm to (33.4, 30.0)
- moved C27 120.4 mm to (33.5, 26.1)
- moved R10 120.4 mm to (37.5, 26.1)
- moved R9 120.4 mm to (37.5, 23.6)
- moved C30 101.3 mm to (92.4, 35.2)
- moved U12 88.8 mm to (98.8, 34.7)
- moved R18 88.8 mm to (94.2, 43.8)
- moved C14 87.2 mm to (74.6, 25.5)
- moved C17 87.2 mm to (74.6, 33.0)
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Connections:
- RN3 pad 5: /Main_uC/GPIO_1 -> /Main_uC/_GPIO_1
- RN3 pad 6: /Main_uC/GPIO_2 -> /Main_uC/_GPIO_2
- RN3 pad 7: /Main_uC/GPIO_3 -> /Main_uC/_GPIO_3
- RN3 pad 8: /Main_uC/GPIO_4 -> /Main_uC/_GPIO_4
- RN4 pad 5: /Main_uC/GPIO_5 -> /Main_uC/_GPIO_5
- RN4 pad 6: /Main_uC/GPIO_6 -> /Main_uC/_GPIO_6
- RN4 pad 7: /Main_uC/GPIO_7 -> /Main_uC/_GPIO_7
- RN4 pad 8: /Main_uC/GPIO_8 -> /Main_uC/_GPIO_8
- U34 pad 12: /Main_uC/GPIO_8 -> /Main_uC/_GPIO_8
- U34 pad 16: /Main_uC/GPIO_5 -> /Main_uC/_GPIO_5
- U34 pad 3: /Main_uC/GPIO_6 -> /Main_uC/_GPIO_6
- U34 pad 9: /Main_uC/GPIO_7 -> /Main_uC/_GPIO_7
- U36 pad 2: /Main_uC/GPIO_1 -> /Main_uC/_GPIO_1
- U36 pad 3: /Main_uC/GPIO_2 -> /Main_uC/_GPIO_2
- U36 pad 4: /Main_uC/GPIO_3 -> /Main_uC/_GPIO_3
- U36 pad 5: /Main_uC/GPIO_4 -> /Main_uC/_GPIO_4
- U40 pad 2: /Main_uC/GPIO_5 -> /Main_uC/_GPIO_5
- U40 pad 3: /Main_uC/GPIO_6 -> /Main_uC/_GPIO_6
- U40 pad 4: /Main_uC/GPIO_7 -> /Main_uC/_GPIO_7
- U40 pad 5: /Main_uC/GPIO_8 -> /Main_uC/_GPIO_8
- U44 pad 12: /Main_uC/GPIO_4 -> /Main_uC/_GPIO_4
- U44 pad 16: /Main_uC/GPIO_1 -> /Main_uC/_GPIO_1
- U44 pad 3: /Main_uC/GPIO_2 -> /Main_uC/_GPIO_2
- U44 pad 9: /Main_uC/GPIO_3 -> /Main_uC/_GPIO_3
Routing:
- net /Main_uC/VBUS: track 0.00 -> 19.5 mm, vias 0 -> 4
- net /Main_uC/_GPIO_4: track 0.00 -> 17.9 mm, vias 0 -> 3
- net /Main_uC/_GPIO_8: track 0.00 -> 17.9 mm, vias 0 -> 3
- net /Main_uC/_GPIO_3: track 0.00 -> 17.1 mm, vias 0 -> 3
- net /Main_uC/_GPIO_7: track 0.00 -> 17.1 mm, vias 0 -> 3
- net /Main_uC/_GPIO_2: track 0.00 -> 13.3 mm, vias 0 -> 3
- net /Main_uC/_GPIO_6: track 0.00 -> 13.3 mm, vias 0 -> 3
- net /Main_uC/_GPIO_1: track 0.00 -> 13.1 mm
- net /Main_uC/_GPIO_5: track 0.00 -> 13.1 mm
- net /Main_uC/GPIO_8: track 0.00 -> 9.88 mm, vias 0 -> 2
- net /Main_uC/GPIO_4: track 0.00 -> 9.88 mm, vias 0 -> 2
- net /Main_uC/GPIO_3: track 0.00 -> 9.45 mm, vias 0 -> 2
- net /Main_uC/GPIO_7: track 0.00 -> 9.45 mm, vias 0 -> 2
- net Net-(U36-B4): track 0.00 -> 8.18 mm
- net Net-(U34-S4B): track 0.00 -> 8.18 mm
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- added copper zone on In2.Cu, net /Main_uC/SYS_3V3
- added copper zone on In1.Cu, net GND

Commit message: More PCB work
Parts:
- removed R104, R105: 10K, Resistor_SMD:R_0402_1005Metric
- added RN8: 10K, Resistor_SMD:R_Array_Convex_2x0402, F.Cu at (96.9, 124.0)
- RN7: value 0R -> 10K
- TP1, TP12, TP13, TP14, TP15, TP16, TP17, TP2, TP3, TP4, TP5, TP6, TP7, TP8, TP9: footprint TestPoint:TestPoint_Pad_D2.0mm -> TestPoint:TestPoint_Pad_D1.5mm
- U37: moved to B.Cu
- moved U35 201.7 mm to (94.0, 153.9)
- moved R100 198.6 mm to (98.0, 152.3), turned to -90 degrees
- moved C97 198.4 mm to (93.8, 151.9)
- moved U32 196.4 mm to (96.2, 152.9)
- moved RN2 195.8 mm to (96.0, 155.8), turned to 180 degrees
- moved C98 195.1 mm to (98.0, 154.3), turned to 90 degrees
- moved U29 180.2 mm to (95.6, 133.6)
- moved U46 174.9 mm to (94.6, 143.0)
- moved U30 174.5 mm to (97.5, 95.9)
- moved R95 173.3 mm to (100.3, 98.0)
- moved RN5 172.8 mm to (94.0, 96.8), turned to 180 degrees
- moved U47 172.2 mm to (98.1, 142.8)
- moved R114 172.1 mm to (98.7, 140.4), turned to 180 degrees
- moved C111 171.8 mm to (94.5, 140.4), turned to 180 degrees
- moved C94 171.2 mm to (92.8, 133.6), turned to -90 degrees
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Connections:
- RN1 pad 5: /Main_uC/SPI1_MOSI -> /Main_uC/_SPI1_MOSI
- RN1 pad 6: /Main_uC/SPI1_SCK -> /Main_uC/_SPI1_SCK
- RN1 pad 7: /Main_uC/SPI1_NSS -> /Main_uC/_SPI1_NSS
- RN1 pad 8: /Main_uC/SPI1_MISO -> /Main_uC/_SPI1_MISO
- RN2 pad 3: /Main_uC/UART1_TX -> /Main_uC/_UART1_TX
- RN2 pad 4: /Main_uC/UART1_RX -> /Main_uC/_UART1_RX
- RN6 pad 3: /Main_uC/I2C1_SCL -> /Main_uC/_I2C1_SCL
- RN6 pad 4: /Main_uC/I2C1_SDA -> /Main_uC/_I2C1_SDA
- U35 pad 4: /Main_uC/UART1_RX -> /Main_uC/_UART1_RX
- U35 pad 5: /Main_uC/UART1_TX -> /Main_uC/_UART1_TX
- U39 pad 3: /Main_uC/I2C1_SCL -> /Main_uC/_I2C1_SCL
- U39 pad 4: /Main_uC/I2C1_SDA -> /Main_uC/_I2C1_SDA
- U46 pad 2: /Main_uC/SPI1_MOSI -> /Main_uC/_SPI1_MOSI
- U46 pad 3: /Main_uC/SPI1_SCK -> /Main_uC/_SPI1_SCK
- U46 pad 4: /Main_uC/SPI1_NSS -> /Main_uC/_SPI1_NSS
- U46 pad 5: /Main_uC/SPI1_MISO -> /Main_uC/_SPI1_MISO
- U47 pad 12: /Main_uC/SPI1_MISO -> /Main_uC/_SPI1_MISO
- U47 pad 16: /Main_uC/SPI1_MOSI -> /Main_uC/_SPI1_MOSI
- U47 pad 3: /Main_uC/SPI1_SCK -> /Main_uC/_SPI1_SCK
- U47 pad 9: /Main_uC/SPI1_NSS -> /Main_uC/_SPI1_NSS
Routing:
- net /SYS_3V3: track 0.00 -> 118.5 mm, vias 0 -> 21
- net /Main_uC/VBUS: track 19.5 -> 50.1 mm, vias 4 -> 8
- net /Programmable_Regulators/SDA_CH2: track 0.00 -> 28.1 mm, vias 0 -> 2
- net /Fixed_Regulators/SDA_3V3: track 0.00 -> 28.1 mm, vias 0 -> 2
- net /Fixed_Regulators/SDA_5V: track 0.00 -> 28.1 mm, vias 0 -> 2
- net /Programmable_Regulators/SDA_CH1: track 0.00 -> 28.1 mm, vias 0 -> 2
- net /Fixed_Regulators/SCL_3V3: track 0.00 -> 27.0 mm, vias 0 -> 2
- net /Programmable_Regulators/SCL_CH2: track 0.00 -> 27.0 mm, vias 0 -> 2
- net /Fixed_Regulators/SCL_5V: track 0.00 -> 27.0 mm, vias 0 -> 2
- net /Programmable_Regulators/SCL_CH1: track 0.00 -> 27.0 mm, vias 0 -> 2
- net GNDA: track 0.00 -> 26.5 mm, vias 0 -> 52
- net /BUS_UNREG: track 0.00 -> 26.3 mm, vias 0 -> 20
- net GND: track 2.21 -> 26.1 mm, vias 8 -> 45
- net Net-(U24-SW1): track 0.00 -> 18.7 mm
- net Net-(U12-SW1): track 0.00 -> 18.7 mm
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- added copper zone on B.Cu, net (none)
- added copper zone on F.Cu, net (none)
- added copper zone on B.Cu, net /BUS_3V3
- added copper zone on F.Cu, net /BUS_3V3
- added copper zone on B.Cu, net /BUS_UNREG
- added copper zone on F.Cu, net /BUS_UNREG
- added copper zone on In2.Cu, net /BUS_UNREG
- added copper zone on B.Cu, net /SYS_5V
- added copper zone on F.Cu, net /SYS_5V
- added copper zone on In4.Cu, net GND
- added copper zone on B.Cu, net GNDA
- added copper zone on F.Cu, net GNDA
- added copper zone on In1.Cu, net GNDA
- added copper zone on In4.Cu, net GNDA
- added copper zone on B.Cu, net Net-(U10-OUT)
- added copper zone on F.Cu, net Net-(U10-OUT)
- added copper zone on B.Cu, net Net-(U11-IN)
- added copper zone on F.Cu, net Net-(U11-IN)
- added copper zone on B.Cu, net Net-(U11-OUT)
- added copper zone on F.Cu, net Net-(U11-OUT)
- added copper zone on F.Cu, net Net-(U12-SW1)
- added copper zone on F.Cu, net Net-(U12-SW2)
- added copper zone on B.Cu, net Net-(U14-OUT)
- added copper zone on F.Cu, net Net-(U14-OUT)
- added copper zone on B.Cu, net Net-(U15-IN)
- added copper zone on F.Cu, net Net-(U15-IN)
- added copper zone on F.Cu, net Net-(U16-SW1)
- added copper zone on F.Cu, net Net-(U16-SW2)
- added copper zone on B.Cu, net Net-(U18-OUT)
- added copper zone on F.Cu, net Net-(U18-OUT)
- added copper zone on B.Cu, net Net-(U19-IN)
- added copper zone on F.Cu, net Net-(U19-IN)
- added copper zone on F.Cu, net Net-(U20-SW1)
- added copper zone on F.Cu, net Net-(U20-SW2)
- added copper zone on B.Cu, net Net-(U22-OUT)
- added copper zone on F.Cu, net Net-(U22-OUT)
- added copper zone on B.Cu, net Net-(U23-IN)
- added copper zone on F.Cu, net Net-(U23-IN)
- added copper zone on F.Cu, net Net-(U24-SW1)
- added copper zone on F.Cu, net Net-(U24-SW2)
- added copper zone on B.Cu, net Net-(U26-SW)
- added copper zone on F.Cu, net Net-(U26-SW)
- added copper zone on B.Cu, net Net-(U27-SW)
- added copper zone on F.Cu, net Net-(U27-SW)
Other:
- board outline added: 90.9 x 99.5 mm

Commit message: Tried to prepare for order
Parts:
- D1, D2, D3, D4, D5, D6: value LED -> TZ-P2-0603GTCS1-0.6T
- U1: value TCA9544A -> TCA9544APWR
- U13, U17, U21, U3, U9: value INA219AxDCN -> INA219AIDCNR
- U2, U6: value DMT3006LDK -> DMT3006LDK-7
- U25: value ~ -> M20-7812045
- U26: value AP63203WU -> AP63203WU-7
- U27: value AP63205WU -> AP63205WU-7
- U28: value TPS2121 -> TPS2121RUXR
- U37: value STM32H753ZITx -> STM32H753ZIT6; moved to F.Cu
- U38: value STM32F072VBTx -> STM32F072VBT6
- U4, U7: value DML3012LDC -> DML3012LDC-7
- U41: value STM32F072VBTx -> STM32F072CBUx; footprint Package_QFP:LQFP-100_14x14mm_P0.5mm -> Package_DFN_QFN:QFN-48-1EP_7x7mm_P0.5mm_EP5.6x5.6mm
- U5, U8: value LM74700 -> AP74700QW6-7
- moved R3 134.8 mm to (78.8, 82.3)
- moved C3 132.4 mm to (82.5, 78.4)
- moved TP7 132.0 mm to (94.1, 71.1)
- moved U3 131.9 mm to (79.0, 79.3)
- moved U28 131.8 mm to (90.9, 71.6)
- moved TP10 131.5 mm to (82.9, 81.8)
- moved U38 131.3 mm to (66.4, 138.3)
- moved C93 131.2 mm to (89.9, 69.2), turned to 180 degrees
- moved R1 128.4 mm to (90.9, 88.8), turned to 90 degrees
- moved R83 128.2 mm to (93.4, 73.5), turned to 90 degrees
- moved R84 128.1 mm to (91.9, 73.9)
- moved R85 127.0 mm to (88.4, 73.5), turned to 90 degrees
- moved C7 125.0 mm to (87.1, 82.9), turned to 90 degrees
- moved R86 124.7 mm to (89.9, 73.9), turned to 180 degrees
- moved R82 124.0 mm to (92.0, 69.2), turned to 180 degrees
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Connections:
- U41 pad 23: unconnected-(U41-PA0-Pad23) -> Net-(U41-VSS-Pad23)
- U41 pad 27: Net-(U41-VSS-Pad27) -> unconnected-(U41-PB14-Pad27)
- U41 pad 35: unconnected-(U41-PB0-Pad35) -> Net-(U41-VSS-Pad23)
- U41 pad 47: unconnected-(U41-PB10-Pad47) -> Net-(U41-VSS-Pad23)
- U41 pad 49: Net-(U41-VSS-Pad27) -> Net-(U41-VSS-Pad23)
Routing:
- net Net-(Q6-G): track 0.00 -> 15.2 mm, vias 0 -> 2
- net Net-(Q5-G): track 0.00 -> 15.2 mm, vias 0 -> 2
- net Net-(D6-K): track 0.00 -> 7.07 mm
- net Net-(D5-K): track 0.00 -> 7.07 mm
- net GNDA: track 26.5 -> 33.1 mm, vias 52 -> 70
- net /SYS_5V: track 0.00 -> 5.87 mm, vias 1 -> 5
- net Net-(U8-VCAP): track 0.00 -> 4.44 mm
- net Net-(U5-VCAP): track 0.00 -> 4.44 mm
- net /System_Power/VBAT: track 0.00 -> 3.48 mm
- net /System_Power/POWER_IN: track 0.00 -> 3.47 mm
- net Net-(U28-OV2): track 0.00 -> 3.02 mm
- net Net-(U28-OV1): track 0.00 -> 2.94 mm
- net Net-(U4-BLEED): track 0.00 -> 2.71 mm
- net Net-(U7-BLEED): track 0.00 -> 2.71 mm
- net Net-(U7-SR): track 0.00 -> 2.51 mm
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- added copper zone on B.Cu, net Net-(U2-D)
- added copper zone on F.Cu, net Net-(U2-D)
- added copper zone on B.Cu, net Net-(U2-S)
- added copper zone on F.Cu, net Net-(U2-S)
- added copper zone on B.Cu, net Net-(U6-S)
- added copper zone on F.Cu, net Net-(U6-S)
