File: ESLGSU_System_Power.kicad_sch (KiCad schematic)
At the start: 53 parts, among them Q1 DMN67D7L-7, U2 DMT3006LDK, U26 AP63203WU, U27 AP63205WU, U28 TPS2121, U3 INA219AxDCN, U4 DML3012LDC, U5 LM74700, U6 DMT3006LDK, U7 DML3012LDC, U8 LM74700

Commit message: Finished interfaces work
Parts:
- C10, C11, C12, C2, C3, C4, C5, C6, C7, C8, C85, C89, C9, C93: footprint Capacitor_SMD:C_0603_1608Metric -> Capacitor_SMD:C_0402_1005Metric
- R1, R2, R4, R5, R8, R82, R83, R84, R85, R86: footprint Resistor_SMD:R_0603_1608Metric -> Resistor_SMD:R_0402_1005Metric
Changed lines of the file:
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@@
       (effects (font (size 1.27 1.27)) (justify left))
     )
-    (property "Footprint" "Capacitor_SMD:C_0603_1608Metric" (at 168.91 111.76 0)
+    (property "Footprint" "Capacitor_SMD:C_0402_1005Metric" (at 168.91 111.76 0)
       (effects (font (size 1.27 1.27)) hide)
     )
@@
       (effects (font (size 1.27 1.27)) (justify right))
     )
-    (property "Footprint" "Resistor_SMD:R_0603_1608Metric" (at 44.45 161.29 0)
+    (property "Footprint" "Resistor_SMD:R_0402_1005Metric" (at 44.45 161.29 0)
       (effects (font (size 1.27 1.27)) hide)
     )
@@
       (effects (font (size 1.27 1.27)))
     )
-    (property "Footprint" "Capacitor_SMD:C_0603_1608Metric" (at 124.46 147.32 0)
+    (property "Footprint" "Capacitor_SMD:C_0402_1005Metric" (at 124.46 147.32 0)
       (effects (font (size 1.27 1.27)) hide)
     )
@@
       (effects (font (size 1.27 1.27)) (justify right))
     )
-    (property "Footprint" "Resistor_SMD:R_0603_1608Metric" (at 71.12 163.83 0)
+    (property "Footprint" "Resistor_SMD:R_0402_1005Metric" (at 71.12 163.83 0)
       (effects (font (size 1.27 1.27)) hide)
     )
@@
       (effects (font (size 1.27 1.27)) (justify left))
     )
-    (property "Footprint" "Capacitor_SMD:C_0603_1608Metric" (at 200.66 36.83 0)
+    (property "Footprint" "Capacitor_SMD:C_0402_1005Metric" (at 200.66 36.83 0)
       (effects (font (size 1.27 1.27)) hide)
     )
@@
       (effects (font (size 1.27 1.27)))
     )
-    (property "Footprint" "Capacitor_SMD:C_0603_1608Metric" (at 74.93 161.29 0)
+    (property "Footprint" "Capacitor_SMD:C_0402_1005Metric" (at 74.93 161.29 0)
       (effects (font (size 1.27 1.27)) hide)
     )
@@
       (effects (font (size 1.27 1.27)))
     )
-    (property "Footprint" "Resistor_SMD:R_0603_1608Metric" (at 144.78 104.14 0)
+    (property "Footprint" "Resistor_SMD:R_0402_1005Metric" (at 144.78 104.14 0)
       (effects (font (size 1.27 1.27)) hide)
     )
@@
       (effects (font (size 1.27 1.27)) (justify left))
     )
-    (property "Footprint" "Capacitor_SMD:C_0603_1608Metric" (at 200.66 93.98 0)
+    (property "Footprint" "Capacitor_SMD:C_0402_1005Metric" (at 200.66 93.98 0)
       (effects (font (size 1.27 1.27)) hide)
     )
@@
       (effects (font (size 1.27 1.27)))
     )
-    (property "Footprint" "Capacitor_SMD:C_0603_1608Metric" (at 124.46 179.07 0)
+    (property "Footprint" "Capacitor_SMD:C_0402_1005Metric" (at 124.46 179.07 0)
       (effects (font (size 1.27 1.27)) hide)
     )
@@
       (effects (font (size 1.27 1.27)) (justify left))
     )
-    (property "Footprint" "Resistor_SMD:R_0603_1608Metric" (at 148.59 39.37 0)
+    (property "Footprint" "Resistor_SMD:R_0402_1005Metric" (at 148.59 39.37 0)
       (effects (font (size 1.27 1.27)) hide)
     )
@@
       (effects (font (size 1.27 1.27)))
     )
-    (property "Footprint" "Resistor_SMD:R_0603_1608Metric" (at 144.78 46.99 0)
+    (property "Footprint" "Resistor_SMD:R_0402_1005Metric" (at 144.78 46.99 0)
       (effects (font (size 1.27 1.27)) hide)
     )
@@
       (effects (font (size 1.27 1.27)) (justify left))
     )
-    (property "Footprint" "Capacitor_SMD:C_0603_1608Metric" (at 110.49 82.55 0)
+    (property "Footprint" "Capacitor_SMD:C_0402_1005Metric" (at 110.49 82.55 0)
       (effects (font (size 1.27 1.27)) hide)
     )
@@
       (effects (font (size 1.27 1.27)) (justify left))
     )
-    (property "Footprint" "Capacitor_SMD:C_0603_1608Metric" (at 166.37 93.98 0)
+    (property "Footprint" "Capacitor_SMD:C_0402_1005Metric" (at 166.37 93.98 0)
       (effects (font (size 1.27 1.27)) hide)
     )
@@
       (effects (font (size 1.27 1.27)) (justify left))
     )
-    (property "Footprint" "Resistor_SMD:R_0603_1608Metric" (at 148.59 96.52 0)
+    (property "Footprint" "Resistor_SMD:R_0402_1005Metric" (at 148.59 96.52 0)
       (effects (font (size 1.27 1.27)) hide)
     )
@@
       (effects (font (size 1.27 1.27)) (justify left))
     )
-    (property "Footprint" "Capacitor_SMD:C_0603_1608Metric" (at 110.49 25.4 0)
+    (property "Footprint" "Capacitor_SMD:C_0402_1005Metric" (at 110.49 25.4 0)
       (effects (font (size 1.27 1.27)) hide)
     )
@@
       (effects (font (size 1.27 1.27)) (justify right))
     )
-    (property "Footprint" "Resistor_SMD:R_0603_1608Metric" (at 41.91 157.48 0)
+    (property "Footprint" "Resistor_SMD:R_0402_1005Metric" (at 41.91 157.48 0)
       (effects (font (size 1.27 1.27)) hide)
     )
@@
       (effects (font (size 1.27 1.27)) (justify right))
     )
-    (property "Footprint" "Resistor_SMD:R_0603_1608Metric" (at 44.45 151.13 0)
+    (property "Footprint" "Resistor_SMD:R_0402_1005Metric" (at 44.45 151.13 0)
       (effects (font (size 1.27 1.27)) hide)
     )
@@
       (effects (font (size 1.27 1.27)) (justify left))
     )
-    (property "Footprint" "Resistor_SMD:R_0603_1608Metric" (at 157.48 90.17 0)
+    (property "Footprint" "Resistor_SMD:R_0402_1005Metric" (at 157.48 90.17 0)
       (effects (font (size 1.27 1.27)) hide)
     )
@@
       (effects (font (size 1.27 1.27)) (justify right))
     )
-    (property "Footprint" "Resistor_SMD:R_0603_1608Metric" (at 41.91 147.32 0)
+    (property "Footprint" "Resistor_SMD:R_0402_1005Metric" (at 41.91 147.32 0)
       (effects (font (size 1.27 1.27)) hide)
     )
@@
       (effects (font (size 1.27 1.27)) (justify left))
     )
-    (property "Footprint" "Capacitor_SMD:C_0603_1608Metric" (at 110.49 109.22 0)
+    (property "Footprint" "Capacitor_SMD:C_0402_1005Metric" (at 110.49 109.22 0)
       (effects (font (size 1.27 1.27)) hide)
     )
@@
       (effects (font (size 1.27 1.27)) (justify left))
     )
-    (property "Footprint" "Capacitor_SMD:C_0603_1608Metric" (at 222.25 26.67 0)
+    (property "Footprint" "Capacitor_SMD:C_0402_1005Metric" (at 222.25 26.67 0)
       (effects (font (size 1.27 1.27)) hide)
     )
@@
       (effects (font (size 1.27 1.27)) (justify left))
     )
-    (property "Footprint" "Capacitor_SMD:C_0603_1608Metric" (at 110.49 52.07 0)
+    (property "Footprint" "Capacitor_SMD:C_0402_1005Metric" (at 110.49 52.07 0)
       (effects (font (size 1.27 1.27)) hide)
     )
@@
       (effects (font (size 1.27 1.27)) (justify left))
     )
-    (property "Footprint" "Capacitor_SMD:C_0603_1608Metric" (at 168.91 54.61 0)
+    (property "Footprint" "Capacitor_SMD:C_0402_1005Metric" (at 168.91 54.61 0)
       (effects (font (size 1.27 1.27)) hide)
     )
@@
       (effects (font (size 1.27 1.27)) (justify left))
     )
-    (property "Footprint" "Resistor_SMD:R_0603_1608Metric" (at 157.48 33.02 0)
+    (property "Footprint" "Resistor_SMD:R_0402_1005Metric" (at 157.48 33.02 0)
       (effects (font (size 1.27 1.27)) hide)
     )
@@
       (effects (font (size 1.27 1.27)) (justify left))
     )
-    (property "Footprint" "Capacitor_SMD:C_0603_1608Metric" (at 166.37 36.83 0)
-      (effects (font (size 1.27 1.27)) hide)
-    )
+    (property "Footprint" "Capacitor_SMD:C_0402_1005Metric" (at 166.37 36.83 0)
+      (effects (font (size 1.27 1.27)) hide)
+    )

Commit message: More PCB work
Parts:
- TP1: footprint TestPoint:TestPoint_Pad_D2.0mm -> TestPoint:TestPoint_Pad_D1.5mm
Changed lines of the file:
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@@
       (effects (font (size 1.27 1.27)) (justify left))
     )
-    (property "Footprint" "TestPoint:TestPoint_Pad_D2.0mm" (at 90.17 144.78 0)
+    (property "Footprint" "TestPoint:TestPoint_Pad_D1.5mm" (at 90.17 144.78 0)
       (effects (font (size 1.27 1.27)) hide)
     )
@@
       (effects (font (size 1.27 1.27)) (justify left))
     )
-    (property "Footprint" "TestPoint:TestPoint_Pad_D2.0mm" (at 161.29 176.53 0)
+    (property "Footprint" "TestPoint:TestPoint_Pad_D1.5mm" (at 161.29 176.53 0)
       (effects (font (size 1.27 1.27)) hide)
     )
@@
       (effects (font (size 1.27 1.27)) (justify left))
     )
-    (property "Footprint" "TestPoint:TestPoint_Pad_D2.0mm" (at 161.29 144.78 0)
-      (effects (font (size 1.27 1.27)) hide)
-    )
+    (property "Footprint" "TestPoint:TestPoint_Pad_D1.5mm" (at 161.29 144.78 0)
+      (effects (font (size 1.27 1.27)) hide)
+    )

Commit message: Tried to prepare for order
Parts:
- D1: value LED -> TZ-P2-0603GTCS1-0.6T
- U2, U6: value DMT3006LDK -> DMT3006LDK-7
- U26: value AP63203WU -> AP63203WU-7
- U27: value AP63205WU -> AP63205WU-7
- U28: value TPS2121 -> TPS2121RUXR
- U3: value INA219AxDCN -> INA219AIDCNR
- U4, U7: value DML3012LDC -> DML3012LDC-7
- U5, U8: value LM74700 -> AP74700QW6-7
Changed lines of the file:
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@@
       (effects (font (size 1.27 1.27)))
     )
-    (property "Value" "DMT3006LDK" (at 195.58 80.01 90)
+    (property "Value" "DMT3006LDK-7" (at 195.58 80.01 90)
       (effects (font (size 1.27 1.27)))
     )
@@
       (effects (font (size 1.27 1.27)) (justify left))
     )
-    (property "Value" "LM74700" (at 189.23 114.3 0)
+    (property "Value" "AP74700QW6-7" (at 189.23 114.3 0)
       (effects (font (size 1.27 1.27)) (justify left))
     )
@@
       (effects (font (size 1.27 1.27)))
     )
-    (property "Value" "TPS2121" (at 60.96 139.7 0)
+    (property "Value" "TPS2121RUXR" (at 60.96 139.7 0)
       (effects (font (size 1.27 1.27)))
     )
@@
       (effects (font (size 1.27 1.27)) (justify right))
     )
-    (property "Value" "LED" (at 152.4 39.37 90)
+    (property "Value" "TZ-P2-0603GTCS1-0.6T" (at 152.4 39.37 90)
       (effects (font (size 1.27 1.27)) (justify right))
     )
@@
       (effects (font (size 1.27 1.27)))
     )
-    (property "Value" "DMT3006LDK" (at 195.58 22.86 90)
+    (property "Value" "DMT3006LDK-7" (at 195.58 22.86 90)
       (effects (font (size 1.27 1.27)))
     )
@@
       (effects (font (size 1.27 1.27)) (justify left))
     )
-    (property "Value" "INA219AxDCN" (at 238.4141 25.4 0)
+    (property "Value" "INA219AIDCNR" (at 238.4141 25.4 0)
       (effects (font (size 1.27 1.27)) (justify left))
     )
@@
       (effects (font (size 1.27 1.27)) (justify left))
     )
-    (property "Value" "DML3012LDC" (at 138.43 86.36 0)
+    (property "Value" "DML3012LDC-7" (at 138.43 86.36 0)
       (effects (font (size 1.27 1.27)))
     )
@@
       (effects (font (size 1.27 1.27)) (justify right))
     )
-    (property "Value" "LED" (at 152.4 96.52 90)
+    (property "Value" "TZ-P2-0603GTCS1-0.6T" (at 152.4 96.52 90)
       (effects (font (size 1.27 1.27)) (justify right))
     )
@@
       (effects (font (size 1.27 1.27)))
     )
-    (property "Value" "AP63203WU" (at 111.76 171.45 0)
+    (property "Value" "AP63203WU-7" (at 111.76 171.45 0)
       (effects (font (size 1.27 1.27)))
     )
@@
       (effects (font (size 1.27 1.27)) (justify left))
     )
-    (property "Value" "DML3012LDC" (at 138.43 29.21 0)
+    (property "Value" "DML3012LDC-7" (at 138.43 29.21 0)
       (effects (font (size 1.27 1.27)))
     )
@@
       (effects (font (size 1.27 1.27)))
     )
-    (property "Value" "AP63205WU" (at 111.76 139.7 0)
+    (property "Value" "AP63205WU-7" (at 111.76 139.7 0)
       (effects (font (size 1.27 1.27)))
     )
@@
       (effects (font (size 1.27 1.27)) (justify left))
     )
-    (property "Value" "LM74700" (at 189.23 57.15 0)
-      (effects (font (size 1.27 1.27)) (justify left))
-    )
+    (property "Value" "AP74700QW6-7" (at 189.23 57.15 0)
+      (effects (font (size 1.27 1.27)) (justify left))
+    )
