File: ESLGSU_System_Power.kicad_sch (KiCad schematic)
At the start: 87 parts, among them J2 XT60U-M, Q1 RE1C002UNTCL, U10 AP63205WU-7, U11 TPS2121RUXR, U12 AP63203WU-7, U2 VBQF1303, U3 INA219AIDCNR, U4 NCP45770IMN24TWG, U5 AP74700QW6-7, U6 VBQF1303, U7 MP2651GVT, U8 NCP45770IMN24TWG, U9 AP74700QW6-7

Commit message: Fixes for next version
Parts:
- added R33: 200K, Resistor_SMD:R_0402_1005Metric, symbol Device:R_Small_US
- R8: value 200R -> 300R; LCSC Part C25087 -> C25102
- U4, U8: footprint Package_DFN_QFN:WDFN-12-1EP_3x3mm_P0.45mm_EP1.7x2.5mm -> Package_DFN_QFN:DFN-12-1EP_3x3mm_P0.5mm_EP1.6x2.5mm
Connections:
- net BUS_UNREG: now also R33.1
- net EPS_SCL: now also U3.7 (A0), U3.8 (A1)
- net GND: now also R33.2; no longer U3.7 (A0), U3.8 (A1)
Other:
- note added: "Adr: 1001111"
- note removed: "Adr: 1000000"
Changed lines of the file:
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@@
   (junction (at 58.42 34.29) (diameter 0) (color 0 0 0 0)
   )
+  (junction (at 246.38 38.1) (diameter 0) (color 0 0 0 0)
+  )
   (junction (at 45.72 41.91) (diameter 0) (color 0 0 0 0)
   )
+  (junction (at 223.52 45.72) (diameter 0) (color 0 0 0 0)
+  )
   (junction (at 194.31 91.44) (diameter 0) (color 0 0 0 0)
   )
@@
   (junction (at 27.94 34.29) (diameter 0) (color 0 0 0 0)
   )
-  (junction (at 246.38 40.64) (diameter 0) (color 0 0 0 0)
-  )
   (junction (at 45.72 78.74) (diameter 0) (color 0 0 0 0)
   )
@@
   (junction (at 69.85 144.78) (diameter 0) (color 0 0 0 0)
   )
+  (junction (at 246.38 33.02) (diameter 0) (color 0 0 0 0)
+  )
   (junction (at 200.66 91.44) (diameter 0) (color 0 0 0 0)
   )
@@
     (stroke (width 0) (type default))
   )
-  (wire (pts (xy 223.52 38.1) (xy 223.52 55.88))
+  (wire (pts (xy 223.52 38.1) (xy 223.52 45.72))
     (stroke (width 0) (type default))
   )
@@
     (stroke (width 0) (type default))
   )
+  (wire (pts (xy 223.52 45.72) (xy 223.52 55.88))
+    (stroke (width 0) (type default))
+  )
   (wire (pts (xy 85.09 144.78) (xy 85.09 176.53))
     (stroke (width 0) (type default))
@@
     (stroke (width 0) (type default))
   )
+  (wire (pts (xy 246.38 33.02) (xy 246.38 38.1))
+    (stroke (width 0) (type default))
+  )
   (wire (pts (xy 129.54 22.86) (xy 148.59 22.86))
     (stroke (width 0) (type default))
@@
     (stroke (width 0) (type default))
   )
-  (wire (pts (xy 246.38 45.72) (xy 236.22 45.72))
-    (stroke (width 0) (type default))
-  )
   (wire (pts (xy 157.48 100.33) (xy 157.48 101.6))
     (stroke (width 0) (type default))
@@
     (stroke (width 0) (type default))
   )
-  (wire (pts (xy 246.38 40.64) (xy 246.38 45.72))
-    (stroke (width 0) (type default))
-  )
   (wire (pts (xy 157.48 80.01) (xy 148.59 80.01))
     (stroke (width 0) (type default))
@@
     (stroke (width 0) (type default))
   )
+  (wire (pts (xy 223.52 45.72) (xy 226.06 45.72))
+    (stroke (width 0) (type default))
+  )
   (wire (pts (xy 101.6 176.53) (xy 101.6 181.61))
     (stroke (width 0) (type default))
@@
     (stroke (width 0) (type default))
   )
+  (wire (pts (xy 231.14 45.72) (xy 236.22 45.72))
+    (stroke (width 0) (type default))
+  )
   (wire (pts (xy 48.26 78.74) (xy 48.26 81.28))
     (stroke (width 0) (type default))
@@
     (effects (font (size 1.27 1.27)) (justify left bottom))
   )
-  (text "Adr: 1000000" (at 248.92 40.64 0)
+  (text "Adr: 1001111" (at 248.92 40.64 0)
     (effects (font (size 1.27 1.27)) (justify left bottom))
   )
@@
       (effects (font (size 1.27 1.27)))
     )
-    (property "Footprint" "Package_DFN_QFN:WDFN-12-1EP_3x3mm_P0.45mm_EP1.7x2.5mm" (at 118.11 86.36 0)
+    (property "Footprint" "Package_DFN_QFN:DFN-12-1EP_3x3mm_P0.5mm_EP1.6x2.5mm" (at 118.11 86.36 0)
       (effects (font (size 1.27 1.27)) hide)
     )
@@
     )
   )
+  (symbol (lib_id "Device:R_Small_US") (at 228.6 45.72 90) (unit 1)
+    (in_bom yes) (on_board yes) (dnp no)
+    (property "Reference" "R33" (at 231.14 48.26 90)
+      (effects (font (size 1.27 1.27)) (justify left))
+    )
+    (property "Value" "200K" (at 232.41 50.8 90)
+      (effects (font (size 1.27 1.27)) (justify left))
+    )
+    (property "Footprint" "Resistor_SMD:R_0402_1005Metric" (at 228.6 45.72 0)
+      (effects (font (size 1.27 1.27)) hide)
+    )
+    (property "Datasheet" "~" (at 228.6 45.72 0)
+      (effects (font (size 1.27 1.27)) hide)
+    )
+    (property "LCSC Part" "C25764" (at 231.14 43.18 90)
+      (effects (font (size 1.27 1.27)) hide)
+    )
+    (pin "1")
+    (pin "2")
+    (instances
+      (project "ESLGSU"
+        (path "/b556fa32-e0cb-409c-ac85-9f2ac606be79/09a64186-e4de-4db7-b903-c6397ff9a54d"
+          (reference "R33") (unit 1)
+        )
+        (path "/b556fa32-e0cb-409c-ac85-9f2ac606be79/e09c623d-ecce-4ff2-a230-f07fbe15280b"
+          (reference "R297") (unit 1)
+        )
+      )
+    )
+  )
   (symbol (lib_id "Connector:TestPoint") (at 166.37 91.44 0) (unit 1)
     (in_bom no) (on_board yes) (dnp no) (fields_autoplaced)
@@
       (effects (font (size 1.27 1.27)) (justify left))
     )
-    (property "Value" "200R" (at 156.3556 31.7663 90)
+    (property "Value" "300R" (at 156.3556 31.7663 90)
       (effects (font (size 1.27 1.27)) (justify left))
     )
@@
       (effects (font (size 1.27 1.27)) hide)
     )
-    (property "LCSC Part" "C25087" (at 156.3556 31.7663 90)
+    (property "LCSC Part" "C25102" (at 156.3556 31.7663 90)
       (effects (font (size 1.27 1.27)) hide)
     )
@@
       (effects (font (size 1.27 1.27)) (justify left))
     )
-    (property "Value" "200R" (at 156.3556 88.9163 90)
+    (property "Value" "300R" (at 156.3556 88.9163 90)
       (effects (font (size 1.27 1.27)) (justify left))
     )
@@
       (effects (font (size 1.27 1.27)) hide)
     )
-    (property "LCSC Part" "C25087" (at 156.3556 88.9163 90)
+    (property "LCSC Part" "C25102" (at 156.3556 88.9163 90)
       (effects (font (size 1.27 1.27)) hide)
     )
@@
       (effects (font (size 1.27 1.27)))
     )
-    (property "Footprint" "Package_DFN_QFN:WDFN-12-1EP_3x3mm_P0.45mm_EP1.7x2.5mm" (at 118.11 29.21 0)
+    (property "Footprint" "Package_DFN_QFN:DFN-12-1EP_3x3mm_P0.5mm_EP1.6x2.5mm" (at 118.11 29.21 0)
       (effects (font (size 1.27 1.27)) hide)
     )
