File: ESLGSU_Fixed_Regulators.kicad_sch (KiCad schematic)
At the start: 98 parts, among them Q1 DMN67D7L-7, Q2 DMN67D7L-7, U10 TPS259474LRPWR, U11 LM73100RPWR, U12 MP28167-A, U14 TPS259474LRPWR, U15 LM73100RPWR, U16 MP28167-A, U5 INA219AxDCN

Commit message: More PCB work
Parts:
- TP1, TP2, TP3, TP4, TP5, TP6: footprint TestPoint:TestPoint_Pad_D2.0mm -> TestPoint:TestPoint_Pad_D1.5mm
Changed lines of the file:
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@@
       (effects (font (size 1.27 1.27)) (justify left))
     )
-    (property "Footprint" "TestPoint:TestPoint_Pad_D2.0mm" (at 92.71 111.76 0)
+    (property "Footprint" "TestPoint:TestPoint_Pad_D1.5mm" (at 92.71 111.76 0)
       (effects (font (size 1.27 1.27)) hide)
     )
@@
       (effects (font (size 1.27 1.27)) (justify left))
     )
-    (property "Footprint" "TestPoint:TestPoint_Pad_D2.0mm" (at 238.76 68.58 0)
+    (property "Footprint" "TestPoint:TestPoint_Pad_D1.5mm" (at 238.76 68.58 0)
       (effects (font (size 1.27 1.27)) hide)
     )
@@
       (effects (font (size 1.27 1.27)) (justify left))
     )
-    (property "Footprint" "TestPoint:TestPoint_Pad_D2.0mm" (at 156.21 111.76 0)
+    (property "Footprint" "TestPoint:TestPoint_Pad_D1.5mm" (at 156.21 111.76 0)
       (effects (font (size 1.27 1.27)) hide)
     )
@@
       (effects (font (size 1.27 1.27)) (justify left))
     )
-    (property "Footprint" "TestPoint:TestPoint_Pad_D2.0mm" (at 156.21 45.72 0)
+    (property "Footprint" "TestPoint:TestPoint_Pad_D1.5mm" (at 156.21 45.72 0)
       (effects (font (size 1.27 1.27)) hide)
     )
@@
       (effects (font (size 1.27 1.27)) (justify left))
     )
-    (property "Footprint" "TestPoint:TestPoint_Pad_D2.0mm" (at 238.76 134.62 0)
+    (property "Footprint" "TestPoint:TestPoint_Pad_D1.5mm" (at 238.76 134.62 0)
       (effects (font (size 1.27 1.27)) hide)
     )
@@
       (effects (font (size 1.27 1.27)) (justify left))
     )
-    (property "Footprint" "TestPoint:TestPoint_Pad_D2.0mm" (at 92.71 45.72 0)
-      (effects (font (size 1.27 1.27)) hide)
-    )
+    (property "Footprint" "TestPoint:TestPoint_Pad_D1.5mm" (at 92.71 45.72 0)
+      (effects (font (size 1.27 1.27)) hide)
+    )

Commit message: Tried to prepare for order
Parts:
- D1, D2: value LED -> TZ-P2-0603GTCS1-0.6T
- U5: value INA219AxDCN -> INA219AIDCNR
Changed lines of the file:
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@@
       (effects (font (size 1.27 1.27)) (justify left))
     )
-    (property "Value" "INA219AxDCN" (at 249.8441 38.1 0)
+    (property "Value" "INA219AIDCNR" (at 249.8441 38.1 0)
       (effects (font (size 1.27 1.27)) (justify left))
     )
@@
       (effects (font (size 1.27 1.27)) (justify right))
     )
-    (property "Value" "LED" (at 220.98 109.22 90)
+    (property "Value" "TZ-P2-0603GTCS1-0.6T" (at 220.98 109.22 90)
       (effects (font (size 1.27 1.27)) (justify right))
     )
@@
       (effects (font (size 1.27 1.27)) (justify right))
     )
-    (property "Value" "LED" (at 220.98 43.18 90)
+    (property "Value" "TZ-P2-0603GTCS1-0.6T" (at 220.98 43.18 90)
       (effects (font (size 1.27 1.27)) (justify right))
     )
@@
       (effects (font (size 1.27 1.27)) (justify left))
     )
-    (property "Value" "INA219AxDCN" (at 249.8441 104.14 0)
-      (effects (font (size 1.27 1.27)) (justify left))
-    )
+    (property "Value" "INA219AIDCNR" (at 249.8441 104.14 0)
+      (effects (font (size 1.27 1.27)) (justify left))
+    )

Commit message: Schematic work
Parts:
- added R101: 200K, Resistor_SMD:R_0402_1005Metric, symbol Device:R_Small_US
- added R102: 15K, Resistor_SMD:R_0402_1005Metric, symbol Device:R_Small_US
- C13, C14, C16, C25, C31, C32, C34, C43, C6: LCSC Part (none) -> C307331
- C17, C35: LCSC Part (none) -> C134220
- C18, C20, C21, C22, C23, C24, C36, C38, C39, C40, C41, C42: LCSC Part (none) -> C45783
- C19, C37: LCSC Part (none) -> C1532
- C26, C29, C30, C44, C47, C48: LCSC Part (none) -> C52923
- C27, C45: value 330p -> 220p; LCSC Part (none) -> C1530
- C28, C46: LCSC Part (none) -> C1531
- D1, D2: LCSC Part (none) -> C2286
- L1, L2: value IHLP4040DZER4R7M01 -> SRP1038A-4R7M; LCSC Part (none) -> C2041319
- Q1, Q2: value DMN67D7L-7 -> RE1C002UNTCL; footprint Package_TO_SOT_SMD:SOT-23 -> Package_TO_SOT_SMD:SOT-416; LCSC Part (none) -> C509959
- R10, R27: value 47K -> 33K; LCSC Part (none) -> C25779
- R11: value 430K -> 150K; LCSC Part (none) -> C25755
- R12: value 31.6K -> 22K; LCSC Part (none) -> C25768
- R14, R31: value 17.4K -> 12K; LCSC Part (none) -> C25752
- R15, R32: value 806K -> 200K; LCSC Part (none) -> C25764
- R16: value 3.74K -> 1.5K; LCSC Part (none) -> C25867
- R17, R34: value 14.7K -> 10K; LCSC Part (none) -> C25744
- R18: value 187K -> 330K; LCSC Part (none) -> C25778
- R19, R36: value 7.5K -> 5.1K; LCSC Part (none) -> C25905
- R2: LCSC Part (none) -> C25900
- R2: LCSC Part (none) -> C346483
- R20: value 16.9K -> 12K; LCSC Part (none) -> C25752
- R21, R38: value 21.5K -> 22K; LCSC Part (none) -> C25768
- R22, R39: value 549R -> 1K; LCSC Part (none) -> C11702
- R23, R24, R6, R7: LCSC Part (none) -> C17168
- R25, R8: value 100R -> 33R; LCSC Part (none) -> C25105
- R26, R9: value 100K -> 68K; LCSC Part (none) -> C36871
- R28: value 430K -> 100K; LCSC Part (none) -> C25741
- R29: value 31.6K -> 51K; LCSC Part (none) -> C25794
- R33: value 2.09K -> 2.2K; LCSC Part (none) -> C25879
- R35: value 107K -> 75K; LCSC Part (none) -> C25798
- R37: value 9.09K -> 15K; LCSC Part (none) -> C25756
- R87, R88: LCSC Part (none) -> C25792
- TP1, TP2, TP3, TP4, TP5, TP6: JLCPCB BOM (none) -> 0; now left out of the parts list
- U10, U14: LCSC Part (none) -> C3662807
- U11, U15: LCSC Part (none) -> C3210761
- U5: LCSC Part (none) -> C87469
Connections:
- net GNDA: now also R11.2; no longer R18.2
- net SYS_3V3: now also R87.1, R88.1
- net at D1.2 (A), R8.2: no longer R87.1
- net at C20.1, C21.1, C22.1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: now also R102.1; no longer R11.1
- net at D2.2 (A), R25.2: no longer R88.1
- net at R32.2, R35.1: now also R101.2; no longer R28.2
- new net: R11.1, R15.2, R18.2
- new net: R101.1, R28.2
- new net: R102.2, R18.1
Other:
- note added: "1.39-4.65V"
- note added: "6A limit 7.5V/ms"
- note added: "gets pulled up to max 4V"
- note removed: "1.28-4.76V"
- note removed: "6A limit 5V/ms"
- moved on the sheet: R35, R87, R88
