File: ESLGSU_Fixed_Regulators.kicad_sch (KiCad schematic)
At the start: 98 parts, among them Q3 RE1C002UNTCL, Q4 RE1C002UNTCL, U14 LM73100RPWR, U15 TPS259474LRPWR, U16 MP28167GQ-A, U18 LM73100RPWR, U19 TPS259474LRPWR, U20 MP28167GQ-A, U5 INA219AIDCNR

Commit message: Final V1 board with notes
Other:
- note added: "Add high-Z pulldown"
- note added: "Pullup LED from other source"
Changed lines of the file:
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@@
+    (effects (font (size 1.27 1.27)) (justify left bottom))
+  )
+  (text "Pullup LED from other source" (at 204.47 26.67 0)
     (effects (font (size 1.27 1.27)) (justify left bottom))
   )
@@
     (effects (font (size 1.27 1.27)) (justify left bottom))
   )
+  (text "Add high-Z pulldown" (at 232.41 71.12 0)
+    (effects (font (size 1.27 1.27)) (justify left bottom))
+  )
