File: ESLGSU_Fixed_Regulators.kicad_sch (KiCad schematic)
At the start: 100 parts, among them Q1 RE1C002UNTCL, Q2 RE1C002UNTCL, U10 TPS259474LRPWR, U11 LM73100RPWR, U12 MP28167-A, U14 TPS259474LRPWR, U15 LM73100RPWR, U16 MP28167-A, U5 INA219AIDCNR

Commit message: Second last bit of schematic work
Parts:
- removed R10, R27: 33K, Resistor_SMD:R_0402_1005Metric, symbol Device:R_Small_US
- removed R17, R34: 10K, Resistor_SMD:R_0402_1005Metric, symbol Device:R_Small_US
Connections:
- net EN_3V3: now also U12.3 (EN); no longer R14.1, R9.2, U10.1 (EN/UVLO), U10.4 (PGTH)
- net EN_5V: now also U16.3 (EN); no longer R26.2, R31.1, U14.1 (EN/UVLO), U14.4 (PGTH)
- net at U14.3 (PG): no longer U16.3 (EN)
- net at U10.3 (PG): no longer U12.3 (EN)
- new net EN_3V3_EF: R14.1, R9.2, U10.1 (EN/UVLO), U10.4 (PGTH)
- new net EN_5V_EF: R26.2, R31.1, U14.1 (EN/UVLO), U14.4 (PGTH)
- no-connect marks 2 -> 4
Other:
- note removed: "1.39-4.65V"

Commit message: Final schematic work, added battery charger, linked everything up
Parts:
- Q1, Q2: footprint Package_TO_SOT_SMD:SOT-416 -> Package_TO_SOT_SMD:SOT-23
Changed lines of the file:
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@@
           (reference "R25") (unit 1)
-        )
-        (path "/b556fa32-e0cb-409c-ac85-9f2ac606be79/bf0312e4-5726-4684-b2e9-b4b5c1d8e876"
-          (reference "R122") (unit 1)
         )
       )
@@
         (path "/b556fa32-e0cb-409c-ac85-9f2ac606be79/09a64186-e4de-4db7-b903-c6397ff9a54d"
           (reference "R8") (unit 1)
-        )
-        (path "/b556fa32-e0cb-409c-ac85-9f2ac606be79/bf0312e4-5726-4684-b2e9-b4b5c1d8e876"
-          (reference "R122") (unit 1)
         )
       )
@@
       (effects (font (size 1.27 1.27)) (justify left))
     )
-    (property "Footprint" "Package_TO_SOT_SMD:SOT-416" (at 228.6 55.245 0)
+    (property "Footprint" "Package_TO_SOT_SMD:SOT-23" (at 228.6 55.245 0)
       (effects (font (size 1.27 1.27) italic) (justify left) hide)
     )
@@
       (effects (font (size 1.27 1.27)) (justify left))
     )
-    (property "Footprint" "Package_TO_SOT_SMD:SOT-416" (at 228.6 121.285 0)
+    (property "Footprint" "Package_TO_SOT_SMD:SOT-23" (at 228.6 121.285 0)
       (effects (font (size 1.27 1.27) italic) (justify left) hide)
     )

Commit message: Last tweaks on schematic
Parts:
- removed R14, R31: 12K, Resistor_SMD:R_0402_1005Metric, symbol Device:R_Small_US
- removed R2 (x2): 5m, Resistor_SMD:R_0603_1608Metric, symbol Device:R_Small_US
- removed R26: 68K, Resistor_SMD:R_0402_1005Metric, symbol Device:R_Small_US
- added R3 (x2): 5m, Resistor_SMD:R_1206_3216Metric, symbol Device:R_Small_US
- added R32, R50: 8.2K, Resistor_SMD:R_0402_1005Metric, symbol Device:R_Small_US
- added R46: 200K, Resistor_SMD:R_0402_1005Metric, symbol Device:R_Small_US
- added R54: 27K, Resistor_SMD:R_0402_1005Metric, symbol Device:R_Small_US
- added R55: 15K, Resistor_SMD:R_0402_1005Metric, symbol Device:R_Small_US
- R28: renamed from R9; value 68K -> 200K; LCSC Part C36871 -> C25764
- R36: value 5.1K -> 27K; LCSC Part C25905 -> C25771
- R37: renamed from R19; value 5.1K -> 15K; LCSC Part C25905 -> C25756
- renumbered C13 to C36, C14 to C37, C16 to C39, C17 to C40, C18 to C41, C19 to C42, C20 to C43, C21 to C44, C22 to C45, C23 to C46, C24 to C47, C25 to C48, C26 to C49, C27 to C50, C28 to C51, C29 to C52, C30 to C53, C31 to C54, C32 to C55, C34 to C57, C35 to C58, C36 to C59, C37 to C60, C38 to C61, C39 to C62, C40 to C63, C41 to C64, C42 to C65, C43 to C66, C44 to C67, C45 to C68, C46 to C69, C47 to C70, C48 to C71, D1 to D3, D2 to D4, L1 to L4, L2 to L5, Q1 to Q3, Q2 to Q4, R6 to R24, R7 to R25, R87 to R26, R8 to R27, R102 to R29, R12 to R30, R15 to R33, R18 to R34, R16 to R35, R20 to R38, R11 to R39, R21 to R40, R22 to R41, R23 to R42, R24 to R43, R88 to R44, R25 to R45, R28 to R47, R29 to R48, R32 to R51, R101 to R52, R33 to R53, R37 to R56, R35 to R57, R38 to R58, R39 to R59, TP1 to TP12, TP2 to TP13, TP6 to TP14, TP3 to TP15, TP4 to TP16, TP5 to TP17, U11 to U14, U10 to U15, U12 to U16, U15 to U18, U14 to U19, U16 to U20
Connections:
- net BUS_3V3: now also R3.2
- net BUS_5V: now also R3.1
- net BUS_UNREG: now also R46.1
- net EN_3V3_EF: now also R36.1, R32.1; no longer R28.2, U15.1 (EN/UVLO), U15.4 (PGTH)
- net EN_5V_EF: now also R50.1, R54.1; no longer U19.1 (EN/UVLO), U19.4 (PGTH)
- net GNDA: now also R55.2; no longer R36.2
- net at U19.2 (OVLO): now also R54.2, R55.1; no longer R36.1
- net at U14.6 (OUT), U5.1 (IN+): now also R3.1
- net at U18.6 (OUT), U5.1 (IN+): now also R3.2
- net at R37.1, U15.2 (OVLO): now also R36.2
- new net: R28.2, R32.2, U15.1 (EN/UVLO), U15.4 (PGTH)
- new net: R46.2, R50.2
- new net: U19.1 (EN/UVLO), U19.4 (PGTH)
Other:
- note added: "gets pulled up to max 3.3V"
- note removed: "gets pulled up to max 4V"

Commit message: Finished initial revision of PCB
Parts:
- Q3, Q4: footprint Package_TO_SOT_SMD:SOT-23 -> Package_TO_SOT_SMD:SOT-416
Connections:
- net at R46.2, R50.2: now also U19.1 (EN/UVLO), U19.4 (PGTH)
Changed lines of the file:
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@@
   (junction (at 189.23 111.76) (diameter 0) (color 0 0 0 0)
   )
+  (junction (at 49.53 116.84) (diameter 0) (color 0 0 0 0)
+  )
   (junction (at 191.77 111.76) (diameter 0) (color 0 0 0 0)
   )
@@
   (junction (at 171.45 58.42) (diameter 0) (color 0 0 0 0)
   )
-  (junction (at 218.44 119.38) (diameter 0) (color 0 0 0 0)
-  )
   (junction (at 36.83 116.84) (diameter 0) (color 0 0 0 0)
   )
@@
   (junction (at 161.29 124.46) (diameter 0) (color 0 0 0 0)
   )
+  (junction (at 44.45 116.84) (diameter 0) (color 0 0 0 0)
+  )
   (junction (at 156.21 124.46) (diameter 0) (color 0 0 0 0)
   )
@@
   (junction (at 132.08 67.31) (diameter 0) (color 0 0 0 0)
   )
+  (junction (at 218.44 119.38) (diameter 0) (color 0 0 0 0)
+  )
   (junction (at 231.14 116.84) (diameter 0) (color 0 0 0 0)
   )
@@
     (stroke (width 0) (type default))
   )
+  (wire (pts (xy 44.45 116.84) (xy 49.53 116.84))
+    (stroke (width 0) (type default))
+  )
   (wire (pts (xy 151.13 124.46) (xy 151.13 111.76))
     (stroke (width 0) (type default))
@@
       (effects (font (size 1.27 1.27)) (justify left))
     )
-    (property "Footprint" "Package_TO_SOT_SMD:SOT-23" (at 228.6 55.245 0)
+    (property "Footprint" "Package_TO_SOT_SMD:SOT-416" (at 228.6 55.245 0)
       (effects (font (size 1.27 1.27) italic) (justify left) hide)
     )
@@
       (effects (font (size 1.27 1.27)) (justify left))
     )
-    (property "Footprint" "Package_TO_SOT_SMD:SOT-23" (at 228.6 121.285 0)
+    (property "Footprint" "Package_TO_SOT_SMD:SOT-416" (at 228.6 121.285 0)
       (effects (font (size 1.27 1.27) italic) (justify left) hide)
     )

Commit message: Fixed MP28167, debug headers
Parts:
- U16, U20: value MP28167-A -> MP28167GQ-A; LCSC Part (none) -> C3188179
Changed lines of the file:
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@@
       (effects (font (size 1.27 1.27)))
     )
-    (property "Value" "MP28167-A" (at 132.08 102.87 0)
+    (property "Value" "MP28167GQ-A" (at 132.08 102.87 0)
       (effects (font (size 1.27 1.27)))
     )
@@
     )
     (property "Datasheet" "" (at 118.11 119.38 0)
+      (effects (font (size 1.27 1.27)) hide)
+    )
+    (property "LCSC Part" "C3188179" (at 118.11 119.38 0)
       (effects (font (size 1.27 1.27)) hide)
     )
@@
       (effects (font (size 1.27 1.27)))
     )
-    (property "Value" "MP28167-A" (at 132.08 36.83 0)
+    (property "Value" "MP28167GQ-A" (at 132.08 36.83 0)
       (effects (font (size 1.27 1.27)))
     )
@@
       (effects (font (size 1.27 1.27)) hide)
     )
+    (property "LCSC Part" "C3188179" (at 118.11 53.34 0)
+      (effects (font (size 1.27 1.27)) hide)
+    )

Commit message: Fixes for next version
Parts:
- added R289, R290: 47K, Resistor_SMD:R_0402_1005Metric, symbol Device:R_Small_US
- added R293, R294: 200K, Resistor_SMD:R_0402_1005Metric, symbol Device:R_Small_US
- R27, R45: value 33R -> 150R; LCSC Part C25105 -> C25082
Connections:
- net BUS_3V3: now also R293.1
- net BUS_5V: now also R294.1
- net GND: now also R289.2, R290.2, R293.2, R294.2
- net SYS_3V3: no longer R26.1, R44.1
- net at Q3.1 (G), R26.2, U14.3 (PG): now also R289.1
- net at C61.1, C62.1, C63.1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: now also R44.1
- net at C43.1, C44.1, C45.1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: now also R26.1
- net at Q4.1 (G), R44.2, U18.3 (PG): now also R290.1
Other:
- moved on the sheet: R26, R44
