File: ESLGSU_Programmable_Regulators.kicad_sch (KiCad schematic)
At the start: 94 parts, among them Q1 DMN67D7L-7, Q2 DMN67D7L-7, U10 MP28167-A, U11 TPS259474LRPWR, U13 TPS259474LRPWR, U14 MP28167-A, U15 LM73100RPWR, U5 INA219AIDCNR, U9 LM73100RPWR

Commit message: Schematic work
Parts:
- removed C16, C31: 330p, Capacitor_SMD:C_0402_1005Metric, symbol Device:C_Small
- removed L1, L2: IHLP4040DZER4R7M01, Inductor_SMD:L_Vishay_IHLP-4040, symbol Device:L
- removed Q1, Q2: DMN67D7L-7, Package_TO_SOT_SMD:SOT-23, symbol Transistor_FET:DMN67D7L
- removed R10, R27: 47K, Resistor_SMD:R_0402_1005Metric, symbol Device:R_Small_US
- removed R14: 549R, Resistor_SMD:R_0402_1005Metric, symbol Device:R_Small_US
- removed R15, R28: 14.7K, Resistor_SMD:R_0402_1005Metric, symbol Device:R_Small_US
- removed R16, R35: 350K, Resistor_SMD:R_0402_1005Metric, symbol Device:R_Small_US
- removed R20, R38: 100R, Resistor_SMD:R_0402_1005Metric, symbol Device:R_Small_US
- removed R23: 100K, Resistor_SMD:R_0402_1005Metric, symbol Device:R_Small_US
- removed R24: 17.4K, Resistor_SMD:R_0402_1005Metric, symbol Device:R_Small_US
- removed R25: 7.5K, Resistor_SMD:R_0402_1005Metric, symbol Device:R_Small_US
- removed R31, R6: 21.5K, Resistor_SMD:R_0402_1005Metric, symbol Device:R_Small_US
- removed R32, R9: 806K, Resistor_SMD:R_0402_1005Metric, symbol Device:R_Small_US
- removed R33, R7: 430K, Resistor_SMD:R_0402_1005Metric, symbol Device:R_Small_US
- removed R34: 107K, Resistor_SMD:R_0402_1005Metric, symbol Device:R_Small_US
- removed R8: 187K, Resistor_SMD:R_0402_1005Metric, symbol Device:R_Small_US
- added C45 (x2): 220p, Capacitor_SMD:C_0402_1005Metric, symbol Device:C_Small
- added L1 (x2): SRP1038A-4R7M, Inductor_SMD:L_Vishay_IHLP-4040, symbol Device:L
- added Q1 (x2): RE1C002UNTCL, Package_TO_SOT_SMD:SOT-416, symbol Transistor_FET:DMN67D7L
- added R10 (x2): 33K, Resistor_SMD:R_0402_1005Metric, symbol Device:R_Small_US
- added R11 (x2): 150K, Resistor_SMD:R_0402_1005Metric, symbol Device:R_Small_US
- added R11 (x2): 51K, Resistor_SMD:R_0402_1005Metric, symbol Device:R_Small_US
- added R11 (x2): 220K, Resistor_SMD:R_0402_1005Metric, symbol Device:R_Small_US
- added R11: 68K, Resistor_SMD:R_0402_1005Metric, symbol Device:R_Small_US
- added R12: 12K, Resistor_SMD:R_0402_1005Metric, symbol Device:R_Small_US
- added R13: 5.1K, Resistor_SMD:R_0402_1005Metric, symbol Device:R_Small_US
- added R15 (x2): 200K, Resistor_SMD:R_0402_1005Metric, symbol Device:R_Small_US
- added R17 (x2): 10K, Resistor_SMD:R_0402_1005Metric, symbol Device:R_Small_US
- added R21 (x2): 22K, Resistor_SMD:R_0402_1005Metric, symbol Device:R_Small_US
- added R26: 1K, Resistor_SMD:R_0402_1005Metric, symbol Device:R_Small_US
- added R8 (x2): 33R, Resistor_SMD:R_0402_1005Metric, symbol Device:R_Small_US
- C12, C13, C18, C21, C35, C37, C38, C40, C6: LCSC Part (none) -> C307331
- C14, C27, C28, C30, C36, C46: LCSC Part (none) -> C52923
- C15, C39: LCSC Part (none) -> C1532
- C17, C32: LCSC Part (none) -> C1531
- C19, C22, C23, C24, C25, C26, C34, C41, C42, C43, C44, C45: LCSC Part (none) -> C45783
- C20, C33: LCSC Part (none) -> C134220
- D1, D2: LCSC Part (none) -> C2286
- R11: value 100K -> 68K; LCSC Part (none) -> C36871
- R12: value 17.4K -> 12K; LCSC Part (none) -> C25752
- R13: value 7.5K -> 5.1K; LCSC Part (none) -> C25905
- R2: LCSC Part (none) -> C346483
- R2: LCSC Part (none) -> C25900
- R26: value 549R -> 1K; LCSC Part (none) -> C11702
- R29, R30, R4, R5: LCSC Part (none) -> C17168
- R87: LCSC Part (none) -> C25792
- TP1: JLCPCB BOM (none) -> 0; now left out of the parts list
- TP1: JLCPCB BOM (none) -> 0
- U11, U13: LCSC Part (none) -> C3662807
- U15, U9: LCSC Part (none) -> C3210761
- U5: LCSC Part (none) -> C87469
Connections:
- net BUS_UNREG: now also R11.1
- net EN_CH1: now also U15.1 (EN/UVLO), U15.4 (PGTH), U9.1 (EN/UVLO), U9.4 (PGTH)
- net EN_CH2: now also R11.2, R12.1
- net GND: now also Q1.2 (S), Q1.2 (S)
- net GNDA: now also C45.2, C45.2, R11.2, R11.2, R13.2, R17.2, R17.2, R21.2, R21.2, R26.2
- net SYS_3V3: now also R87.1, R87.1, R8.1, R8.1
- net at D1.1 (K): now also Q1.3 (D)
- net at D1.2 (A): now also R8.2; no longer R87.1
- net at C21.1, C22.1, C23.1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: now also R11.1
- net at U10.3 (EN), U11.3 (PG): now also R10.2, R17.1
- net at C18.1, C19.1, C20.1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: now also R10.1
- net at U11.7 (dVdt): now also C45.1
- net at U11.9 (ILM): now also R26.1
- net at C40.1, C41.1, C42.1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: now also R11.1
- net at R87.2, U15.3 (PG): now also Q1.1 (G)
- net at C33.1, C34.1, C35.1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: now also R10.1
- net at C38.1, U14.14 (SW2): now also L1.2
- net at R87.2, U9.3 (PG): now also Q1.1 (G)
- net at U13.2 (OVLO): now also R12.2, R13.1
- net at U13.3 (PG), U14.3 (EN): now also R10.2, R17.1
- net at C13.1, U10.14 (SW2): now also L1.2
- net at C12.1, U10.15 (SW1): now also L1.1
- net at C15.1, U10.7 (OC): now also R21.1
- net at U10.8 (FB): now also R15.1
- net at C37.1, U14.15 (SW1): now also L1.1
- net at D2.1 (K): now also Q1.3 (D)
- net at D2.2 (A): now also R8.2; no longer R87.1
- net at U14.8 (FB): now also R15.1
- net at C39.1, U14.7 (OC): now also R21.1
- net at U13.7 (dVdt): now also C45.1
- new net: R11.1, R11.2 (x2)
- new net: R11.1, R11.2, R15.2 (x2)
Other:
- note added: "1.39-4.65V"
- note added: "6A limit 7.5V/ms"
- note added: "gets pulled up to max 4V"
- note removed: "1.28-4.76V"
- note removed: "6A limit 5V/ms"
- moved on the sheet: R87
