File: ESLGSU_Programmable_Regulators.kicad_sch (KiCad schematic)
At the start: 92 parts, among them Q3 RE1C002UNTCL, U10 MP28167-A, U11 TPS259474LRPWR, U13 TPS259474LRPWR, U14 MP28167-A, U15 LM73100RPWR, U5 INA219AIDCNR, U9 LM73100RPWR

Commit message: Last save
Parts:
- TP1: now left out of the parts list
Changed lines of the file:
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@@
   )
   (symbol (lib_id "Connector:TestPoint") (at 149.86 116.84 0) (unit 1)
-    (in_bom yes) (on_board yes) (dnp no) (fields_autoplaced)
+    (in_bom no) (on_board yes) (dnp no) (fields_autoplaced)
     (property "Reference" "TP1" (at 152.4 112.268 0)
       (effects (font (size 1.27 1.27)) (justify left))
@@
   )
   (symbol (lib_id "Connector:TestPoint") (at 149.86 50.8 0) (unit 1)
-    (in_bom yes) (on_board yes) (dnp no) (fields_autoplaced)
+    (in_bom no) (on_board yes) (dnp no) (fields_autoplaced)
     (property "Reference" "TP1" (at 152.4 46.228 0)
       (effects (font (size 1.27 1.27)) (justify left))

Commit message: Fixed MP28167, debug headers
Parts:
- U10, U14: value MP28167-A -> MP28167GQ-A; LCSC Part (none) -> C3188179
Changed lines of the file:
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@@
       (effects (font (size 1.27 1.27)))
     )
-    (property "Value" "MP28167-A" (at 130.81 41.91 0)
+    (property "Value" "MP28167GQ-A" (at 130.81 41.91 0)
       (effects (font (size 1.27 1.27)))
     )
@@
     )
     (property "Datasheet" "" (at 116.84 58.42 0)
+      (effects (font (size 1.27 1.27)) hide)
+    )
+    (property "LCSC Part" "C3188179" (at 116.84 58.42 0)
       (effects (font (size 1.27 1.27)) hide)
     )
@@
       (effects (font (size 1.27 1.27)))
     )
-    (property "Value" "MP28167-A" (at 130.81 107.95 0)
+    (property "Value" "MP28167GQ-A" (at 130.81 107.95 0)
       (effects (font (size 1.27 1.27)))
     )
@@
       (effects (font (size 1.27 1.27)) hide)
     )
+    (property "LCSC Part" "C3188179" (at 116.84 124.46 0)
+      (effects (font (size 1.27 1.27)) hide)
+    )
