File: ESLGSU_Main_uC.kicad_sch (KiCad schematic)
At the start: 0 parts

Commit message: uC Interface work
Parts:
- added C6 (x9): 100n, Capacitor_SMD:C_0603_1608Metric, symbol Device:C_Small
- added R10: 200K, Resistor_SMD:R_0603_1608Metric, symbol Device:R_Small_US
- added R10 (x8): 0R, Resistor_SMD:R_0603_1608Metric, symbol Device:R_Small_US
- added R10: 120R, Resistor_SMD:R_0603_1608Metric, symbol Device:R_Small_US
- added R10: 50R, Resistor_SMD:R_0603_1608Metric, symbol Device:R_Small_US
- added R10 (x2): 10K, Resistor_SMD:R_0603_1608Metric, symbol Device:R_Small_US
- added U29: TCAN1051GVDRBRQ, Package_DFN_QFN:DFN-8-1EP_3x3mm_P0.65mm_EP1.55x2.4mm, symbol ESLGSU_Parts_Lib:TCAN1051GVDRBRQ1
- added U30: THVD1450DRBR, Package_DFN_QFN:DFN-8-1EP_3x3mm_P0.65mm_EP1.55x2.4mm, symbol ESLGSU_Parts_Lib:THVD1450
- added U31, U38: TXU0304RUTR, ESLGSU_Parts_Lib:T-UQFN-12, symbol ESLGSU_Parts_Lib:TXU0304-Q1
- added U32: TS5A23159RSER, Package_DFN_QFN:Texas_UQFN-10_1.5x2mm_P0.5mm, symbol ESLGSU_Parts_Lib:TS5A23159RSER
- added U33, U35: TXU0202DTTR, ESLGSU_Parts_Lib:SOT833-1-XSON8, symbol ESLGSU_Parts_Lib:TXU0202-Q1
- added U34, U36, U37, U40: 74LVC2G53GT, ESLGSU_Parts_Lib:SOT833-1-XSON8, symbol ESLGSU_Parts_Lib:74LVC2G53GT
- added U39: PCA9306, symbol Interface:PCA9306
- added U41: 74LVC2G66GT, ESLGSU_Parts_Lib:SOT833-1-XSON8, symbol ESLGSU_Parts_Lib:74LVC2G66GT
Connections:
- new net: R10.1, U40.1 (Z), U41.1 (1Y), U41.5 (2Y), U41.8 (VCC)
- new net: R10.2, U39.7 (VREF2), U39.8 (EN)
- new net: R10.2, U39.2 (VREF1), U40.7 (Y0)
- new net: R10.2, U34.6 (Y1)
- new net: C6.2, U37.6 (Y1), U38.1 (VCCA), U38.12 (OE)
- new net: C6.2, R10.2, R10.2, U30.8 (VCC), U33.7 (VCCB)
- new net: R10.2, U36.6 (Y1)
- new net: C6.2, U31.11 (VCCB), U31.12 (OE), U37.7 (Y0)
- new net: R10.2, U40.6 (Y1)
- new net: U30.1 (R), U33.1 (B2)
- new net: U30.4 (D), U33.8 (B1Y)
- new net: R10.1, U41.2 (1Z)
- new net: R10.1, U41.6 (2Z)
- new net: U32.6 (COM2), U35.1 (B2)
- new net: C6.2, U32.8 (VCC), U34.1 (Z), U35.7 (VCCB)
- new net: U32.10 (COM1), U35.8 (B1Y)
- new net: U36.1 (Z), U37.1 (Z)
- new net: R10.2, U34.7 (Y0)
- new net: R10.2, U36.7 (Y0)
- new net CAN1_H: R10.1, U29.7 (CANH)
- new net CAN1_L: R10.2, U29.6 (CANL)
- new net CAN1_RX: U29.4 (RXD)
- new net CAN1_SE: U29.8 (S)
- new net CAN1_TX: U29.1 (TXD)
- new net GND: C6.1, C6.1, C6.1, C6.1, C6.1, C6.1, C6.1, C6.1, C6.1, U29.2 (GND), U29.9 (GND), U30.2 (nRE), U30.5 (GND), U30.9 (GND), U31.6 (GND), U32.3 (GND), U33.2 (GND), U34.3 (GND), U34.4 (GND), U35.2 (GND), U36.3 (GND), U36.4 (GND), U37.2 (nE), U37.3 (GND), U37.4 (GND), U38.6 (GND), U39.1 (GND), U40.3 (GND), U40.4 (GND), U41.4 (GND)
- new net I2C1_5V: U40.5 (S)
- new net I2C1_PEN: U41.3 (2E), U41.7 (1E)
- new net I2C1_SCL: R10.2, U39.3 (SCL1), U39.6 (SCL2)
- new net I2C1_SDA: R10.2, U39.4 (SDA1), U39.5 (SDA2)
- new net I2C1_nEN: U40.2 (nE)
- new net RS4851_A: R10.2, U30.6 (A)
- new net RS4851_B: R10.1, U30.7 (B)
- new net RS4851_RX: U33.4 (A2Y)
- new net RS4851_TX: U33.5 (A1)
- new net RS4851_TXE: U30.3 (DE)
- new net SPI1_5V: U36.5 (S)
- new net SPI1_MISO: U31.5 (A4Y), U31.7 (B4), U38.5 (A4Y), U38.7 (B4)
- new net SPI1_MM: U37.5 (S)
- new net SPI1_MOSI: U31.10 (B1Y), U31.2 (A1), U38.10 (B1Y), U38.2 (A1)
- new net SPI1_NSS: U31.4 (A3), U31.8 (B3Y), U38.4 (A3), U38.8 (B3Y)
- new net SPI1_SCK: U31.3 (A2), U31.9 (B2Y), U38.3 (A2), U38.9 (B2Y)
- new net SPI1_nEN: U36.2 (nE)
- new net SYS_3V3: C6.2, C6.2, C6.2, C6.2, R10.1, R10.1, R10.1, R10.1, U29.5 (VIO), U31.1 (VCCA), U33.3 (VCCA), U33.6 (OE), U35.3 (VCCA), U35.6 (OE), U38.11 (VCCB)
- new net SYS_5V: C6.2, R10.1, R10.1, R10.1, R10.1, U29.3 (VCC), U34.8 (VCC), U36.8 (VCC), U37.8 (VCC), U40.8 (VCC)
- new net UART1_5V: U34.5 (S)
- new net UART1_REV: U32.1 (IN1), U32.5 (IN2)
- new net UART1_RX: U32.2 (NO1), U32.7 (NC2), U35.4 (A2Y)
- new net UART1_TX: U32.4 (NO2), U32.9 (NC1), U35.5 (A1)
- new net UART1_nEN: U34.2 (nE)
Other:
- note added: "CAN Transceiver"
- note added: "DO NOT SOLDER BOTH"
- note added: "I2C Transceiver"
- note added: "RS485 Transceiver"
- note added: "SPI Transceiver"
- note added: "UART Transceiver"

Commit message: Finished interfaces work
Parts:
- removed C6 (x3): 100n, Capacitor_SMD:C_0603_1608Metric, symbol Device:C_Small
- removed R10 (x8): 0R, Resistor_SMD:R_0603_1608Metric, symbol Device:R_Small_US
- removed U31, U38: TXU0304RUTR, ESLGSU_Parts_Lib:T-UQFN-12, symbol ESLGSU_Parts_Lib:TXU0304-Q1
- removed U32: TS5A23159RSER, Package_DFN_QFN:Texas_UQFN-10_1.5x2mm_P0.5mm, symbol ESLGSU_Parts_Lib:TS5A23159RSER
- removed U34, U36, U37, U40: 74LVC2G53GT, ESLGSU_Parts_Lib:SOT833-1-XSON8, symbol ESLGSU_Parts_Lib:74LVC2G53GT
- removed U41: 74LVC2G66GT, ESLGSU_Parts_Lib:SOT833-1-XSON8, symbol ESLGSU_Parts_Lib:74LVC2G66GT
- added C6: 100p, Capacitor_SMD:C_0402_1005Metric, symbol Device:C_Small
- added C6 (x7): 100n, Capacitor_SMD:C_0402_1005Metric, symbol Device:C_Small
- added R10 (x7): 200K, Resistor_SMD:R_0402_1005Metric, symbol Device:R_Small_US
- added RN1, RN3, RN4: 0R, Resistor_SMD:R_Array_Concave_4x0402, symbol Device:R_Pack04
- added RN2, RN5, RN6, RN7: 0R, Resistor_SMD:R_Array_Convex_2x0402, symbol Device:R_Pack02
- added U31, U32, U34, U44, U47: TMUX1574RSVR, ESLGSU_Parts_Lib:T-UQFN-16, symbol ESLGSU_Parts_Lib:TMUX1574RSVR
- added U36, U40, U46: TXB0104RUT, ESLGSU_Parts_Lib:T-UQFN-12, symbol ESLGSU_Parts_Lib:TXB0104RUTR
- added U37: STM32H753ZITx, Package_QFP:LQFP-144_20x20mm_P0.5mm, symbol MCU_ST_STM32H7:STM32H753ZITx
- C6: footprint Capacitor_SMD:C_0603_1608Metric -> Capacitor_SMD:C_0402_1005Metric
- R10: footprint Resistor_SMD:R_0603_1608Metric -> Resistor_SMD:R_0402_1005Metric
- U39: footprint (none) -> ESLGSU_Parts_Lib:SOT833-1-XSON8
Connections:
- net CAN1_SE: now also R10.1
- net GND: now also C6.1, C6.1, C6.1, C6.1, C6.1, C6.1, C6.1, C6.2, R10.2, U31.15 (SEL), U31.6 (GND), U32.6 (GND), U34.6 (GND), U36.6 (GND), U40.6 (GND), U44.6 (GND), U46.6 (GND), U47.6 (GND); no longer U30.2 (nRE)
- net I2C1_SCL: now also RN6.2 (R2.1), RN6.3 (R2.2), RN7.3 (R2.2)
- net I2C1_SDA: now also RN6.1 (R1.1), RN6.4 (R1.2), RN7.4 (R1.2)
- net RS4851_RX: now also RN5.4 (R1.2)
- net RS4851_TX: now also RN5.3 (R2.2)
- net RS4851_TXE: now also U30.2 (nRE), R10.1
- net SPI1_MISO: now also RN1.1 (R1.1), RN1.8 (R1.2), U46.5 (A4), U47.10 (D4), U47.12 (S4A)
- net SPI1_MOSI: now also RN1.4 (R4.1), RN1.5 (R4.2), U46.2 (A1), U47.16 (S1A), U47.2 (D1)
- net SPI1_NSS: now also RN1.2 (R2.1), RN1.7 (R2.2), U46.4 (A3), U47.7 (D3), U47.9 (S3A)
- net SPI1_SCK: now also RN1.3 (R3.1), RN1.6 (R3.2), U46.3 (A2), U47.3 (S2A), U47.5 (D2)
- net SPI1_nEN: now also R10.1, U47.13 (nEN)
- net SYS_3V3: now also U39.2 (VREF1), C6.2, C6.2, C6.2, R10.1, R10.2, R10.2, R10.2, R10.2, R10.2, RN7.1 (R1.1), RN7.2 (R2.1), U36.1 (VCCA), U40.1 (VCCA), U46.1 (VCCA)
- net UART1_REV: now also U32.15 (SEL)
- net UART1_RX: now also RN2.1 (R1.1), RN2.4 (R1.2), U32.5 (D2)
- net UART1_TX: now also RN2.2 (R2.1), RN2.3 (R2.2), U32.2 (D1)
- net UART1_nEN: now also R10.1, U32.13 (nEN)
- net VBUS: now reaches R10.1
- net VBUS: now also C6.2, C6.2, U30.8 (VCC), U33.7 (VCCB), U35.7 (VCCB), C6.1, C6.2, C6.2, C6.2, U31.14 (VDD), U31.2 (D1), U31.5 (D2), U32.14 (VDD), U34.14 (VDD), U36.11 (VCCB), U40.11 (VCCB), U44.14 (VDD), U46.11 (VCCB), U47.14 (VDD)
- net at R10.2, U39.7 (VREF2): now also C6.2; no longer U39.8 (EN)
- net at U30.1 (R), U33.1 (B2): now also RN5.1 (R1.1)
- net at U30.4 (D), U33.8 (B1Y): now also RN5.2 (R2.1)
- net at R10.1: now also U31.3 (S2A)
- net at R10.1: now also U31.16 (S1A)
- net at U35.1 (B2): now also U32.1 (S1B), U32.3 (S2A)
- net at U35.8 (B1Y): now also U32.16 (S1A), U32.4 (S2B)
- new net: U46.10 (B1), U47.1 (S1B)
- new net: U46.7 (B4), U47.11 (S4B)
- new net: U46.9 (B2), U47.4 (S2B)
- new net: U46.8 (B3), U47.8 (S3B)
- new net: U36.10 (B1), U44.1 (S1B)
- new net: U36.7 (B4), U44.11 (S4B)
- new net: U36.9 (B2), U44.4 (S2B)
- new net: U36.8 (B3), U44.8 (S3B)
- new net: U34.1 (S1B), U40.10 (B1)
- new net: U34.11 (S4B), U40.7 (B4)
- new net: U34.8 (S3B), U40.8 (B3)
- new net: U34.4 (S2B), U40.9 (B2)
- new net: U37.107 (VSS), U37.120 (VSS), U37.130 (VSS), U37.16 (VSS), U37.38 (VSS), U37.51 (VSS), U37.61 (VSS), U37.83 (VSS), U37.94 (VSS)
- new net GPIO_1: RN3.4 (R4.1), RN3.5 (R4.2), U36.2 (A1), U44.16 (S1A), U44.2 (D1)
- new net GPIO_2: RN3.3 (R3.1), RN3.6 (R3.2), U36.3 (A2), U44.3 (S2A), U44.5 (D2)
- new net GPIO_3: RN3.2 (R2.1), RN3.7 (R2.2), U36.4 (A3), U44.7 (D3), U44.9 (S3A)
- new net GPIO_4: RN3.1 (R1.1), RN3.8 (R1.2), U36.5 (A4), U44.10 (D4), U44.12 (S4A)
- new net GPIO_5: RN4.4 (R4.1), RN4.5 (R4.2), U34.16 (S1A), U34.2 (D1), U40.2 (A1)
- new net GPIO_6: RN4.3 (R3.1), RN4.6 (R3.2), U34.3 (S2A), U34.5 (D2), U40.3 (A2)
- new net GPIO_7: RN4.2 (R2.1), RN4.7 (R2.2), U34.7 (D3), U34.9 (S3A), U40.4 (A3)
- new net GPIO_8: RN4.1 (R1.1), RN4.8 (R1.2), U34.10 (D4), U34.12 (S4A), U40.5 (A4)
- new net GPIO_A_SHIFT: U36.12 (OE), U44.15 (SEL)
- new net GPIO_A_nEN: R10.1, U44.13 (nEN)
- new net GPIO_B_SHIFT: U34.15 (SEL), U40.12 (OE)
- new net GPIO_B_nEN: R10.1, U34.13 (nEN)
- new net I2C1_EN: U39.8 (EN)
- new net I2C1_nPEN: R10.2, U31.13 (nEN)
- new net SPI1_SHIFT: U46.12 (OE), U47.15 (SEL)
- no-connect marks 0 -> 14
Other:
- note added: "GPIO Transceiver"
- note removed: "DO NOT SOLDER BOTH"
- moved on the sheet: C6, R10, U30, U33, U35, U39

Commit message: Started some PCB layout work
Connections:
- net GPIO_1: no longer RN3.5 (R4.2), U36.2 (A1), U44.16 (S1A)
- net GPIO_2: no longer RN3.6 (R3.2), U36.3 (A2), U44.3 (S2A)
- net GPIO_3: no longer RN3.7 (R2.2), U36.4 (A3), U44.9 (S3A)
- net GPIO_4: no longer RN3.8 (R1.2), U36.5 (A4), U44.12 (S4A)
- net GPIO_5: no longer RN4.5 (R4.2), U34.16 (S1A), U40.2 (A1)
- net GPIO_6: no longer RN4.6 (R3.2), U34.3 (S2A), U40.3 (A2)
- net GPIO_7: no longer RN4.7 (R2.2), U34.9 (S3A), U40.4 (A3)
- net GPIO_8: no longer RN4.8 (R1.2), U34.12 (S4A), U40.5 (A4)
- net I2C1_SCL: no longer RN6.3 (R2.2), U39.3 (SCL1)
- net I2C1_SDA: no longer RN6.4 (R1.2), U39.4 (SDA1)
- net SPI1_MISO: no longer RN1.8 (R1.2), U46.5 (A4), U47.12 (S4A)
- net SPI1_MOSI: no longer RN1.5 (R4.2), U46.2 (A1), U47.16 (S1A)
- net SPI1_NSS: no longer RN1.7 (R2.2), U46.4 (A3), U47.9 (S3A)
- net SPI1_SCK: no longer RN1.6 (R3.2), U46.3 (A2), U47.3 (S2A)
- net UART1_RX: no longer RN2.4 (R1.2), U35.4 (A2Y)
- net UART1_TX: no longer RN2.3 (R2.2), U35.5 (A1)
- new net _GPIO_1: RN3.5 (R4.2), U36.2 (A1), U44.16 (S1A)
- new net _GPIO_2: RN3.6 (R3.2), U36.3 (A2), U44.3 (S2A)
- new net _GPIO_3: RN3.7 (R2.2), U36.4 (A3), U44.9 (S3A)
- new net _GPIO_4: RN3.8 (R1.2), U36.5 (A4), U44.12 (S4A)
- new net _GPIO_5: RN4.5 (R4.2), U34.16 (S1A), U40.2 (A1)
- new net _GPIO_6: RN4.6 (R3.2), U34.3 (S2A), U40.3 (A2)
- new net _GPIO_7: RN4.7 (R2.2), U34.9 (S3A), U40.4 (A3)
- new net _GPIO_8: RN4.8 (R1.2), U34.12 (S4A), U40.5 (A4)
- new net _I2C1_SCL: RN6.3 (R2.2), U39.3 (SCL1)
- new net _I2C1_SDA: RN6.4 (R1.2), U39.4 (SDA1)
- new net _SPI1_MISO: RN1.8 (R1.2), U46.5 (A4), U47.12 (S4A)
- new net _SPI1_MOSI: RN1.5 (R4.2), U46.2 (A1), U47.16 (S1A)
- new net _SPI1_NSS: RN1.7 (R2.2), U46.4 (A3), U47.9 (S3A)
- new net _SPI1_SCK: RN1.6 (R3.2), U46.3 (A2), U47.3 (S2A)
- new net _UART1_RX: RN2.4 (R1.2), U35.4 (A2Y)
- new net _UART1_TX: RN2.3 (R2.2), U35.5 (A1)

Commit message: More PCB work
Parts:
- removed R10 (x2): 10K, Resistor_SMD:R_0402_1005Metric, symbol Device:R_Small_US
- added RN8: 10K, Resistor_SMD:R_Array_Convex_2x0402, symbol Device:R_Pack02
- RN7: value 0R -> 10K
Connections:
- net I2C1_SCL: now also RN8.3 (R2.2)
- net I2C1_SDA: now also RN8.4 (R1.2)
- net at U31.3 (S2A): now also RN8.1 (R1.1)
- net at U31.16 (S1A): now also RN8.2 (R2.1)
Other:
- moved on the sheet: R10, U31

Commit message: Tried to prepare for order
Parts:
- U37: value STM32H753ZITx -> STM32H753ZIT6
Changed lines of the file:
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@@
       (effects (font (size 1.27 1.27)) (justify left))
     )
-    (property "Value" "STM32H753ZITx" (at 106.3341 238.76 0)
+    (property "Value" "STM32H753ZIT6" (at 106.3341 238.76 0)
       (effects (font (size 1.27 1.27)) (justify left))
     )

Commit message: Schematic work
Parts:
- removed R10: 50R, Resistor_SMD:R_0402_1005Metric, symbol Device:R_Small_US
- removed RN8: 10K, Resistor_SMD:R_Array_Convex_2x0402, symbol Device:R_Pack02
- removed U39: PCA9306, ESLGSU_Parts_Lib:SOT833-1-XSON8, symbol Interface:PCA9306
- added C6 (x2): 100n, Capacitor_SMD:C_0402_1005Metric, symbol Device:C_Small
- added R10 (x4): 10K, Resistor_SMD:R_0402_1005Metric, symbol Device:R_Small_US
- added R10: 200K, Resistor_SMD:R_0402_1005Metric, symbol Device:R_Small_US
- added R10: 120R, Resistor_SMD:R_0805_2012Metric, symbol Device:R_Small_US
- added RN8: 0R, Resistor_SMD:R_Array_Concave_4x0402, symbol Device:R_Pack04
- added U39: FXMA2102L8X, symbol ESLGSU_Parts_Lib:FXMA2102L8X
- added U43: TXB0104RUT, ESLGSU_Parts_Lib:T-UQFN-12, symbol ESLGSU_Parts_Lib:TXB0104RUTR
- added U45: TMUX1574RSVR, ESLGSU_Parts_Lib:T-UQFN-16, symbol ESLGSU_Parts_Lib:TMUX1574RSVR
- C6: LCSC Part (none) -> C1546
- C6: LCSC Part (none) -> C307331
- R10: LCSC Part (none) -> C25764
- R10: footprint Resistor_SMD:R_0402_1005Metric -> Resistor_SMD:R_0805_2012Metric; JLCPCB BOM (none) -> 0; LCSC Part (none) -> C17437; now left out of the parts list
- RN1, RN3, RN4: JLCPCB BOM (none) -> 0; LCSC Part (none) -> C2001; now left out of the parts list
- RN2, RN5, RN6: JLCPCB BOM (none) -> 0; LCSC Part (none) -> C75375; now left out of the parts list
- RN7: JLCPCB BOM (none) -> 0; LCSC Part (none) -> C695179; now left out of the parts list
- U29: LCSC Part (none) -> C1848110
- U30: LCSC Part (none) -> C1850226
- U31, U32, U34, U44, U47: LCSC Part (none) -> C2673120
- U33, U35: LCSC Part (none) -> C18197534
- U36, U40, U46: LCSC Part (none) -> C105266
- U37: LCSC Part (none) -> C114408
Connections:
- net GND: now also C6.1, C6.1, U39.4 (GND), U43.6 (GND), U45.6 (GND)
- net I2C1_EN: now also U39.5 (OE)
- net I2C1_SCL: now also R10.2, U39.7 (SCL2)
- net I2C1_SDA: now also R10.2, U39.6 (SDA2)
- net RS4851_A: now also R10.2
- net RS4851_B: now also R10.1
- net SYS_3V3: now also C6.2, R10.1, R10.1, R10.2, U39.1 (VREF1), U43.1 (VCCA)
- net VBUS: now also C6.2, U43.11 (VCCB), U45.14 (VDD)
- net _I2C1_SCL: now also R10.2, U39.2 (SCL1)
- net _I2C1_SDA: now also R10.2, U39.3 (SDA1)
- net at C6.2, R10.2: now also U39.8 (VREF2)
- net at U31.3 (S2A): now also R10.1
- net at U31.16 (S1A): now also R10.1
- new net: U43.10 (B1), U45.1 (S1B)
- new net: U43.7 (B4), U45.11 (S4B)
- new net: U43.8 (B3), U45.8 (S3B)
- new net: U43.9 (B2), U45.4 (S2B)
- new net SPI2_MISO: RN8.1 (R1.1), U45.10 (D4)
- new net SPI2_MOSI: RN8.4 (R4.1), U45.2 (D1)
- new net SPI2_NSS: RN8.2 (R2.1), U45.7 (D3)
- new net SPI2_SCK: RN8.3 (R3.1), U45.5 (D2)
- new net SPI2_SHIFT: U43.12 (OE), U45.15 (SEL)
- new net SPI2_nEN: R10.1, U45.13 (nEN)
- new net _SPI2_MISO: RN8.8 (R1.2), U43.5 (A4), U45.12 (S4A)
- new net _SPI2_MOSI: RN8.5 (R4.2), U43.2 (A1), U45.16 (S1A)
- new net _SPI2_NSS: RN8.7 (R2.2), U43.4 (A3), U45.9 (S3A)
- new net _SPI2_SCK: RN8.6 (R3.2), U43.3 (A2), U45.3 (S2A)
Other:
- moved on the sheet: C6, R10, RN1, RN2, RN3, RN4, RN5, RN6, RN7, U29, U30, U31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

Commit message: Second last bit of schematic work
Parts:
- removed C6 (x2): 100n, Capacitor_SMD:C_0402_1005Metric, symbol Device:C_Small
- removed R10 (x2): 200K, Resistor_SMD:R_0402_1005Metric, symbol Device:R_Small_US
- removed U36, U40: TXB0104RUT, ESLGSU_Parts_Lib:T-UQFN-12, symbol ESLGSU_Parts_Lib:TXB0104RUTR
- removed U37: STM32H753ZIT6, Package_QFP:LQFP-144_20x20mm_P0.5mm, symbol MCU_ST_STM32H7:STM32H753ZITx
- added C25 (x14), C6 (x11): 100n, Capacitor_SMD:C_0402_1005Metric, symbol Device:C_Small
- added C29 (x2): 1u, Capacitor_SMD:C_0402_1005Metric, symbol Device:C_Small
- added C29 (x2): 2.2u, Capacitor_SMD:C_0402_1005Metric, symbol Device:C_Small
- added C29: 4.7u, Capacitor_SMD:C_0402_1005Metric, symbol Device:C_Small
- added C6: 100p, Capacitor_SMD:C_0402_1005Metric, symbol Device:C_Small
- added D1: TZ-P2-0603GTCS1-0.6T, LED_SMD:LED_0603_1608Metric, symbol Device:LED
- added D10: 1N5819, Diode_SMD:D_SOD-323, symbol Diode:1N5819
- added J2: Conn_01x06_Pin, Connector_PinHeader_1.27mm:PinHeader_1x06_P1.27mm_Vertical_SMD_Pin1Right, symbol Connector:Conn_01x06_Pin
- added R10 (x2): 120R, Resistor_SMD:R_0805_2012Metric, symbol Device:R_Small_US
- added R10 (x4): 10K, Resistor_SMD:R_0402_1005Metric, symbol Device:R_Small_US
- added R10 (x3): 510R, Resistor_SMD:R_0402_1005Metric, symbol Device:R_Small_US
- added R10 (x15): 200K, Resistor_SMD:R_0402_1005Metric, symbol Device:R_Small_US
- added R10 (x2): 100K, Resistor_SMD:R_0402_1005Metric, symbol Device:R_Small_US
- added R6 (x8): 0R, Resistor_SMD:R_0402_1005Metric, symbol Device:R_Small_US
- added R8: 33R, Resistor_SMD:R_0402_1005Metric, symbol Device:R_Small_US
- added RN13, RN14, RN16: 0R, Resistor_SMD:R_Array_Convex_2x0402, symbol Device:R_Pack02
- added RN15: 10K, Resistor_SMD:R_Array_Convex_2x0402, symbol Device:R_Pack02
- added U37: STM32H743ZITx, Package_QFP:LQFP-144_20x20mm_P0.5mm, symbol MCU_ST_STM32H7:STM32H743ZITx
- added U58, U62: TXU0202DTTR, ESLGSU_Parts_Lib:SOT833-1-XSON8, symbol ESLGSU_Parts_Lib:TXU0202-Q1
- added U59, U60: TMUX1574RSVR, ESLGSU_Parts_Lib:T-UQFN-16, symbol ESLGSU_Parts_Lib:TMUX1574RSVR
- added U61: FXMA2102L8X, symbol ESLGSU_Parts_Lib:FXMA2102L8X
- added U63: THVD1450DRBR, Package_DFN_QFN:DFN-8-1EP_3x3mm_P0.65mm_EP1.55x2.4mm, symbol ESLGSU_Parts_Lib:THVD1450
- added U64: TCAN1051GVDRBRQ, Package_DFN_QFN:DFN-8-1EP_3x3mm_P0.65mm_EP1.55x2.4mm, symbol ESLGSU_Parts_Lib:TCAN1051GVDRBRQ1
- added U66 (x2): 74LS573, symbol 74xx:74LS573
- added U68, U70, U72: TPS2115ADRBR, Package_SON:VSON-8-1EP_3x3mm_P0.65mm_EP1.65x2.4mm_ThermalVias, symbol ESLGSU_Parts_Lib:TPS2115ADRBR
Connections:
- net CAN1_RX: now also U37.139 (PB8)
- net CAN1_SE: now also R10.1, R10.2, U66.15 (Q4)
- net CAN1_TX: now also U37.140 (PB9)
- net GND: now also U34.15 (SEL), U44.15 (SEL), C25.2, C25.2, C25.2, C25.2, C25.2, C25.2, C25.2, C25.2, C25.2, C25.2, C25.2, C25.2, C25.2, C25.2, C29.2, C29.2, C29.2, C29.2, C29.2, C6.1, C6.1, C6.1, C6.1, C6.1, C6.1, C6.1, C6.1, C6.1, C6.1, C6.1, C6.2, D1.1 (K), J2.6 (Pin_6), R10.1, R10.1, R10.1, R10.2, R10.2, R10.2, R10.2, R10.2, R10.2, U37.107 (VSS), U37.120 (VSS), U37.130 (VSS), U37.143 (PDR_ON), U37.16 (VSS), U37.31 (VSSA), U37.38 (VSS), U37.51 (VSS), U37.61 (VSS), U37.83 (VSS), U37.94 (VSS), U58.2 (GND), U59.6 (GND), U60.15 (SEL), U60.6 (GND), U61.4 (GND), U62.2 (GND), U63.5 (GND), U63.9 (GND), U64.2 (GND), U64.9 (GND), U66.10 (GND), U66.10 (GND), U68.5 (GND), U68.9 (GND), U70.5 (GND), U70.9 (GND), U72.5 (GND), U72.9 (GND)
- net GPIO_A_SHIFT: now also U37.21 (PF9); no longer U44.15 (SEL)
- net GPIO_A_nEN: now also U37.20 (PF8); no longer R10.1, U44.13 (nEN)
- net GPIO_B_SHIFT: now also U37.49 (PF11); no longer U34.15 (SEL)
- net GPIO_B_nEN: now also U37.22 (PF10); no longer U34.13 (nEN)
- net I2C1_EN: now also R10.1, U66.19 (Q0)
- net I2C1_nPEN: now also U66.18 (Q1)
- net RS4851_RX: now also U37.114 (PD0)
- net RS4851_TX: now also U37.115 (PD1)
- net RS4851_TXE: now also U37.118 (PD4)
- net SPI1_SHIFT: now also U66.14 (Q5); no longer U46.12 (OE), U47.15 (SEL)
- net SPI1_nEN: now also U66.15 (Q4)
- net SPI2_SHIFT: now also U66.12 (Q7); no longer U43.12 (OE), U45.15 (SEL)
- net SPI2_nEN: now also U66.13 (Q6)
- net SYS_3V3: now also C6.2, C6.2, R10.1, R10.1, R10.1, R6.2, R6.2, U68.8 (IN1), U70.3 (D1), U70.8 (IN1); no longer C6.2, C6.2, C6.2, C6.2, C6.2, R10.1, R10.1, R10.1, R10.2, R10.2, R10.2, R10.2, RN7.1 (R1.1), RN7.2 (R2.1), U29.5 (VIO), U33.3 (VCCA), U33.6 (OE), U35.3 (VCCA), U35.6 (OE), U39.1 (VREF1), U43.1 (VCCA), U46.1 (VCCA)
- net SYS_5V: now also C6.2, C6.2, R10.1, R6.2, R6.2, U68.6 (IN2), U72.3 (D1), U72.8 (IN1); no longer C6.2, U29.3 (VCC)
- net UART1_REV: now also U66.18 (Q1)
- net UART1_nEN: now also U66.19 (Q0)
- net VBUS: now also R10.1, R10.2, R10.2, R10.2, R10.2, C6.1, C6.2, C6.2, R10.1, R10.1, R10.2, R6.1, R6.1, U58.7 (VCCB), U59.14 (VDD), U60.14 (VDD), U60.2 (D1), U60.5 (D2), U62.7 (VCCB), U63.8 (VCC), U66.20 (VCC), U68.7 (OUT)
- net _GPIO_1: now also U37.10 (PF0)
- net _GPIO_2: now also U37.11 (PF1)
- net _GPIO_3: now also U37.12 (PF2)
- net _GPIO_4: now also U37.13 (PF3)
- net _GPIO_5: now also U37.14 (PF4)
- net _GPIO_6: now also U37.15 (PF5)
- net _GPIO_7: now also U37.18 (PF6)
- net _GPIO_8: now also U37.19 (PF7)
- net _I2C1_SCL: now also U37.136 (PB6)
- net _I2C1_SDA: now also U37.137 (PB7)
- net _SPI1_MISO: now also U37.75 (PB14)
- net _SPI1_MOSI: now also U37.76 (PB15)
- net _SPI1_NSS: now also U37.73 (PB12)
- net _SPI1_SCK: now also U37.74 (PB13)
- net _SPI2_MISO: now also U37.66 (PE13)
- net _SPI2_MOSI: now also U37.67 (PE14)
- net _SPI2_NSS: now also U37.64 (PE11)
- net _SPI2_SCK: now also U37.65 (PE12)
- net _UART1_RX: now also U37.37 (PA3)
- net _UART1_TX: now also U37.36 (PA2)
- new net: R10.1, U72.4 (ILIM)
- new net: R6.2, U37.101 (PA9)
- new net: R6.2, U37.102 (PA10)
- new net: C29.1, U37.106 (VCAP)
- new net: C29.1, U37.71 (VCAP)
- new net: RN16.1 (R1.1), U62.1 (B2), U63.1 (R)
- new net: RN16.2 (R2.1), U62.8 (B1Y), U63.4 (D)
- new net: R10.1, U60.16 (S1A)
- new net: R10.1, U60.3 (S2A)
- new net: D10.2 (A), J2.1 (Pin_1)
- new net: C6.2, R10.2, U61.8 (VREF2)
- new net: R10.1, U70.4 (ILIM)
- new net: D1.2 (A), R8.2
- new net: R10.1, U68.4 (ILIM)
- new net: U58.1 (B2), U59.1 (S1B), U59.3 (S2A)
- new net: U58.8 (B1Y), U59.16 (S1A), U59.4 (S2B)
- new net BOOTLDR: R10.2, U37.138 (BOOT0)
- new net BUS_3V3: R6.2
- new net BUS_5V: R6.2
- new net CAN2_H: R10.1, U64.7 (CANH)
- new net CAN2_L: R10.2, U64.6 (CANL)
- new net CAN2_RX: U37.78 (PD9), U64.4 (RXD)
- new net CAN2_SE: R10.1, R10.2, U64.8 (S), U66.14 (Q5)
- new net CAN2_TX: U37.79 (PD10), U64.1 (TXD)
- new net CFG_LOAD: U37.8 (PC14), U66.11 (Load), U66.11 (Load)
- new net CONFIG_nOE: R10.1, R10.1, U37.9 (PC15), U66.1 (OE), U66.1 (OE)
- new net GPIO_nEN: R10.1, U34.13 (nEN), U44.13 (nEN)
- new net I2C2_EN: R10.1, U61.5 (OE), U66.17 (Q2)
- new net I2C2_SCL: R10.2, RN14.2 (R2.1), RN15.3 (R2.2), U61.7 (SCL2)
- new net I2C2_SDA: R10.2, RN14.1 (R1.1), RN15.4 (R1.2), U61.6 (SDA2)
- new net I2C2_nPEN: R10.2, U60.13 (nEN), U66.16 (Q3)
- new net LED: R8.1, U37.34 (PA0)
- new net PISER_RX: R6.1
- new net PISER_TX: R6.1
- new net PISPI_MISO: U37.42 (PA6)
- new net PISPI_MOSI: U37.43 (PA7)
- new net PISPI_NSS: U37.40 (PA4)
- new net PISPI_SCK: U37.41 (PA5)
- new net PWR_nEN: R10.2, R10.2, U70.2 (D0), U72.2 (D0)
- new net RS4852_A: R10.2, U63.6 (A)
- new net RS4852_B: R10.1, U63.7 (B)
- new net RS4852_RX: RN16.4 (R1.2), U37.116 (PD2), U62.4 (A2Y)
- new net RS4852_TX: RN16.3 (R2.2), U37.113 (PC12), U62.5 (A1)
- new net RS4852_TXE: R10.1, U37.119 (PD5), U63.2 (nRE), U63.3 (DE)
- new net SPI_SHIFT: U43.12 (OE), U45.15 (SEL), U46.12 (OE), U47.15 (SEL)
- new net SUB3V3: C25.1, C25.1, C25.1, C25.1, C25.1, C25.1, C25.1, C25.1, C25.1, C25.1, C25.1, C25.1, C25.1, C25.1, C29.1, C29.1, C29.1, C6.2, C6.2, C6.2, C6.2, C6.2, C6.2, C6.2, C6.2, D10.1 (K), R10.1, R10.1, R10.1, R10.1, R10.2, R10.2, R6.1, R6.1, RN15.1 (R1.1), RN15.2 (R2.1), RN7.1 (R1.1), RN7.2 (R2.1), U29.5 (VIO), U33.3 (VCCA), U33.6 (OE), U35.3 (VCCA), U35.6 (OE), U37.108 (VDD), U37.121 (VDD), U37.131 (VDD), U37.144 (VDD), U37.17 (VDD), U37.30 (VDD), U37.32 (VREF+), U37.33 (VDDA), U37.39 (VDD), U37.52 (VDD), U37.6 (VBAT), U37.62 (VDD), U37.72 (VDD), U37.84 (VDD), U37.95 (VDD33_USB), U39.1 (VREF1), U43.1 (VCCA), U46.1 (VCCA), U58.3 (VCCA), U58.6 (OE), U61.1 (VREF1), U62.3 (VCCA), U62.6 (OE), U64.5 (VIO), U66.20 (VCC), U70.7 (OUT), U72.7 (OUT)
- new net SUB5V: C6.2, C6.2, R10.2, R10.2, R6.1, R6.1, U29.3 (VCC), U64.3 (VCC)
- new net SWCLK: J2.4 (Pin_4), U37.109 (PA14)
- new net SWDIO: J2.3 (Pin_3), U37.105 (PA13)
- new net SWO: J2.5 (Pin_5), U37.133 (PB3)
- new net UART2_REV: U59.15 (SEL), U66.16 (Q3)
- new net UART2_RX: RN13.1 (R1.1), U59.5 (D2)
- new net UART2_TX: RN13.2 (R2.1), U59.2 (D1)
- new net UART2_nEN: R10.1, U59.13 (nEN), U66.17 (Q2)
- new net _CAN1_SE: U37.134 (PB4), U66.6 (D4)
- new net _CAN2_SE: U37.135 (PB5), U66.7 (D5)
- new net _I2C1_EN: U37.26 (PC0), U66.2 (D0)
- new net _I2C1_nPEN: U37.27 (PC1), U66.3 (D1)
- new net _I2C2_EN: U37.28 (PC2_C), U66.4 (D2)
- new net _I2C2_SCL: R10.2, RN14.3 (R2.2), U37.69 (PB10), U61.2 (SCL1)
- new net _I2C2_SDA: R10.2, RN14.4 (R1.2), U37.70 (PB11), U61.3 (SDA1)
- new net _I2C2_nPEN: U37.29 (PC3_C), U66.5 (D3)
- new net _SPI1_SHIFT: U37.45 (PC5), U66.7 (D5)
- new net _SPI1_nEN: U37.44 (PC4), U66.6 (D4)
- new net _SPI2_SHIFT: U37.97 (PC7), U66.9 (D7)
- new net _SPI2_nEN: U37.96 (PC6), U66.8 (D6)
- new net _UART1_REV: U37.53 (PF13), U66.3 (D1)
- new net _UART1_nEN: U37.50 (PF12), U66.2 (D0)
- new net _UART2_REV: U37.55 (PF15), U66.5 (D3)
- new net _UART2_RX: RN13.4 (R1.2), U37.112 (PC11), U58.4 (A2Y)
- new net _UART2_TX: RN13.3 (R2.2), U37.111 (PC10), U58.5 (A1)
- new net _UART2_nEN: U37.54 (PF14), U66.4 (D2)
- new net _nVB5V: U37.47 (PB1), U66.9 (D7)
- new net _nVBPWR: U37.46 (PB0), U66.8 (D6)
- new net nRST: J2.2 (Pin_2), U37.25 (NRST)
- new net nVB5V: R10.2, U66.12 (Q7), U68.3 (D1)
- new net nVBPWR: R10.2, U66.13 (Q6), U68.2 (D0)
- no-connect marks 14 -> 89
Other:
- note added: "Bus Power"
- note added: "Config Latches"
- note added: "Debug Header"
- note added: "Decoupling Capacitors"
- note added: "EPS Power Switches"
- note added: "Indicator LED"
- note added: "Microcontroller"
- note added: "VDDA: 1u, 100u VDD: 4.7u, 11x100n VREF: 1u, 100u VUSB: 100n"
- note added: "crystal can be added here"
- moved on the sheet: C6, R10, RN3, RN4, U34, U44
