File: ESLGSU_Main_uC.kicad_sch (KiCad schematic)
At the start: 134 parts, among them J2 Conn_01x06_Pin, U29 TCAN1051GVDRBRQ, U30 THVD1450DRBR, U31 TMUX1574RSVR, U32 TMUX1574RSVR, U33 TXU0202DTTR, U34 TMUX1574RSVR, U35 TXU0202DTTR, U37 STM32H743ZITx, U39 FXMA2102L8X, U43 TXB0104RUT, U44 TMUX1574RSVR, U45 TMUX1574RSVR, U46 TXB0104RUT, U47 TMUX1574RSVR, U58 TXU0202DTTR, U59 TMUX1574RSVR, U60 TMUX1574RSVR, U61 FXMA2102L8X, U62 TXU0202DTTR, U63 THVD1450DRBR, U64 TCAN1051GVDRBRQ, U66 74LS573, U68 TPS2115ADRBR, U70 TPS2115ADRBR, U72 TPS2115ADRBR

Commit message: Final schematic work, added battery charger, linked everything up
Parts:
- removed C6 (x2): 100n, Capacitor_SMD:C_0402_1005Metric, symbol Device:C_Small
- removed R10 (x11): 200K, Resistor_SMD:R_0402_1005Metric, symbol Device:R_Small_US
- removed R10 (x2): 510R, Resistor_SMD:R_0402_1005Metric, symbol Device:R_Small_US
- removed R6 (x2): 0R, Resistor_SMD:R_0402_1005Metric, symbol Device:R_Small_US
- removed U66 (x2): 74LS573, symbol 74xx:74LS573
- removed U70, U72: TPS2115ADRBR, Package_SON:VSON-8-1EP_3x3mm_P0.65mm_EP1.65x2.4mm_ThermalVias, symbol ESLGSU_Parts_Lib:TPS2115ADRBR
- added C6 (x5): 100n, Capacitor_SMD:C_0402_1005Metric, symbol Device:C_Small
- added J7: 10118194-0001LF, ESLGSU_Parts_Lib:AMPHENOL_10118194-0001LF, symbol Connector:USB_B_Micro
- added R10 (x7): 100K, Resistor_SMD:R_0402_1005Metric, symbol Device:R_Small_US
- added R10 (x15): 200K, Resistor_SMD:R_0402_1005Metric, symbol Device:R_Small_US
- added R10 (x2): 10K, Resistor_SMD:R_0402_1005Metric, symbol Device:R_Small_US
- added R10 (x2): 510R, Resistor_SMD:R_0402_1005Metric, symbol Device:R_Small_US
- added R6 (x3): 0R, Resistor_SMD:R_0402_1005Metric, symbol Device:R_Small_US
- added U52, U56: TPS2115ADRBR, Package_SON:VSON-8-1EP_3x3mm_P0.65mm_EP1.65x2.4mm_ThermalVias, symbol ESLGSU_Parts_Lib:TPS2115ADRBR
- added U57: CY8C9520A, Package_SO:SSOP-28_5.3x10.2mm_P0.65mm, symbol ESLGSU_Parts_Lib:CY8C9520A
- added U74: PCAL6524HEAZ, Package_DFN_QFN:HVQFN-32-1EP_5x5mm_P0.5mm_EP3.1x3.1mm, symbol ESLGSU_Parts_Lib:PCAL6524
- added U81: ESD7004MUTAG, symbol ESLGSU_Parts_Lib:ESD7004MUTAG
- added Y1: CSTNE8M00G55A, Crystal:Resonator_SMD_Murata_CSTxExxV-3Pin_3.0x1.1mm, symbol Device:Crystal_GND2_Small
- D10: footprint Diode_SMD:D_SOD-323 -> Diode_THT:D_DO-41_SOD81_P10.16mm_Horizontal
- R6: LCBPCB BOM (none) -> 0; now not fitted; now left out of the parts list
- renumbered J2 to J4, U68 to U73
Connections:
- net GPIO_A_SHIFT is gone; now on net _GPIO_8: U37.21 (PF9)
- net GPIO_A_nEN is gone; now on net _GPIO_7: U37.20 (PF8)
- net _SPI2_SHIFT is gone; now on net RS4852_RX: U37.97 (PC7)
- net _SPI2_nEN is gone; now on net RS4852_TX: U37.96 (PC6)
- net BUS_3V3: now also C6.2, U52.8 (IN1)
- net BUS_5V: now also C6.2, U56.8 (IN1)
- net CAN1_SE: now also U57.1 (P0_0), U74.1 (P0_0)
- net CAN2_SE: now also U57.2 (P0_1), U74.2 (P0_1)
- net GND: now also C6.1, C6.1, C6.1, C6.1, C6.1, J7.5 (GND), J7.S1 (S), J7.S2 (S), J7.S3 (S), J7.S4 (S), J7.S5 (S), J7.S6 (S), R10.1, R10.1, R10.1, R10.1, R10.1, R10.1, R10.1, R10.1, R10.2, R10.2, R10.2, R10.2, U52.5 (GND), U52.9 (GND), U56.5 (GND), U56.9 (GND), U57.13 (A0), U57.14 (GND), U57.9 (GND), U74.25 (GND), U81.3 (GND), U81.8 (GND), Y1.2
- net GPIO_nEN: now also R10.1, R10.2, U57.20 (P1_7_A4), U74.16 (P1_7)
- net I2C1_EN: now also U57.5 (P0_4), U74.5 (P0_4)
- net I2C1_nPEN: now also R10.1, R10.1, U57.6 (P0_5), U74.6 (P0_5)
- net I2C2_EN: now also U57.7 (P0_6), U74.7 (P0_6)
- net I2C2_nPEN: now also R10.1, R10.1, U57.8 (P0_7), U74.8 (P0_7)
- net PISER_RX: now also R6.1
- net PISER_TX: now also R6.1
- net RS4851_TXE: now also R10.1; no longer R10.1, U30.2 (nRE), U30.3 (DE)
- net RS4852_RX: no longer U37.116 (PD2)
- net RS4852_TX: no longer U37.113 (PC12)
- net RS4852_TXE: now also R10.1; no longer R10.1, U63.2 (nRE), U63.3 (DE)
- net SPI1_nEN: now also R10.1, R10.2, U57.23 (P1_4), U74.13 (P1_4)
- net SPI2_nEN: now also R10.1, R10.2, U57.22 (P1_5_A6), U74.14 (P1_5)
- net SPI_SHIFT: now also R10.2, U57.21 (P1_6_A5), U74.15 (P1_6)
- net SUB3V3: now also U52.7 (OUT); no longer RN15.1 (R1.1), RN15.2 (R2.1), RN7.1 (R1.1), RN7.2 (R2.1)
- net SUB5V: now also U56.7 (OUT)
- net SYS_3V3: now also C6.2, C6.2, R10.1, R10.1, R10.1, R10.1, R10.1, U52.6 (IN2), U57.28 (VDD), U74.27 (VDDP), U74.31 (VDDI)
- net SYS_5V: now also C6.2, U56.6 (IN2)
- net UART1_REV: now also R10.2, U57.26 (P1_1), U74.10 (P1_1)
- net UART1_nEN: now also R10.1, R10.2, U57.27 (P1_0), U74.9 (P1_0)
- net UART2_REV: now also R10.2, U57.24 (P1_3), U74.12 (P1_3)
- net UART2_nEN: now also R10.1, R10.2, U57.25 (P1_2), U74.11 (P1_2)
- net VBUS: now also RN15.1 (R1.1), RN15.2 (R2.1), RN7.1 (R1.1), RN7.2 (R2.1), R10.2, R10.2, R10.2, R10.2, R10.2, R10.2, R10.2
- net _GPIO_1: now also U37.12 (PF2); no longer U37.10 (PF0)
- net _GPIO_2: now also U37.13 (PF3); no longer U37.11 (PF1)
- net _GPIO_3: now also U37.14 (PF4); no longer U37.12 (PF2)
- net _GPIO_4: now also U37.15 (PF5); no longer U37.13 (PF3)
- net _GPIO_5: now also U37.18 (PF6); no longer U37.14 (PF4)
- net _GPIO_6: now also U37.19 (PF7); no longer U37.15 (PF5)
- net _GPIO_7: no longer U37.18 (PF6)
- net _GPIO_8: no longer U37.19 (PF7)
- net _I2C2_SCL: now also U37.11 (PF1); no longer U37.69 (PB10)
- net _I2C2_SDA: now also U37.10 (PF0); no longer U37.70 (PB11)
- net _SPI1_MISO: now also U37.112 (PC11); no longer U37.75 (PB14)
- net _SPI1_MOSI: now also U37.113 (PC12); no longer U37.76 (PB15)
- net _SPI1_NSS: now also U37.110 (PA15); no longer U37.73 (PB12)
- net _SPI1_SCK: now also U37.111 (PC10); no longer U37.74 (PB13)
- net _UART2_RX: now also U37.70 (PB11); no longer U37.112 (PC11)
- net _UART2_TX: now also U37.69 (PB10); no longer U37.111 (PC10)
- net USB_VBUS: now reaches U37.101 (PA9)
- net USB_VBUS: now also J7.1 (VBUS), U81.1 (IO1), U81.10 (NC1)
- net USB_ID: now reaches U37.102 (PA10)
- net USB_ID: now also J7.4 (ID), U81.5 (IO4), U81.6 (NC4)
- net USB_D-: now reaches U37.103 (PA11)
- net USB_D-: now also J7.2 (D-), U81.2 (IO2), U81.9 (NC2)
- net USB_D+: now reaches U37.104 (PA12)
- net USB_D+: now also J7.3 (D+), U81.4 (IO3), U81.7 (NC3)
- net at U37.23 (PH0): now also Y1.1
- net at U37.24 (PH1): now also R6.1
- net CFG_LOAD: no longer names the net of U37.8 (PC14)
- net CONFIG_nOE: no longer names the net of U37.9 (PC15)
- net GPIO_B_SHIFT: no longer names the net of U37.49 (PF11)
- net GPIO_B_nEN: no longer names the net of U37.22 (PF10)
- net _CAN1_SE: no longer names the net of U37.134 (PB4)
- net _CAN2_SE: no longer names the net of U37.135 (PB5)
- net _I2C1_EN: no longer names the net of U37.26 (PC0)
- net _I2C1_nPEN: no longer names the net of U37.27 (PC1)
- net _I2C2_EN: no longer names the net of U37.28 (PC2_C)
- net _I2C2_nPEN: no longer names the net of U37.29 (PC3_C)
- net _SPI1_SHIFT: no longer names the net of U37.45 (PC5)
- net _SPI1_nEN: no longer names the net of U37.44 (PC4)
- net _UART1_REV: no longer names the net of U37.53 (PF13)
- net _UART1_nEN: no longer names the net of U37.50 (PF12)
- net _UART2_REV: no longer names the net of U37.55 (PF15)
- net _UART2_nEN: no longer names the net of U37.54 (PF14)
- net _nVB5V: no longer names the net of U37.47 (PB1)
- net _nVBPWR: no longer names the net of U37.46 (PB0)
- net nVB5V renamed nVT5V
- net nVT5V: now also U57.17 (P2_1_A2), U74.18 (P2_1)
- net nVBPWR renamed nVT3V3
- net nVT3V3: now also U57.18 (P2_0_A3), U74.17 (P2_0)
- new net: R10.1, U52.4 (ILIM)
- new net: R6.2, U37.75 (PB14)
- new net: R6.2, U37.76 (PB15)
- new net: R10.1, U56.4 (ILIM)
- new net: R10.2, U74.28 (nRST)
- new net: R6.2, Y1.3
- new net CFGI2C_SCL: U57.10 (SCL), U74.26 (ADDR), U74.29 (SCL)
- new net CFGI2C_SDA: U57.11 (SDA), U74.30 (SDA)
- new net RS4851_EN: R10.1, R10.2, U30.2 (nRE), U30.3 (DE), U57.3 (P0_2), U74.3 (P0_2)
- new net RS4852_EN: R10.1, R10.2, U57.4 (P0_3), U63.2 (nRE), U63.3 (DE), U74.4 (P0_3)
- new net nVBUS: R10.2, R10.2, U52.2 (D0), U56.2 (D0), U57.12 (P2_3_A1), U74.19 (P2_2)
- new net nVSYS: R10.2, R10.2, U52.3 (D1), U56.3 (D1), U57.15 (P2_2_WD), U74.20 (P2_3)
- no-connect marks 89 -> 110
Other:
- note added: "Addr: 0100000"
- note added: "Addr: 0100000 1010000"
- note added: "Config Expander Options"
- note added: "Subcircuit Power Switches"
- note added: "Transceiver Power"
- note added: "USB Port"
- note removed: "Bus Power"
- note removed: "Config Latches"
- note removed: "EPS Power Switches"
- note removed: "crystal can be added here"
- moved on the sheet: C29, C6, D1, D10, J4, R10, R6, R8, RN3, RN4, U34, U37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

Commit message: Last tweaks on schematic
Parts:
- added TP1 (x3): TestPoint, TestPoint:TestPoint_Pad_D1.5mm, symbol Connector:TestPoint
- D11: renamed from D10; footprint Diode_THT:D_DO-41_SOD81_P10.16mm_Horizontal -> Diode_SMD:D_SOD-323
- U54: renamed from U81; footprint (none) -> ESLGSU_Parts_Lib:UDFN10_ESD
- U58: renamed from U39; footprint (none) -> ESLGSU_Parts_Lib:UQFN8_MICROPAK
- U59: renamed from U61; footprint (none) -> ESLGSU_Parts_Lib:UQFN8_MICROPAK
- renumbered J7 to J5, J4 to J6, RN5 to RN10, RN16 to RN11, RN6 to RN12, RN7 to RN13, RN13 to RN16, RN2 to RN17, RN8 to RN18, RN1 to RN19, RN3 to RN8, RN4 to RN9, U29 to U45, U64 to U46, U44 to U47, U57 to U48, U33 to U49, U62 to U50, U30 to U51, U63 to U52, U34 to U53, U74 to U55, U31 to U56, U60 to U57, U58 to U60, U35 to U61, U59 to U62, U32 to U63, U37 to U64, U73 to U65, U43 to U66, U46 to U67, U45 to U68, U47 to U69, U52 to U70, U56 to U71
Connections:
- net SUB3V3: now also TP1.1
- net SUB5V: now also TP1.1
- net VBUS: now also TP1.1

Commit message: Some PCB work
Connections:
- net nVBUS: now also U55.20 (P2_3); no longer U55.19 (P2_2)
- net nVSYS: now also U55.19 (P2_2); no longer U55.20 (P2_3)
Changed lines of the file:
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@@
     (effects (font (size 1.27 1.27)) (justify right bottom))
-  )
-  (label "nVSYS" (at 184.15 91.44 0) (fields_autoplaced)
-    (effects (font (size 1.27 1.27)) (justify left bottom))
   )
   (label "UART1_REV" (at 158.75 104.14 180) (fields_autoplaced)
@@
     (effects (font (size 1.27 1.27)) (justify left bottom))
   )
+  (label "nVBUS" (at 184.15 91.44 0) (fields_autoplaced)
+    (effects (font (size 1.27 1.27)) (justify left bottom))
+  )
   (label "USB_VBUS" (at 124.46 35.56 0) (fields_autoplaced)
     (effects (font (size 1.27 1.27)) (justify left bottom))
@@
     (effects (font (size 1.27 1.27)) (justify left bottom))
   )
-  (label "nVBUS" (at 184.15 93.98 0) (fields_autoplaced)
-    (effects (font (size 1.27 1.27)) (justify left bottom))
-  )
   (label "_GPIO_5" (at 33.02 77.47 180) (fields_autoplaced)
     (effects (font (size 1.27 1.27)) (justify right bottom))
@@
     (effects (font (size 1.27 1.27)) (justify left bottom))
   )
+  (label "nVSYS" (at 184.15 93.98 0) (fields_autoplaced)
+    (effects (font (size 1.27 1.27)) (justify left bottom))
+  )

Commit message: Finished for production
Parts:
- U65, U70, U71: footprint Package_SON:VSON-8-1EP_3x3mm_P0.65mm_EP1.65x2.4mm_ThermalVias -> Package_SON:VSON-8-1EP_3x3mm_P0.65mm_EP1.65x2.4mm
Changed lines of the file:
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@@
       (effects (font (size 1.27 1.27)))
     )
-    (property "Footprint" "Package_SON:VSON-8-1EP_3x3mm_P0.65mm_EP1.65x2.4mm_ThermalVias" (at 186.69 236.22 0)
+    (property "Footprint" "Package_SON:VSON-8-1EP_3x3mm_P0.65mm_EP1.65x2.4mm" (at 186.69 236.22 0)
       (effects (font (size 1.27 1.27)) hide)
     )
@@
       (effects (font (size 1.27 1.27)))
     )
-    (property "Footprint" "Package_SON:VSON-8-1EP_3x3mm_P0.65mm_EP1.65x2.4mm_ThermalVias" (at 186.69 266.7 0)
+    (property "Footprint" "Package_SON:VSON-8-1EP_3x3mm_P0.65mm_EP1.65x2.4mm" (at 186.69 266.7 0)
       (effects (font (size 1.27 1.27)) hide)
     )
@@
       (effects (font (size 1.27 1.27)))
     )
-    (property "Footprint" "Package_SON:VSON-8-1EP_3x3mm_P0.65mm_EP1.65x2.4mm_ThermalVias" (at 191.77 193.04 0)
+    (property "Footprint" "Package_SON:VSON-8-1EP_3x3mm_P0.65mm_EP1.65x2.4mm" (at 191.77 193.04 0)
       (effects (font (size 1.27 1.27)) hide)
     )

Commit message: Removed some parts
Parts:
- removed C25 (x14), C6 (x27): 100n, Capacitor_SMD:C_0402_1005Metric, symbol Device:C_Small
- removed C29 (x2): 1u, Capacitor_SMD:C_0402_1005Metric, symbol Device:C_Small
- removed C29 (x2): 2.2u, Capacitor_SMD:C_0402_1005Metric, symbol Device:C_Small
- removed C29: 4.7u, Capacitor_SMD:C_0402_1005Metric, symbol Device:C_Small
- removed C6 (x2): 100p, Capacitor_SMD:C_0402_1005Metric, symbol Device:C_Small
- removed R10 (x4): 120R, Resistor_SMD:R_0805_2012Metric, symbol Device:R_Small_US
- removed R10 (x26): 200K, Resistor_SMD:R_0402_1005Metric, symbol Device:R_Small_US
- removed R10 (x10): 10K, Resistor_SMD:R_0402_1005Metric, symbol Device:R_Small_US
- removed R10 (x9): 100K, Resistor_SMD:R_0402_1005Metric, symbol Device:R_Small_US
- removed R10 (x3): 510R, Resistor_SMD:R_0402_1005Metric, symbol Device:R_Small_US
- removed R6 (x9): 0R, Resistor_SMD:R_0402_1005Metric, symbol Device:R_Small_US
- removed TP1 (x3): TestPoint, TestPoint:TestPoint_Pad_D1.5mm, symbol Connector:TestPoint
- added C25 (x14), C6 (x27): 100n, Capacitor_SMD:C_0402_1005Metric, symbol Device:C_Small
- added C29 (x2): 1u, Capacitor_SMD:C_0402_1005Metric, symbol Device:C_Small
- added C29 (x2): 2.2u, Capacitor_SMD:C_0402_1005Metric, symbol Device:C_Small
- added C29: 4.7u, Capacitor_SMD:C_0402_1005Metric, symbol Device:C_Small
- added C6 (x2): 100p, Capacitor_SMD:C_0402_1005Metric, symbol Device:C_Small
- added R10 (x26): 200K, Resistor_SMD:R_0402_1005Metric, symbol Device:R_Small_US
- added R10 (x9): 100K, Resistor_SMD:R_0402_1005Metric, symbol Device:R_Small_US
- added R10 (x10): 10K, Resistor_SMD:R_0402_1005Metric, symbol Device:R_Small_US
- added R10 (x3): 510R, Resistor_SMD:R_0402_1005Metric, symbol Device:R_Small_US
- added R10 (x4): 120R, Resistor_SMD:R_0805_2012Metric, symbol Device:R_Small_US
- added R6 (x9): 0R, Resistor_SMD:R_0402_1005Metric, symbol Device:R_Small_US
- added TP1 (x3): TestPoint, TestPoint:TestPoint_Pad_D1.5mm, symbol Connector:TestPoint
- D1, D11, J5, J6, R8, U45, U46, U47, U48, U49, U50, U51, U52, U53, U54, U56, U57, U58, U59, U60, U61, U62, U63, U64, U65, U66, U67, U68, U69, U70, U71, Y1: now not fitted; now left out of the parts list
Connections:
- net BOOTLDR: now also R10.2
- net BUS_3V3: now also C6.2, R6.2
- net BUS_5V: now also C6.2, R6.2
- net CAN1_H: now also R10.1
- net CAN1_L: now also R10.2
- net CAN1_SE: now also R10.1, R10.2
- net CAN2_H: now also R10.1
- net CAN2_L: now also R10.2
- net CAN2_SE: now also R10.1, R10.2
- net GND: now also C25.2, C25.2, C25.2, C25.2, C25.2, C25.2, C25.2, C25.2, C25.2, C25.2, C25.2, C25.2, C25.2, C25.2, C29.2, C29.2, C29.2, C29.2, C29.2, C6.1, C6.1, C6.1, C6.1, C6.1, C6.1, C6.1, C6.1, C6.1, C6.1, C6.1, C6.1, C6.1, C6.1, C6.1, C6.1, C6.1, C6.1, C6.1, C6.1, C6.1, C6.1, C6.1, C6.1, C6.1, C6.1, C6.1, C6.2, C6.2, R10.1, R10.1, R10.1, R10.1, R10.1, R10.1, R10.1, R10.1, R10.1, R10.1, R10.1, R10.2, R10.2, R10.2, R10.2, R10.2, R10.2, R10.2, R10.2, R10.2
- net GPIO_nEN: now also R10.1, R10.2
- net I2C1_EN: now also R10.1
- net I2C1_SCL: now also R10.2
- net I2C1_SDA: now also R10.2
- net I2C1_nPEN: now also R10.1, R10.1
- net I2C2_EN: now also R10.1
- net I2C2_SCL: now also R10.2
- net I2C2_SDA: now also R10.2
- net I2C2_nPEN: now also R10.1, R10.1
- net PISER_RX: now also R6.1
- net PISER_TX: now also R6.1
- net RS4851_A: now also R10.2
- net RS4851_B: now also R10.1
- net RS4851_EN: now also R10.1, R10.2
- net RS4851_TXE: now also R10.1
- net RS4852_A: now also R10.2
- net RS4852_B: now also R10.1
- net RS4852_EN: now also R10.1, R10.2
- net RS4852_TXE: now also R10.1
- net SPI1_nEN: now also R10.1, R10.2
- net SPI2_nEN: now also R10.1, R10.2
- net SPI_SHIFT: now also R10.2
- net SUB3V3: now also C25.1, C25.1, C25.1, C25.1, C25.1, C25.1, C25.1, C25.1, C25.1, C25.1, C25.1, C25.1, C25.1, C25.1, C29.1, C29.1, C29.1, C6.2, C6.2, C6.2, C6.2, C6.2, C6.2, C6.2, C6.2, R10.1, R10.1, R10.1, R10.1, R6.1, R6.1, TP1.1
- net SUB5V: now also C6.2, C6.2, R10.2, R10.2, R6.1, R6.1, TP1.1
- net SYS_3V3: now also C6.2, C6.2, C6.2, R10.1, R10.1, R10.1, R10.1, R10.1, R10.1, R10.1, R6.2, R6.2
- net SYS_5V: now also C6.2, C6.2, R6.2, R6.2
- net UART1_REV: now also R10.2
- net UART1_nEN: now also R10.1, R10.2
- net UART2_REV: now also R10.2
- net UART2_nEN: now also R10.1, R10.2
- net VBUS: now also C6.1, C6.1, C6.2, C6.2, C6.2, C6.2, C6.2, C6.2, C6.2, C6.2, R10.1, R10.1, R10.2, R10.2, R10.2, R10.2, R10.2, R10.2, R10.2, R6.1, R6.1, TP1.1
- net _I2C1_SCL: now also R10.2
- net _I2C1_SDA: now also R10.2
- net _I2C2_SCL: now also R10.2
- net _I2C2_SDA: now also R10.2
- net nVBUS: now also R10.2, R10.2
- net nVSYS: now also R10.2, R10.2
- net nVT3V3: now also R10.2
- net nVT5V: now also R10.2
- net at U70.4 (ILIM): now also R10.1
- net at U58.8 (VREF2): now also C6.2, R10.2
- net at U64.106 (VCAP): now also C29.1
- net at U64.24 (PH1): now also R6.1
- net at U64.71 (VCAP): now also C29.1
- net at U64.75 (PB14): now also R6.2
- net at U64.76 (PB15): now also R6.2
- net at U56.16 (S1A): now also R10.1
- net at U71.4 (ILIM): now also R10.1
- net at U57.16 (S1A): now also R10.1
- net at U57.3 (S2A): now also R10.1
- net at U59.8 (VREF2): now also C6.2, R10.2
- net at U55.28 (nRST): now also R10.2
- net at U65.4 (ILIM): now also R10.1
- net at Y1.3: now also R6.2
- net at U56.3 (S2A): now also R10.1
