File: ESLGSU_Main_uC.kicad_sch (KiCad schematic)
At the start: 159 parts, among them J5 10118194-0001LF, J6 Conn_01x06_Pin, U45 TCAN1051GVDRBRQ, U46 TCAN1051GVDRBRQ, U47 TMUX1574RSVR, U48 CY8C9520A, U49 TXU0202DTTR, U50 TXU0202DTTR, U51 THVD1450DRBR, U52 THVD1450DRBR, U53 TMUX1574RSVR, U54 ESD7004MUTAG, U55 PCAL6524HEAZ, U56 TMUX1574RSVR, U57 TMUX1574RSVR, U58 FXMA2102L8X, U59 FXMA2102L8X, U60 TXU0202DTTR, U61 TXU0202DTTR, U62 TMUX1574RSVR, U63 TMUX1574RSVR, U64 STM32H743ZITx, U65 TPS2115ADRBR, U66 TXB0104RUT, U67 TXB0104RUT, U68 TMUX1574RSVR, U69 TMUX1574RSVR, U70 TPS2115ADRBR, U71 TPS2115ADRBR, Y1 CSTNE8M00G55A

Commit message: Should be done with minimal version
Parts:
- C25, C29, C6, D1, D11, J5, J6, R10, R8, U45, U46, U47, U48, U49, U50, U51, U52, U53, U54, U56, U57, U58, U59, U60, U61, U62, U63, U64, U65, U66, U67, U68, U69, U70, U71, Y1: now not fitted; now left out of the parts list

Commit message: Fixed MP28167, debug headers
Parts:
- J6: LCSC Part C2881612 -> C2881573
Changed lines of the file:
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@@
       (effects (font (size 1.27 1.27)) hide)
     )
-    (property "LCSC Part" "C2881612" (at 203.2 152.4 0)
+    (property "LCSC Part" "C2881573" (at 203.2 152.4 0)
       (effects (font (size 1.27 1.27)) hide)
     )

Commit message: Final V1 board with notes
Parts:
- J6: LCSC Part C2881573 -> C2881496
Changed lines of the file:
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@@
       (effects (font (size 1.27 1.27)) hide)
     )
-    (property "LCSC Part" "C2881573" (at 203.2 152.4 0)
+    (property "LCSC Part" "C2881496" (at 203.2 152.4 0)
       (effects (font (size 1.27 1.27)) hide)
     )
