File: ESLGSU_Misc_uCs.kicad_sch (KiCad schematic)
At the start: 0 parts

Commit message: uC Interface work
Other:
- company: (none) -> Electronic Systems Laboratory
Changed lines of the file:
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@@
 (kicad_sch (version 20230121) (generator eeschema)
   (paper "A4")
+  (title_block
+    (date "2024-01-18")
+    (rev "1")
+    (company "Electronic Systems Laboratory")
+  )
 )

Commit message: Finished interfaces work
Parts:
- added U38: STM32F072VBTx, Package_QFP:LQFP-100_14x14mm_P0.5mm, symbol MCU_ST_STM32F0:STM32F072VBTx
Connections:
- new net: U38.27 (VSS), U38.49 (VSS), U38.74 (VSS), U38.99 (VSS)
Changed lines of the file:
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@@
     (company "Electronic Systems Laboratory")
   )
+  (symbol (lib_id "MCU_ST_STM32F0:STM32F072VBTx") (at 63.5 100.33 0) (unit 1)
+    (in_bom yes) (on_board yes) (dnp no) (fields_autoplaced)
+    (property "Reference" "U38" (at 68.2341 168.91 0)
+      (effects (font (size 1.27 1.27)) (justify left))
+    )
+    (property "Value" "STM32F072VBTx" (at 68.2341 171.45 0)
+      (effects (font (size 1.27 1.27)) (justify left))
+    )
+    (property "Footprint" "Package_QFP:LQFP-100_14x14mm_P0.5mm" (at 48.26 166.37 0)
+      (effects (font (size 1.27 1.27)) (justify right) hide)
+    )
+    (property "Datasheet" "https://www.st.com/resource/en/datasheet/stm32f072vb.pdf" (at 63.5 100.33 0)
+      (effects (font (size 1.27 1.27)) hide)
+    )
+    (pin "1")
+    (pin "10")
+    (pin "100")
+    (pin "11")
+    (pin "12")
+    (pin "13")
+    (pin "14")
+    (pin "15")
+    (pin "16")
+    (pin "17")
+    (pin "18")
+    (pin "19")
+    (pin "2")
+    (pin "20")
+    (pin "21")
+    (pin "22")
+    (pin "23")
+    (pin "24")
+    (pin "25")
+    (pin "26")
+    (pin "27")
+    (pin "28")
+    (pin "29")
+    (pin "3")
+    (pin "30")
+    (pin "31")
+    (pin "32")
+    (pin "33")
+    (pin "34")
+    (pin "35")
+    (pin "36")
+    (pin "37")
+    (pin "38")
+    (pin "39")
+    (pin "4")
+    (pin "40")
+    (pin "41")
+    (pin "42")
+    (pin "43")
+    (pin "44")
+    (pin "45")
+    (pin "46")
+    (pin "47")
+    (pin "48")
+    (pin "49")
+    (pin "5")
+    (pin "50")
+    (pin "51")
+    (pin "52")
+    (pin "53")
+    (pin "54")
+    (pin "55")
+    (pin "56")
+    (pin "57")
+    (pin "58")
+    (pin "59")
+    (pin "6")
+    (pin "60")
+    (pin "61")
+    (pin "62")
+    (pin "63")
+    (pin "64")
+    (pin "65")
+    (pin "66")
+    (pin "67")
+    (pin "68")
+    (pin "69")
+    (pin "7")
+    (pin "70")
+    (pin "71")
+    (pin "72")
+    (pin "73")
+    (pin "74")
+    (pin "75")
+    (pin "76")
+    (pin "77")
+    (pin "78")
+    (pin "79")
+    (pin "8")
+    (pin "80")
+    (pin "81")
+    (pin "82")
+    (pin "83")
+    (pin "84")
+    (pin "85")
+    (pin "86")
+    (pin "87")
+    (pin "88")
+    (pin "89")
+    (pin "9")
+    (pin "90")
+    (pin "91")
+    (pin "92")
+    (pin "93")
+    (pin "94")
+    (pin "95")
+    (pin "96")
+    (pin "97")
+    (pin "98")
+    (pin "99")
+    (instances
+      (project "ESLGSU"
+        (path "/b556fa32-e0cb-409c-ac85-9f2ac606be79/c41d3519-67b9-43b9-97c4-d20822b3d6ca"
+          (reference "U38") (unit 1)
+        )
+        (path "/b556fa32-e0cb-409c-ac85-9f2ac606be79/bf0312e4-5726-4684-b2e9-b4b5c1d8e876"
+          (reference "U41") (unit 1)
+        )
+      )
+    )
+  )
 )

Commit message: Tried to prepare for order
Parts:
- removed U38: STM32F072VBTx, Package_QFP:LQFP-100_14x14mm_P0.5mm, symbol MCU_ST_STM32F0:STM32F072VBTx
- added U41: STM32F072CBUx, Package_DFN_QFN:QFN-48-1EP_7x7mm_P0.5mm_EP5.6x5.6mm, symbol MCU_ST_STM32F0:STM32F072CBUx
Connections:
- new net: U41.23 (VSS), U41.35 (VSS), U41.47 (VSS), U41.49 (VSS)
Changed lines of the file:
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@@
     (company "Electronic Systems Laboratory")
   )
-  (symbol (lib_id "MCU_ST_STM32F0:STM32F072VBTx") (at 63.5 100.33 0) (unit 1)
+  (symbol (lib_id "MCU_ST_STM32F0:STM32F072CBUx") (at 62.23 118.11 0) (unit 1)
     (in_bom yes) (on_board yes) (dnp no) (fields_autoplaced)
-    (property "Reference" "U38" (at 68.2341 168.91 0)
+    (property "Reference" "U41" (at 66.9641 156.21 0)
       (effects (font (size 1.27 1.27)) (justify left))
     )
-    (property "Value" "STM32F072VBTx" (at 68.2341 171.45 0)
+    (property "Value" "STM32F072CBUx" (at 66.9641 158.75 0)
       (effects (font (size 1.27 1.27)) (justify left))
     )
-    (property "Footprint" "Package_QFP:LQFP-100_14x14mm_P0.5mm" (at 48.26 166.37 0)
+    (property "Footprint" "Package_DFN_QFN:QFN-48-1EP_7x7mm_P0.5mm_EP5.6x5.6mm" (at 49.53 153.67 0)
       (effects (font (size 1.27 1.27)) (justify right) hide)
     )
-    (property "Datasheet" "https://www.st.com/resource/en/datasheet/stm32f072vb.pdf" (at 63.5 100.33 0)
+    (property "Datasheet" "https://www.st.com/resource/en/datasheet/stm32f072cb.pdf" (at 62.23 118.11 0)
       (effects (font (size 1.27 1.27)) hide)
     )
-    (pin "1")
-    (pin "10")
-    (pin "100")
-    (pin "11")
-    (pin "12")
+    (pin "3")
+    (pin "9")
+    (pin "46")
+    (pin "32")
+    (pin "15")
+    (pin "2")
+    (pin "24")
+    (pin "38")
     (pin "13")
-    (pin "14")
-    (pin "15")
     (pin "16")
-    (pin "17")
-    (pin "18")
-    (pin "19")
-    (pin "2")
-    (pin "20")
-    (pin "21")
-    (pin "22")
-    (pin "23")
-    (pin "24")
-    (pin "25")
-    (pin "26")
-    (pin "27")
-    (pin "28")
-    (pin "29")
-    (pin "3")
-    (pin "30")
     (pin "31")
-    (pin "32")
-    (pin "33")
     (pin "34")
-    (pin "35")
-    (pin "36")
-    (pin "37")
-    (pin "38")
-    (pin "39")
-    (pin "4")
-    (pin "40")
     (pin "41")
     (pin "42")
+    (pin "35")
+    (pin "44")
+    (pin "11")
+    (pin "18")
+    (pin "33")
+    (pin "37")
+    (pin "12")
+    (pin "1")
+    (pin "22")
+    (pin "10")
+    (pin "17")
+    (pin "19")
+    (pin "23")
+    (pin "30")
+    (pin "4")
+    (pin "29")
+    (pin "40")
+    (pin "25")
+    (pin "45")
+    (pin "48")
+    (pin "28")
+    (pin "49")
+    (pin "39")
+    (pin "47")
     (pin "43")
-    (pin "44")
-    (pin "45")
-    (pin "46")
-    (pin "47")
-    (pin "48")
-    (pin "49")
     (pin "5")
-    (pin "50")
-    (pin "51")
-    (pin "52")
-    (pin "53")
-    (pin "54")
-    (pin "55")
-    (pin "56")
-    (pin "57")
-    (pin "58")
-    (pin "59")
+    (pin "7")
+    (pin "8")
+    (pin "27")
+    (pin "21")
+    (pin "14")
+    (pin "26")
+    (pin "36")
+    (pin "20")
     (pin "6")
-    (pin "60")
-    (pin "61")
-    (pin "62")
-    (pin "63")
-    (pin "64")
-    (pin "65")
-    (pin "66")
-    (pin "67")
-    (pin "68")
-    (pin "69")
-    (pin "7")
-    (pin "70")
-    (pin "71")
-    (pin "72")
-    (pin "73")
-    (pin "74")
-    (pin "75")
-    (pin "76")
-    (pin "77")
-    (pin "78")
-    (pin "79")
-    (pin "8")
-    (pin "80")
-    (pin "81")
-    (pin "82")
-    (pin "83")
-    (pin "84")
-    (pin "85")
-    (pin "86")
-    (pin "87")
-    (pin "88")
-    (pin "89")
-    (pin "9")
-    (pin "90")
-    (pin "91")
-    (pin "92")
-    (pin "93")
-    (pin "94")
-    (pin "95")
-    (pin "96")
-    (pin "97")
-    (pin "98")
-    (pin "99")
     (instances
       (project "ESLGSU"
-        (path "/b556fa32-e0cb-409c-ac85-9f2ac606be79/c41d3519-67b9-43b9-97c4-d20822b3d6ca"
-          (reference "U38") (unit 1)
-        )
         (path "/b556fa32-e0cb-409c-ac85-9f2ac606be79/bf0312e4-5726-4684-b2e9-b4b5c1d8e876"
           (reference "U41") (unit 1)

Commit message: Schematic work
Parts:
- removed U41: STM32F072CBUx, Package_DFN_QFN:QFN-48-1EP_7x7mm_P0.5mm_EP5.6x5.6mm, symbol MCU_ST_STM32F0:STM32F072CBUx
- added C25 (x3), C6 (x5): 100n, Capacitor_SMD:C_0402_1005Metric, symbol Device:C_Small
- added C25: 10n, Capacitor_SMD:C_0402_1005Metric, symbol Device:C_Small
- added C29: 4.7u, Capacitor_SMD:C_0402_1005Metric, symbol Device:C_Small
- added C29: 1u, Capacitor_SMD:C_0402_1005Metric, symbol Device:C_Small
- added C6: 100p, Capacitor_SMD:C_0402_1005Metric, symbol Device:C_Small
- added D1: TZ-P2-0603GTCS1-0.6T, LED_SMD:LED_0603_1608Metric, symbol Device:LED
- added J2: Conn_01x06_Pin, Connector_PinHeader_1.27mm:PinHeader_1x06_P1.27mm_Vertical_SMD_Pin1Right, symbol Connector:Conn_01x06_Pin
- added R10 (x4): 10K, Resistor_SMD:R_0402_1005Metric, symbol Device:R_Small_US
- added R10 (x5): 200K, Resistor_SMD:R_0402_1005Metric, symbol Device:R_Small_US
- added R10: 120R, Resistor_SMD:R_0805_2012Metric, symbol Device:R_Small_US
- added R6 (x2): 0R, Resistor_SMD:R_0402_1005Metric, symbol Device:R_Small_US
- added R8: 33R, Resistor_SMD:R_0402_1005Metric, symbol Device:R_Small_US
- added RN6: 0R, Resistor_SMD:R_Array_Convex_2x0402, symbol Device:R_Pack02
- added RN7: 10K, Resistor_SMD:R_Array_Convex_2x0402, symbol Device:R_Pack02
- added U29: TCAN1051GVDRBRQ, Package_DFN_QFN:DFN-8-1EP_3x3mm_P0.65mm_EP1.55x2.4mm, symbol ESLGSU_Parts_Lib:TCAN1051GVDRBRQ1
- added U31, U44: TMUX1574RSVR, ESLGSU_Parts_Lib:T-UQFN-16, symbol ESLGSU_Parts_Lib:TMUX1574RSVR
- added U36: TXB0104RUT, ESLGSU_Parts_Lib:T-UQFN-12, symbol ESLGSU_Parts_Lib:TXB0104RUTR
- added U39: FXMA2102L8X, symbol ESLGSU_Parts_Lib:FXMA2102L8X
- added U41: STM32L431CCTx, Package_QFP:LQFP-48_7x7mm_P0.5mm, symbol MCU_ST_STM32L4:STM32L431CCTx
Connections:
- new net: R6.2, U41.21 (PB10)
- new net: R6.2, U41.22 (PB11)
- new net: C6.2, R10.2, U39.8 (VREF2)
- new net: D1.2 (A), R8.2
- new net: U36.10 (B1), U44.1 (S1B)
- new net: U36.7 (B4), U44.11 (S4B)
- new net: U36.9 (B2), U44.4 (S2B)
- new net: U36.8 (B3), U44.8 (S3B)
- new net: R10.1, U31.16 (S1A)
- new net: R10.1, U31.3 (S2A)
- new net BOOTLDR: R10.2, U41.44 (PH3)
- new net BUS_5V: U41.41 (PB5)
- new net CAN1_H: R10.1, U29.7 (CANH)
- new net CAN1_L: R10.2, U29.6 (CANL)
- new net CAN1_RX: U29.4 (RXD), U41.45 (PB8)
- new net CAN1_SE: R10.1, U29.8 (S), U41.40 (PB4)
- new net CAN1_TX: U29.1 (TXD), U41.46 (PB9)
- new net GND: C25.2, C25.2, C25.2, C25.2, C29.2, C29.2, C6.1, C6.1, C6.1, C6.1, C6.1, C6.2, D1.1 (K), J2.6 (Pin_6), R10.1, U29.2 (GND), U29.9 (GND), U31.15 (SEL), U31.6 (GND), U36.6 (GND), U39.4 (GND), U41.23 (VSS), U41.35 (VSS), U41.47 (VSS), U41.8 (VSSA), U44.6 (GND)
- new net GPIO_1: U44.2 (D1)
- new net GPIO_2: U44.5 (D2)
- new net GPIO_3: U44.7 (D3)
- new net GPIO_4: U44.10 (D4)
- new net GPIO_A_SHIFT: U36.12 (OE), U41.17 (PA7), U44.15 (SEL)
- new net GPIO_A_nEN: R10.1, U41.16 (PA6), U44.13 (nEN)
- new net I2C1_EN: U39.5 (OE), U41.18 (PB0)
- new net I2C1_SCL: R10.2, RN6.2 (R2.1), RN7.3 (R2.2), U39.7 (SCL2)
- new net I2C1_SDA: R10.2, RN6.1 (R1.1), RN7.4 (R1.2), U39.6 (SDA2)
- new net I2C1_nPEN: R10.2, U31.13 (nEN), U41.19 (PB1)
- new net LED: R8.1, U41.20 (PB2)
- new net PISER_RX: R6.1
- new net PISER_TX: R6.1
- new net PISPI_MISO: U41.27 (PB14)
- new net PISPI_MOSI: U41.28 (PB15)
- new net PISPI_NSS: U41.25 (PB12)
- new net PISPI_SCK: U41.26 (PB13)
- new net SWCLK: J2.4 (Pin_4), U41.37 (PA14)
- new net SWDIO: J2.3 (Pin_3), U41.34 (PA13)
- new net SWO: J2.5 (Pin_5), U41.39 (PB3)
- new net SYS_3V3: C25.1, C25.1, C25.1, C25.1, C29.1, C29.1, C6.2, C6.2, J2.1 (Pin_1), R10.1, R10.1, R10.1, R10.2, R10.2, RN7.1 (R1.1), RN7.2 (R2.1), U29.5 (VIO), U36.1 (VCCA), U39.1 (VREF1), U41.24 (VDD), U41.36 (VDD), U41.48 (VDD), U41.9 (VDDA)
- new net SYS_5V: C6.2, U29.3 (VCC)
- new net VBUS: C6.1, C6.2, R10.1, U31.14 (VDD), U31.2 (D1), U31.5 (D2), U36.11 (VCCB), U44.14 (VDD)
- new net _GPIO_1: U36.2 (A1), U41.29 (PA8), U44.16 (S1A)
- new net _GPIO_2: U36.3 (A2), U41.30 (PA9), U44.3 (S2A)
- new net _GPIO_3: U36.4 (A3), U41.31 (PA10), U44.9 (S3A)
- new net _GPIO_4: U36.5 (A4), U41.32 (PA11), U44.12 (S4A)
- new net _I2C1_SCL: R10.2, RN6.3 (R2.2), U39.2 (SCL1), U41.42 (PB6)
- new net _I2C1_SDA: R10.2, RN6.4 (R1.2), U39.3 (SDA1), U41.43 (PB7)
- new net nRST: J2.2 (Pin_2), U41.7 (NRST)
- no-connect marks 0 -> 22
Other:
- note added: "CAN Transceiver"
- note added: "Debug Header"
- note added: "GPIO Transceiver"
- note added: "I2C Transceiver"
- note added: "crystal can be added here"

Commit message: Second last bit of schematic work
Parts:
- removed C25: 10n, Capacitor_SMD:C_0402_1005Metric, symbol Device:C_Small
- removed C6 (x2): 100n, Capacitor_SMD:C_0402_1005Metric, symbol Device:C_Small
- removed J2: Conn_01x06_Pin, Connector_PinHeader_1.27mm:PinHeader_1x06_P1.27mm_Vertical_SMD_Pin1Right, symbol Connector:Conn_01x06_Pin
- removed R10 (x2): 200K, Resistor_SMD:R_0402_1005Metric, symbol Device:R_Small_US
- removed U36: TXB0104RUT, ESLGSU_Parts_Lib:T-UQFN-12, symbol ESLGSU_Parts_Lib:TXB0104RUTR
- removed U41: STM32L431CCTx, Package_QFP:LQFP-48_7x7mm_P0.5mm, symbol MCU_ST_STM32L4:STM32L431CCTx
- added C25 (x2), C6 (x6): 100n, Capacitor_SMD:C_0402_1005Metric, symbol Device:C_Small
- added C29: 2.2u, Capacitor_SMD:C_0402_1005Metric, symbol Device:C_Small
- added D10: 1N5819, Diode_SMD:D_SOD-323, symbol Diode:1N5819
- added J3: Conn_01x06_Pin, Connector_PinHeader_1.27mm:PinHeader_1x06_P1.27mm_Vertical_SMD_Pin1Right, symbol Connector:Conn_01x06_Pin
- added R10 (x8): 200K, Resistor_SMD:R_0402_1005Metric, symbol Device:R_Small_US
- added R10: 100K, Resistor_SMD:R_0402_1005Metric, symbol Device:R_Small_US
- added R10 (x3): 510R, Resistor_SMD:R_0402_1005Metric, symbol Device:R_Small_US
- added R6 (x6): 0R, Resistor_SMD:R_0402_1005Metric, symbol Device:R_Small_US
- added RN3, RN4: 0R, Resistor_SMD:R_Array_Concave_4x0402, symbol Device:R_Pack04
- added U34: TMUX1574RSVR, ESLGSU_Parts_Lib:T-UQFN-16, symbol ESLGSU_Parts_Lib:TMUX1574RSVR
- added U55: STM32F412RETx, Package_QFP:LQFP-64_10x10mm_P0.5mm, symbol MCU_ST_STM32F4:STM32F412RETx
- added U66: 74LS573, symbol 74xx:74LS573
- added U68, U70, U72: TPS2115ADRBR, Package_SON:VSON-8-1EP_3x3mm_P0.65mm_EP1.65x2.4mm_ThermalVias, symbol ESLGSU_Parts_Lib:TPS2115ADRBR
Connections:
- net BOOTLDR: now also U55.60 (BOOT0)
- net BUS_5V: now also R6.2
- net CAN1_RX: now also U55.57 (PB5)
- net CAN1_SE: now also R10.1, R10.2, U66.15 (Q4)
- net CAN1_TX: now also U55.34 (PB13)
- net GND: now also U44.15 (SEL), C25.2, C25.2, C29.2, C6.1, C6.1, C6.1, C6.1, C6.1, C6.1, J3.6 (Pin_6), R10.1, R10.2, R10.2, R10.2, R10.2, U34.15 (SEL), U34.6 (GND), U55.12 (VSSA), U55.18 (VSS), U55.31 (VSS), U55.47 (VSS), U55.63 (VSS), U66.10 (GND), U68.5 (GND), U68.9 (GND), U70.5 (GND), U70.9 (GND), U72.5 (GND), U72.9 (GND)
- net GPIO_1: now also RN3.4 (R4.1)
- net GPIO_2: now also RN3.3 (R3.1)
- net GPIO_3: now also RN3.2 (R2.1)
- net GPIO_4: now also RN3.1 (R1.1)
- net GPIO_A_SHIFT: now also U55.16 (PA2); no longer U44.15 (SEL)
- net GPIO_A_nEN: now also U55.15 (PA1); no longer U44.13 (nEN)
- net I2C1_EN: now also R10.1, U66.17 (Q2)
- net I2C1_nPEN: now also U66.16 (Q3)
- net LED: now also U55.14 (PA0)
- net PISPI_MISO: now also U55.52 (PC11)
- net PISPI_MOSI: now also U55.53 (PC12)
- net PISPI_NSS: now also U55.50 (PA15)
- net PISPI_SCK: now also U55.51 (PC10)
- net SWCLK: now also J3.4 (Pin_4), U55.49 (PA14)
- net SWDIO: now also J3.3 (Pin_3), U55.46 (PA13)
- net SWO: now also J3.5 (Pin_5), U55.55 (PB3)
- net SYS_3V3: now also C6.2, C6.2, R10.1, R10.1, R10.1, R6.2, R6.2, U68.8 (IN1), U70.3 (D1), U70.8 (IN1); no longer C25.1, C25.1, C25.1, C29.1, C29.1, C6.2, R10.1, R10.1, R10.1, RN7.1 (R1.1), RN7.2 (R2.1), U29.5 (VIO), U39.1 (VREF1)
- net SYS_5V: now also C6.2, C6.2, R10.1, R6.2, R6.2, U68.6 (IN2), U72.3 (D1), U72.8 (IN1); no longer C6.2, U29.3 (VCC)
- net VBUS: now also R10.1, C6.2, C6.2, R10.2, R6.1, R6.1, U34.14 (VDD), U68.7 (OUT)
- net _GPIO_1: now also RN3.5 (R4.2), U55.8 (PC0)
- net _GPIO_2: now also RN3.6 (R3.2), U55.9 (PC1)
- net _GPIO_3: now also RN3.7 (R2.2), U55.10 (PC2)
- net _GPIO_4: now also RN3.8 (R1.2), U55.11 (PC3)
- net _I2C1_SCL: now also U55.58 (PB6)
- net _I2C1_SDA: now also U55.59 (PB7)
- net nRST: now also J3.2 (Pin_2), U55.7 (NRST)
- net at R6.2: now also U55.42 (PA9)
- net at R6.2: now also U55.43 (PA10)
- new net: D10.2 (A), J3.1 (Pin_1)
- new net: C29.1, U55.30 (VCAP_1)
- new net: R10.1, U72.4 (ILIM)
- new net: R10.1, U68.4 (ILIM)
- new net: R10.1, U70.4 (ILIM)
- new net BUS_3V3: R6.2
- new net CFG_LOAD: U55.3 (PC14), U66.11 (Load)
- new net CONFIG_nOE: R10.1, U55.4 (PC15), U66.1 (OE)
- new net GPIO_5: RN4.4 (R4.1), U34.2 (D1)
- new net GPIO_6: RN4.3 (R3.1), U34.5 (D2)
- new net GPIO_7: RN4.2 (R2.1), U34.7 (D3)
- new net GPIO_8: RN4.1 (R1.1), U34.10 (D4)
- new net GPIO_nEN: R10.1, U34.13 (nEN), U44.13 (nEN)
- new net PWR_nEN: R10.2, R10.2, U70.2 (D0), U72.2 (D0)
- new net SUB3V3: C25.1, C25.1, C25.1, C25.1, C25.1, C29.1, C29.1, C6.2, D10.1 (K), R10.1, R10.1, R10.2, R6.1, R6.1, RN7.1 (R1.1), RN7.2 (R2.1), U29.5 (VIO), U39.1 (VREF1), U55.1 (VBAT), U55.13 (VDDA), U55.19 (VDD), U55.32 (VDD), U55.48 (VDD), U55.64 (VDD), U66.20 (VCC), U70.7 (OUT), U72.7 (OUT)
- new net SUB5V: C6.2, R10.2, R6.1, R6.1, U29.3 (VCC)
- new net _CAN1_SE: U55.21 (PA5), U66.6 (D4)
- new net _GPIO_5: RN4.5 (R4.2), U34.16 (S1A)
- new net _GPIO_6: RN4.6 (R3.2), U34.3 (S2A)
- new net _GPIO_7: RN4.7 (R2.2), U34.9 (S3A)
- new net _GPIO_8: RN4.8 (R1.2), U34.12 (S4A)
- new net _I2C1_EN: U55.17 (PA3), U66.4 (D2)
- new net _I2C1_nPEN: U55.20 (PA4), U66.5 (D3)
- new net _nVB5V: U55.27 (PB1), U66.9 (D7)
- new net _nVBPWR: U55.26 (PB0), U66.8 (D6)
- new net nVB5V: R10.2, U66.12 (Q7), U68.3 (D1)
- new net nVBPWR: R10.2, U66.13 (Q6), U68.2 (D0)
- no-connect marks 22 -> 50
Other:
- note added: "Bus Power"
- note added: "Config Latch"
- note added: "Decoupling Capacitors"
- note added: "EPS Power Switches"
- note added: "Indicator LED"
- note added: "Microcontroller"
- note added: "VDDA: 1u, 100u VDD: 4.7u, 4x100n"
- moved on the sheet: C25, C29, D1, R10, R6, R8

Commit message: Final schematic work, added battery charger, linked everything up
Parts:
- removed C6 (x5): 100n, Capacitor_SMD:C_0402_1005Metric, symbol Device:C_Small
- removed R10 (x8): 200K, Resistor_SMD:R_0402_1005Metric, symbol Device:R_Small_US
- removed R10: 100K, Resistor_SMD:R_0402_1005Metric, symbol Device:R_Small_US
- removed R10 (x3): 510R, Resistor_SMD:R_0402_1005Metric, symbol Device:R_Small_US
- removed R6 (x6): 0R, Resistor_SMD:R_0402_1005Metric, symbol Device:R_Small_US
- removed RN4: 0R, Resistor_SMD:R_Array_Concave_4x0402, symbol Device:R_Pack04
- removed U34: TMUX1574RSVR, ESLGSU_Parts_Lib:T-UQFN-16, symbol ESLGSU_Parts_Lib:TMUX1574RSVR
- removed U66: 74LS573, symbol 74xx:74LS573
- removed U68, U70, U72: TPS2115ADRBR, Package_SON:VSON-8-1EP_3x3mm_P0.65mm_EP1.65x2.4mm_ThermalVias, symbol ESLGSU_Parts_Lib:TPS2115ADRBR
- added C6 (x6): 100n, Capacitor_SMD:C_0402_1005Metric, symbol Device:C_Small
- added R10 (x9): 200K, Resistor_SMD:R_0402_1005Metric, symbol Device:R_Small_US
- added R10 (x3): 100K, Resistor_SMD:R_0402_1005Metric, symbol Device:R_Small_US
- added R10 (x3): 510R, Resistor_SMD:R_0402_1005Metric, symbol Device:R_Small_US
- added R6 (x7): 0R, Resistor_SMD:R_0402_1005Metric, symbol Device:R_Small_US
- added U52, U56, U73: TPS2115ADRBR, Package_SON:VSON-8-1EP_3x3mm_P0.65mm_EP1.65x2.4mm_ThermalVias, symbol ESLGSU_Parts_Lib:TPS2115ADRBR
- added Y1: CSTNE8M00G55A, Crystal:Resonator_SMD_Murata_CSTxExxV-3Pin_3.0x1.1mm, symbol Device:Crystal_GND2_Small
- D10: footprint Diode_SMD:D_SOD-323 -> Diode_THT:D_DO-41_SOD81_P10.16mm_Horizontal
- renumbered J3 to J4, U55 to U51
Connections:
- net BUS_3V3: now also C6.2, R6.2, U52.8 (IN1)
- net BUS_5V: now also C6.2, R6.2, U56.8 (IN1)
- net CAN1_SE: now also R10.1, R10.2
- net GND: now also C6.1, C6.1, C6.1, C6.1, C6.1, C6.1, R10.1, R10.1, R10.2, R10.2, R10.2, R10.2, U52.5 (GND), U52.9 (GND), U56.5 (GND), U56.9 (GND), U73.5 (GND), U73.9 (GND), Y1.2
- net GPIO_nEN: now also R10.1, R10.2
- net I2C1_nPEN: now also R10.1, R10.1
- net SUB3V3: now also R6.1, R6.1, U52.7 (OUT); no longer RN7.1 (R1.1), RN7.2 (R2.1)
- net SUB5V: now also R10.2, R6.1, R6.1, U56.7 (OUT)
- net SYS_3V3: now also C6.2, C6.2, R10.1, R10.1, R10.1, R10.1, R10.1, R10.1, R6.2, R6.2, U52.6 (IN2), U73.8 (IN1)
- net SYS_5V: now also C6.2, C6.2, R6.2, R6.2, U56.6 (IN2), U73.6 (IN2)
- net VBUS: now also RN7.1 (R1.1), RN7.2 (R2.1), R10.2, R10.2, R6.1, R6.1, U73.7 (OUT)
- net at U51.5 (PH0): now also Y1.1
- net at U51.6 (PH1): now also R6.1
- net CFG_LOAD: no longer names the net of U51.3 (PC14)
- net CONFIG_nOE: no longer names the net of U51.4 (PC15)
- net GPIO_A_SHIFT: no longer names the net of U51.16 (PA2)
- net GPIO_A_nEN: no longer names the net of U51.15 (PA1)
- net _CAN1_SE: no longer names the net of U51.21 (PA5)
- net _I2C1_EN: no longer names the net of U51.17 (PA3)
- net _I2C1_nPEN: no longer names the net of U51.20 (PA4)
- net _nVB5V: no longer names the net of U51.27 (PB1)
- net _nVBPWR: no longer names the net of U51.26 (PB0)
- new net: R6.2, Y1.3
- new net: R10.1, U52.4 (ILIM)
- new net: R10.1, U56.4 (ILIM)
- new net: R10.1, U73.4 (ILIM)
- new net nVBUS: R10.2, R10.2, U52.2 (D0), U56.2 (D0)
- new net nVSYS: R10.2, R10.2, U52.3 (D1), U56.3 (D1)
- new net nVT3V3: R10.2, U73.2 (D0)
- new net nVT5V: R10.2, U73.3 (D1)
- no-connect marks 50 -> 45
Other:
- note added: "Subcircuit Power Switches"
- note added: "Transceiver Power"
- note removed: "Bus Power"
- note removed: "Config Latch"
- note removed: "EPS Power Switches"
- note removed: "crystal can be added here"
- moved on the sheet: C25, C29, C6, D1, D10, J4, R10, R6, R8, RN3, U44, U51

Commit message: Last tweaks on schematic
Parts:
- added TP1 (x3): TestPoint, TestPoint:TestPoint_Pad_D1.5mm, symbol Connector:TestPoint
- D10: footprint Diode_THT:D_DO-41_SOD81_P10.16mm_Horizontal -> Diode_SMD:D_SOD-323
- U39: footprint (none) -> ESLGSU_Parts_Lib:UQFN8_MICROPAK
- renumbered U51 to U39
Connections:
- net SUB3V3: now also TP1.1
- net SUB5V: now also TP1.1
- net VBUS: now also TP1.1
