File: ESLGSU_Misc_uCs.kicad_sch (KiCad schematic)
At the start: 71 parts, among them J4 Conn_01x06_Pin, U29 TCAN1051GVDRBRQ, U31 TMUX1574RSVR, U39 FXMA2102L8X, U39 STM32F412RETx, U44 TMUX1574RSVR, U52 TPS2115ADRBR, U56 TPS2115ADRBR, U73 TPS2115ADRBR, Y1 CSTNE8M00G55A

Commit message: Should be done with minimal version
Parts:
- C25, C29, C6, D1, D10, J4, R10, R8, U29, U31, U39, U44, U52, U56, U73: now not fitted; now left out of the parts list

Commit message: Fixed MP28167, debug headers
Parts:
- J4: LCSC Part C2881612 -> C2881573
Changed lines of the file:
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@@
       (effects (font (size 1.27 1.27)) hide)
     )
-    (property "LCSC Part" "C2881612" (at 114.3 146.05 0)
+    (property "LCSC Part" "C2881573" (at 114.3 146.05 0)
       (effects (font (size 1.27 1.27)) hide)
     )

Commit message: Final V1 board with notes
Parts:
- J4: LCSC Part C2881573 -> C2881496
Changed lines of the file:
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@@
       (effects (font (size 1.27 1.27)) hide)
     )
-    (property "LCSC Part" "C2881573" (at 114.3 146.05 0)
+    (property "LCSC Part" "C2881496" (at 114.3 146.05 0)
       (effects (font (size 1.27 1.27)) hide)
     )
