File: ESLGSU_Misc_uCs.kicad_sch (KiCad schematic)
At the start: 71 parts, among them J4 Conn_01x06_Pin, U29 TCAN1051GVDRBRQ, U31 TMUX1574RSVR, U39 FXMA2102L8X, U39 STM32F412RETx, U44 TMUX1574RSVR, U52 TPS2115ADRBR, U56 TPS2115ADRBR, U73 TPS2115ADRBR, Y1 CSTNE8M00G55A

Commit message: Fixed MP28167, debug headers
Parts:
- J4: LCSC Part C2881612 -> C2881573
Changed lines of the file:
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@@
       (effects (font (size 1.27 1.27)) hide)
     )
-    (property "LCSC Part" "C2881612" (at 114.3 146.05 0)
+    (property "LCSC Part" "C2881573" (at 114.3 146.05 0)
       (effects (font (size 1.27 1.27)) hide)
     )

Commit message: Fixes for next version
Parts:
- added R10: 200K, Resistor_SMD:R_0402_1005Metric, symbol Device:R_Small_US
- J4: LCSC Part C2881573 -> C2881496
- R8: value 33R -> 150R; LCSC Part C25105 -> C25082
Connections:
- net SUB3V3: now also R10.1
- net nRST: now also R10.2
Changed lines of the file:
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@@
   (junction (at 246.38 102.87) (diameter 0) (color 0 0 0 0)
   )
+  (junction (at 43.18 27.94) (diameter 0) (color 0 0 0 0)
+  )
   (junction (at 143.51 60.96) (diameter 0) (color 0 0 0 0)
   )
@@
     (stroke (width 0) (type default))
   )
+  (wire (pts (xy 43.18 25.4) (xy 43.18 27.94))
+    (stroke (width 0) (type default))
+  )
   (wire (pts (xy 127 46.99) (xy 127 52.07))
     (stroke (width 0) (type default))
@@
     (stroke (width 0) (type default))
   )
+  (wire (pts (xy 43.18 27.94) (xy 46.99 27.94))
+    (stroke (width 0) (type default))
+  )
   (wire (pts (xy 251.46 40.64) (xy 257.81 40.64))
     (stroke (width 0) (type default))
@@
     (stroke (width 0) (type default))
   )
-  (wire (pts (xy 40.64 27.94) (xy 46.99 27.94))
+  (wire (pts (xy 40.64 27.94) (xy 43.18 27.94))
     (stroke (width 0) (type default))
   )
@@
     (effects (font (size 1.27 1.27)) (justify left bottom))
   )
+  (label "SUB3V3" (at 38.1 25.4 180) (fields_autoplaced)
+    (effects (font (size 1.27 1.27)) (justify right bottom))
+  )
   (label "VBUS" (at 242.57 60.96 180) (fields_autoplaced)
     (effects (font (size 1.27 1.27)) (justify right bottom))
@@
       (effects (font (size 1.27 1.27)) hide)
     )
-    (property "LCSC Part" "C2881573" (at 114.3 146.05 0)
+    (property "LCSC Part" "C2881496" (at 114.3 146.05 0)
       (effects (font (size 1.27 1.27)) hide)
     )
@@
       (effects (font (size 1.27 1.27)) (justify left))
     )
-    (property "Value" "33R" (at 80.01 139.7 0)
+    (property "Value" "150R" (at 80.01 139.7 0)
       (effects (font (size 1.27 1.27)) (justify left))
     )
@@
       (effects (font (size 1.27 1.27)) hide)
     )
-    (property "LCSC Part" "C25105" (at 86.5056 137.1763 90)
+    (property "LCSC Part" "C25082" (at 86.5056 137.1763 90)
       (effects (font (size 1.27 1.27)) hide)
     )
@@
         )
       )
+    )
+  )
+  (symbol (lib_id "Device:R_Small_US") (at 40.64 25.4 90) (mirror x) (unit 1)
+    (in_bom yes) (on_board yes) (dnp no)
+    (property "Reference" "R10" (at 30.5714 23.6763 90)
+      (effects (font (size 1.27 1.27)) (justify left))
+    )
+    (property "Value" "200K" (at 30.48 25.4 90)
+      (effects (font (size 1.27 1.27)) (justify left))
+    )
+    (property "Footprint" "Resistor_SMD:R_0402_1005Metric" (at 40.64 25.4 0)
+      (effects (font (size 1.27 1.27)) hide)
+    )
+    (property "Datasheet" "~" (at 40.64 25.4 0)
+      (effects (font (size 1.27 1.27)) hide)
+    )
+    (property "LCSC Part" "C25764" (at 35.1063 22.7686 0)
+      (effects (font (size 1.27 1.27)) hide)
+    )
+    (pin "1")
+    (pin "2")
+    (instances
+      (project "ESLGSU"
+        (path "/b556fa32-e0cb-409c-ac85-9f2ac606be79/09a64186-e4de-4db7-b903-c6397ff9a54d"
+          (reference "R10") (unit 1)
+        )
+        (path "/b556fa32-e0cb-409c-ac85-9f2ac606be79/62656839-ead6-4c9d-b4ee-68fd3b49c6dd"
+          (reference "R118") (unit 1)
+        )
+        (path "/b556fa32-e0cb-409c-ac85-9f2ac606be79/9412c7fa-2c7e-459e-92bb-96befc1cea15/9d9b9fbb-be95-4e78-92da-55ca1e06a336"
+          (reference "R301") (unit 1)
+        )
+        (path "/b556fa32-e0cb-409c-ac85-9f2ac606be79/9412c7fa-2c7e-459e-92bb-96befc1cea15/2a317018-6d88-41d1-86f4-cb6f86a8c68d"
+          (reference "R300") (unit 1)
+        )
+      )
