File: ESLGSU_EPS_uC.kicad_sch (KiCad schematic)
At the start: 0 parts

Commit message: uC Interface work
Other:
- company: (none) -> Electronic Systems Laboratory
Changed lines of the file:
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@@
 (kicad_sch (version 20230121) (generator eeschema)
   (paper "A4")
+  (title_block
+    (date "2024-01-18")
+    (rev "1")
+    (company "Electronic Systems Laboratory")
+  )
 )

Commit message: Finished interfaces work
Parts:
- added U38: STM32F072VBTx, Package_QFP:LQFP-100_14x14mm_P0.5mm, symbol MCU_ST_STM32F0:STM32F072VBTx
Connections:
- new net: U38.27 (VSS), U38.49 (VSS), U38.74 (VSS), U38.99 (VSS)
Changed lines of the file:
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@@
     (company "Electronic Systems Laboratory")
   )
+  (symbol (lib_id "MCU_ST_STM32F0:STM32F072VBTx") (at 71.12 100.33 0) (unit 1)
+    (in_bom yes) (on_board yes) (dnp no) (fields_autoplaced)
+    (property "Reference" "U38" (at 75.8541 168.91 0)
+      (effects (font (size 1.27 1.27)) (justify left))
+    )
+    (property "Value" "STM32F072VBTx" (at 75.8541 171.45 0)
+      (effects (font (size 1.27 1.27)) (justify left))
+    )
+    (property "Footprint" "Package_QFP:LQFP-100_14x14mm_P0.5mm" (at 55.88 166.37 0)
+      (effects (font (size 1.27 1.27)) (justify right) hide)
+    )
+    (property "Datasheet" "https://www.st.com/resource/en/datasheet/stm32f072vb.pdf" (at 71.12 100.33 0)
+      (effects (font (size 1.27 1.27)) hide)
+    )
+    (pin "1")
+    (pin "10")
+    (pin "100")
+    (pin "11")
+    (pin "12")
+    (pin "13")
+    (pin "14")
+    (pin "15")
+    (pin "16")
+    (pin "17")
+    (pin "18")
+    (pin "19")
+    (pin "2")
+    (pin "20")
+    (pin "21")
+    (pin "22")
+    (pin "23")
+    (pin "24")
+    (pin "25")
+    (pin "26")
+    (pin "27")
+    (pin "28")
+    (pin "29")
+    (pin "3")
+    (pin "30")
+    (pin "31")
+    (pin "32")
+    (pin "33")
+    (pin "34")
+    (pin "35")
+    (pin "36")
+    (pin "37")
+    (pin "38")
+    (pin "39")
+    (pin "4")
+    (pin "40")
+    (pin "41")
+    (pin "42")
+    (pin "43")
+    (pin "44")
+    (pin "45")
+    (pin "46")
+    (pin "47")
+    (pin "48")
+    (pin "49")
+    (pin "5")
+    (pin "50")
+    (pin "51")
+    (pin "52")
+    (pin "53")
+    (pin "54")
+    (pin "55")
+    (pin "56")
+    (pin "57")
+    (pin "58")
+    (pin "59")
+    (pin "6")
+    (pin "60")
+    (pin "61")
+    (pin "62")
+    (pin "63")
+    (pin "64")
+    (pin "65")
+    (pin "66")
+    (pin "67")
+    (pin "68")
+    (pin "69")
+    (pin "7")
+    (pin "70")
+    (pin "71")
+    (pin "72")
+    (pin "73")
+    (pin "74")
+    (pin "75")
+    (pin "76")
+    (pin "77")
+    (pin "78")
+    (pin "79")
+    (pin "8")
+    (pin "80")
+    (pin "81")
+    (pin "82")
+    (pin "83")
+    (pin "84")
+    (pin "85")
+    (pin "86")
+    (pin "87")
+    (pin "88")
+    (pin "89")
+    (pin "9")
+    (pin "90")
+    (pin "91")
+    (pin "92")
+    (pin "93")
+    (pin "94")
+    (pin "95")
+    (pin "96")
+    (pin "97")
+    (pin "98")
+    (pin "99")
+    (instances
+      (project "ESLGSU"
+        (path "/b556fa32-e0cb-409c-ac85-9f2ac606be79/c41d3519-67b9-43b9-97c4-d20822b3d6ca"
+          (reference "U38") (unit 1)
+        )
+      )
+    )
+  )
 )

Commit message: Tried to prepare for order
Parts:
- U38: value STM32F072VBTx -> STM32F072VBT6
Changed lines of the file:
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@@
       (effects (font (size 1.27 1.27)) (justify left))
     )
-    (property "Value" "STM32F072VBTx" (at 75.8541 171.45 0)
+    (property "Value" "STM32F072VBT6" (at 75.8541 171.45 0)
       (effects (font (size 1.27 1.27)) (justify left))
     )

Commit message: Second last bit of schematic work
Parts:
- removed U38: STM32F072VBT6, Package_QFP:LQFP-100_14x14mm_P0.5mm, symbol MCU_ST_STM32F0:STM32F072VBTx
Changed lines of the file:
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@@
 (kicad_sch (version 20230121) (generator eeschema)
-  (paper "A4")
+  (paper "A3")
   (title_block
     (date "2024-01-18")
@@
     (company "Electronic Systems Laboratory")
   )
-  (symbol (lib_id "MCU_ST_STM32F0:STM32F072VBTx") (at 71.12 100.33 0) (unit 1)
-    (in_bom yes) (on_board yes) (dnp no) (fields_autoplaced)
-    (property "Reference" "U38" (at 75.8541 168.91 0)
-      (effects (font (size 1.27 1.27)) (justify left))
-    )
-    (property "Value" "STM32F072VBT6" (at 75.8541 171.45 0)
-      (effects (font (size 1.27 1.27)) (justify left))
-    )
-    (property "Footprint" "Package_QFP:LQFP-100_14x14mm_P0.5mm" (at 55.88 166.37 0)
-      (effects (font (size 1.27 1.27)) (justify right) hide)
-    )
-    (property "Datasheet" "https://www.st.com/resource/en/datasheet/stm32f072vb.pdf" (at 71.12 100.33 0)
-      (effects (font (size 1.27 1.27)) hide)
-    )
-    (pin "1")
-    (pin "10")
-    (pin "100")
-    (pin "11")
-    (pin "12")
-    (pin "13")
-    (pin "14")
-    (pin "15")
-    (pin "16")
-    (pin "17")
-    (pin "18")
-    (pin "19")
-    (pin "2")
-    (pin "20")
-    (pin "21")
-    (pin "22")
-    (pin "23")
-    (pin "24")
-    (pin "25")
-    (pin "26")
-    (pin "27")
-    (pin "28")
-    (pin "29")
-    (pin "3")
-    (pin "30")
-    (pin "31")
-    (pin "32")
-    (pin "33")
-    (pin "34")
-    (pin "35")
-    (pin "36")
-    (pin "37")
-    (pin "38")
-    (pin "39")
-    (pin "4")
-    (pin "40")
-    (pin "41")
-    (pin "42")
-    (pin "43")
-    (pin "44")
-    (pin "45")
-    (pin "46")
-    (pin "47")
-    (pin "48")
-    (pin "49")
-    (pin "5")
-    (pin "50")
-    (pin "51")
-    (pin "52")
-    (pin "53")
-    (pin "54")
-    (pin "55")
-    (pin "56")
-    (pin "57")
-    (pin "58")
-    (pin "59")
-    (pin "6")
-    (pin "60")
-    (pin "61")
-    (pin "62")
-    (pin "63")
-    (pin "64")
-    (pin "65")
-    (pin "66")
-    (pin "67")
-    (pin "68")
-    (pin "69")
-    (pin "7")
-    (pin "70")
-    (pin "71")
-    (pin "72")
-    (pin "73")
-    (pin "74")
-    (pin "75")
-    (pin "76")
-    (pin "77")
-    (pin "78")
-    (pin "79")
-    (pin "8")
-    (pin "80")
-    (pin "81")
-    (pin "82")
-    (pin "83")
-    (pin "84")
-    (pin "85")
-    (pin "86")
-    (pin "87")
-    (pin "88")
-    (pin "89")
-    (pin "9")
-    (pin "90")
-    (pin "91")
-    (pin "92")
-    (pin "93")
-    (pin "94")
-    (pin "95")
-    (pin "96")
-    (pin "97")
-    (pin "98")
-    (pin "99")
-    (instances
-      (project "ESLGSU"
-        (path "/b556fa32-e0cb-409c-ac85-9f2ac606be79/c41d3519-67b9-43b9-97c4-d20822b3d6ca"
-          (reference "U38") (unit 1)
-        )
-      )
-    )
-  )
 )

Commit message: Final schematic work, added battery charger, linked everything up
Parts:
- added C25 (x14), C6 (x16): 100n, Capacitor_SMD:C_0402_1005Metric, symbol Device:C_Small
- added C29 (x2): 1u, Capacitor_SMD:C_0402_1005Metric, symbol Device:C_Small
- added C29 (x2): 2.2u, Capacitor_SMD:C_0402_1005Metric, symbol Device:C_Small
- added C29: 4.7u, Capacitor_SMD:C_0402_1005Metric, symbol Device:C_Small
- added C6: 100p, Capacitor_SMD:C_0402_1005Metric, symbol Device:C_Small
- added D1: TZ-P2-0603GTCS1-0.6T, LED_SMD:LED_0603_1608Metric, symbol Device:LED
- added D10: 1N5819, Diode_THT:D_DO-41_SOD81_P10.16mm_Horizontal, symbol Diode:1N5819
- added J4: Conn_01x06_Pin, Connector_PinHeader_1.27mm:PinHeader_1x06_P1.27mm_Vertical_SMD_Pin1Right, symbol Connector:Conn_01x06_Pin
- added J7: 10118194-0001LF, ESLGSU_Parts_Lib:AMPHENOL_10118194-0001LF, symbol Connector:USB_B_Micro
- added R10 (x15): 200K, Resistor_SMD:R_0402_1005Metric, symbol Device:R_Small_US
- added R10 (x2): 120R, Resistor_SMD:R_0805_2012Metric, symbol Device:R_Small_US
- added R10 (x7): 10K, Resistor_SMD:R_0402_1005Metric, symbol Device:R_Small_US
- added R10 (x5): 100K, Resistor_SMD:R_0402_1005Metric, symbol Device:R_Small_US
- added R10 (x3): 510R, Resistor_SMD:R_0402_1005Metric, symbol Device:R_Small_US
- added R6 (x7): 0R, Resistor_SMD:R_0402_1005Metric, symbol Device:R_Small_US
- added R8: 33R, Resistor_SMD:R_0402_1005Metric, symbol Device:R_Small_US
- added RN1, RN3, RN4: 0R, Resistor_SMD:R_Array_Concave_4x0402, symbol Device:R_Pack04
- added RN2, RN5, RN6 (x2): 0R, Resistor_SMD:R_Array_Convex_2x0402, symbol Device:R_Pack02
- added RN7: 10K, Resistor_SMD:R_Array_Convex_2x0402, symbol Device:R_Pack02
- added U29: TCAN1051GVDRBRQ, Package_DFN_QFN:DFN-8-1EP_3x3mm_P0.65mm_EP1.55x2.4mm, symbol ESLGSU_Parts_Lib:TCAN1051GVDRBRQ1
- added U30: THVD1450DRBR, Package_DFN_QFN:DFN-8-1EP_3x3mm_P0.65mm_EP1.55x2.4mm, symbol ESLGSU_Parts_Lib:THVD1450
- added U31, U32, U34, U44, U47: TMUX1574RSVR, ESLGSU_Parts_Lib:T-UQFN-16, symbol ESLGSU_Parts_Lib:TMUX1574RSVR
- added U33, U35: TXU0202DTTR, ESLGSU_Parts_Lib:SOT833-1-XSON8, symbol ESLGSU_Parts_Lib:TXU0202-Q1
- added U37: STM32H743ZITx, Package_QFP:LQFP-144_20x20mm_P0.5mm, symbol MCU_ST_STM32H7:STM32H743ZITx
- added U39: FXMA2102L8X, symbol ESLGSU_Parts_Lib:FXMA2102L8X
- added U46: TXB0104RUT, ESLGSU_Parts_Lib:T-UQFN-12, symbol ESLGSU_Parts_Lib:TXB0104RUTR
- added U52, U56, U73: TPS2115ADRBR, Package_SON:VSON-8-1EP_3x3mm_P0.65mm_EP1.65x2.4mm_ThermalVias, symbol ESLGSU_Parts_Lib:TPS2115ADRBR
- added U57: CY8C9520A, Package_SO:SSOP-28_5.3x10.2mm_P0.65mm, symbol ESLGSU_Parts_Lib:CY8C9520A
- added U74: PCAL6524HEAZ, Package_DFN_QFN:HVQFN-32-1EP_5x5mm_P0.5mm_EP3.1x3.1mm, symbol ESLGSU_Parts_Lib:PCAL6524
- added U81: ESD7004MUTAG, symbol ESLGSU_Parts_Lib:ESD7004MUTAG
- added Y1: CSTNE8M00G55A, Crystal:Resonator_SMD_Murata_CSTxExxV-3Pin_3.0x1.1mm, symbol Device:Crystal_GND2_Small
Connections:
- new net: R6.1, U37.24 (PH1)
- new net: R6.2, Y1.3
- new net: RN5.1 (R1.1), U30.1 (R), U33.1 (B2)
- new net: RN5.2 (R2.1), U30.4 (D), U33.8 (B1Y)
- new net: C6.2, R10.2, U39.8 (VREF2)
- new net: D10.2 (A), J4.1 (Pin_1)
- new net: R10.1, U52.4 (ILIM)
- new net: D1.2 (A), R8.2
- new net: R6.2, U37.76 (PB15)
- new net: C29.1, U37.106 (VCAP)
- new net: R10.1, U73.4 (ILIM)
- new net: R10.2, U74.28 (nRST)
- new net: U46.10 (B1), U47.1 (S1B)
- new net: U46.7 (B4), U47.11 (S4B)
- new net: U46.8 (B3), U47.8 (S3B)
- new net: U46.9 (B2), U47.4 (S2B)
- new net: R10.1, U56.4 (ILIM)
- new net: U37.23 (PH0), Y1.1
- new net: R10.1, U31.16 (S1A)
- new net: R10.1, U31.3 (S2A)
- new net: R6.2, U37.75 (PB14)
- new net: C29.1, U37.71 (VCAP)
- new net: U32.1 (S1B), U32.3 (S2A), U35.1 (B2)
- new net: U32.16 (S1A), U32.4 (S2B), U35.8 (B1Y)
- new net BOOTLDR: R10.2, U37.138 (BOOT0)
- new net CAN1_H: R10.1, U29.7 (CANH)
- new net CAN1_L: R10.2, U29.6 (CANL)
- new net CAN1_RX: U29.4 (RXD), U37.139 (PB8)
- new net CAN1_SE: R10.1, R10.2, U29.8 (S), U57.1 (P0_0), U74.1 (P0_0)
- new net CAN1_TX: U29.1 (TXD), U37.140 (PB9)
- new net CFGI2C_SCL: RN6.1 (R1.1), U57.10 (SCL), U74.29 (SCL)
- new net CFGI2C_SDA: RN6.2 (R2.1), U57.11 (SDA), U74.26 (ADDR), U74.30 (SDA)
- new net EPS_I2C_INT: U37.80 (PD11)
- new net EPS_I2C_SCL: R10.2, RN6.4 (R1.2), U37.81 (PD12)
- new net EPS_I2C_SDA: R10.2, RN6.3 (R2.2), U37.82 (PD13)
- new net GND: C25.2, C25.2, C25.2, C25.2, C25.2, C25.2, C25.2, C25.2, C25.2, C25.2, C25.2, C25.2, C25.2, C25.2, C29.2, C29.2, C29.2, C29.2, C29.2, C6.1, C6.1, C6.1, C6.1, C6.1, C6.1, C6.1, C6.1, C6.1, C6.1, C6.1, C6.1, C6.1, C6.1, C6.1, C6.1, C6.2, D1.1 (K), J4.6 (Pin_6), J7.5 (GND), J7.S1 (S), J7.S2 (S), J7.S3 (S), J7.S4 (S), J7.S5 (S), J7.S6 (S), R10.1, R10.1, R10.1, R10.1, R10.1, R10.1, R10.2, R10.2, R10.2, R10.2, R10.2, R10.2, U29.2 (GND), U29.9 (GND), U30.5 (GND), U30.9 (GND), U31.15 (SEL), U31.6 (GND), U32.6 (GND), U33.2 (GND), U34.15 (SEL), U34.6 (GND), U35.2 (GND), U37.107 (VSS), U37.120 (VSS), U37.130 (VSS), U37.143 (PDR_ON), U37.16 (VSS), U37.31 (VSSA), U37.38 (VSS), U37.51 (VSS), U37.61 (VSS), U37.83 (VSS), U37.94 (VSS), U39.4 (GND), U44.15 (SEL), U44.6 (GND), U46.6 (GND), U47.6 (GND), U52.5 (GND), U52.9 (GND), U56.5 (GND), U56.9 (GND), U57.14 (GND), U57.9 (GND), U73.5 (GND), U73.9 (GND), U74.25 (GND), U81.3 (GND), U81.8 (GND), Y1.2
- new net GPIO_1: RN3.4 (R4.1), U44.2 (D1)
- new net GPIO_2: RN3.3 (R3.1), U44.5 (D2)
- new net GPIO_3: RN3.2 (R2.1), U44.7 (D3)
- new net GPIO_4: RN3.1 (R1.1), U44.10 (D4)
- new net GPIO_5: RN4.4 (R4.1), U34.2 (D1)
- new net GPIO_6: RN4.3 (R3.1), U34.5 (D2)
- new net GPIO_7: RN4.2 (R2.1), U34.7 (D3)
- new net GPIO_8: RN4.1 (R1.1), U34.10 (D4)
- new net GPIO_nEN: R10.1, R10.2, U34.13 (nEN), U44.13 (nEN), U57.12 (P2_3_A1), U74.19 (P2_2)
- new net I2C1_EN: R10.1, U39.5 (OE), U57.3 (P0_2), U74.3 (P0_2)
- new net I2C1_SCL: R10.2, RN6.2 (R2.1), RN7.3 (R2.2), U39.7 (SCL2)
- new net I2C1_SDA: R10.2, RN6.1 (R1.1), RN7.4 (R1.2), U39.6 (SDA2)
- new net I2C1_nPEN: R10.1, R10.1, U31.13 (nEN), U57.4 (P0_3), U74.4 (P0_3)
- new net LED: R8.1, U37.34 (PA0)
- new net PISER_RX: R6.1
- new net PISER_TX: R6.1
- new net PISPI_MISO: U37.42 (PA6)
- new net PISPI_MOSI: U37.43 (PA7)
- new net PISPI_NSS: U37.40 (PA4)
- new net PISPI_SCK: U37.41 (PA5)
- new net RAW_BAT_BUS: U57.22 (P1_5_A6), U74.14 (P1_5)
- new net RAW_PIN_BAT: U74.15 (P1_6)
- new net RAW_PIN_BUS: U57.23 (P1_4)
- new net REG_3V3_EF: U57.27 (P1_0), U74.9 (P1_0)
- new net REG_3V3_EN: U37.87 (PG2)
- new net REG_5V_EF: U57.26 (P1_1), U74.10 (P1_1)
- new net REG_5V_EN: U37.88 (PG3)
- new net REG_CH1_EF: U57.25 (P1_2), U74.11 (P1_2)
- new net REG_CH1_EN: U37.89 (PG4)
- new net REG_CH2_EF: U57.24 (P1_3), U74.12 (P1_3)
- new net REG_CH2_EN: U37.90 (PG5)
- new net RS4851_A: R10.2, U30.6 (A)
- new net RS4851_B: R10.1, U30.7 (B)
- new net RS4851_EN: R10.1, R10.2, U30.2 (nRE), U30.3 (DE), U57.2 (P0_1), U74.2 (P0_1)
- new net RS4851_RX: RN5.4 (R1.2), U33.4 (A2Y), U37.114 (PD0)
- new net RS4851_TX: RN5.3 (R2.2), U33.5 (A1), U37.115 (PD1)
- new net RS4851_TXE: R10.1, U37.118 (PD4)
- new net SPI1_MISO: RN1.1 (R1.1), U47.10 (D4)
- new net SPI1_MOSI: RN1.4 (R4.1), U47.2 (D1)
- new net SPI1_NSS: RN1.2 (R2.1), U47.7 (D3)
- new net SPI1_SCK: RN1.3 (R3.1), U47.5 (D2)
- new net SPI1_nEN: R10.1, R10.2, U47.13 (nEN), U57.7 (P0_6), U74.7 (P0_6)
- new net SPI_SHIFT: U46.12 (OE), U47.15 (SEL), U57.8 (P0_7), U74.8 (P0_7)
- new net SUB3V3: C25.1, C25.1, C25.1, C25.1, C25.1, C25.1, C25.1, C25.1, C25.1, C25.1, C25.1, C25.1, C25.1, C25.1, C29.1, C29.1, C29.1, C6.2, C6.2, C6.2, C6.2, D10.1 (K), R10.1, R10.1, R10.1, R10.1, R6.1, U29.5 (VIO), U33.3 (VCCA), U33.6 (OE), U35.3 (VCCA), U35.6 (OE), U37.108 (VDD), U37.121 (VDD), U37.131 (VDD), U37.144 (VDD), U37.17 (VDD), U37.30 (VDD), U37.32 (VREF+), U37.33 (VDDA), U37.39 (VDD), U37.52 (VDD), U37.6 (VBAT), U37.62 (VDD), U37.72 (VDD), U37.84 (VDD), U37.95 (VDD33_USB), U39.1 (VREF1), U46.1 (VCCA), U52.7 (OUT)
- new net SUB5V: C6.2, R10.2, R6.1, U29.3 (VCC), U56.7 (OUT)
- new net SWCLK: J4.4 (Pin_4), U37.109 (PA14)
- new net SWDIO: J4.3 (Pin_3), U37.105 (PA13)
- new net SWO: J4.5 (Pin_5), U37.133 (PB3)
- new net SYS_3V3: C6.2, C6.2, C6.2, R10.1, R10.1, R10.1, R10.1, R10.1, R6.2, R6.2, U52.3 (D1), U52.8 (IN1), U56.3 (D1), U57.13 (A0), U57.28 (VDD), U73.8 (IN1), U74.27 (VDDP), U74.31 (VDDI)
- new net SYS_5V: C6.2, C6.2, R6.2, R6.2, U56.8 (IN1), U73.6 (IN2)
- new net UART1_REV: R10.2, U32.15 (SEL), U57.6 (P0_5), U74.6 (P0_5)
- new net UART1_RX: RN2.1 (R1.1), U32.5 (D2)
- new net UART1_TX: RN2.2 (R2.1), U32.2 (D1)
- new net UART1_nEN: R10.1, R10.2, U32.13 (nEN), U57.5 (P0_4), U74.5 (P0_4)
- new net USB_D+: J7.3 (D+), U37.104 (PA12), U81.4 (IO3), U81.7 (NC3)
- new net USB_D-: J7.2 (D-), U37.103 (PA11), U81.2 (IO2), U81.9 (NC2)
- new net USB_ID: J7.4 (ID), U37.102 (PA10), U81.5 (IO4), U81.6 (NC4)
- new net USB_VBUS: J7.1 (VBUS), U37.101 (PA9), U81.1 (IO1), U81.10 (NC1)
- new net VBUS: C6.1, C6.2, C6.2, C6.2, C6.2, C6.2, R10.1, R10.2, R10.2, R10.2, R10.2, R6.1, R6.1, RN7.1 (R1.1), RN7.2 (R2.1), U30.8 (VCC), U31.14 (VDD), U31.2 (D1), U31.5 (D2), U32.14 (VDD), U33.7 (VCCB), U34.14 (VDD), U35.7 (VCCB), U44.14 (VDD), U46.11 (VCCB), U47.14 (VDD), U73.7 (OUT)
- new net _GPIO_1: RN3.5 (R4.2), U37.12 (PF2), U44.16 (S1A)
- new net _GPIO_2: RN3.6 (R3.2), U37.13 (PF3), U44.3 (S2A)
- new net _GPIO_3: RN3.7 (R2.2), U37.14 (PF4), U44.9 (S3A)
- new net _GPIO_4: RN3.8 (R1.2), U37.15 (PF5), U44.12 (S4A)
- new net _GPIO_5: RN4.5 (R4.2), U34.16 (S1A), U37.18 (PF6)
- new net _GPIO_6: RN4.6 (R3.2), U34.3 (S2A), U37.19 (PF7)
- new net _GPIO_7: RN4.7 (R2.2), U34.9 (S3A), U37.20 (PF8)
- new net _GPIO_8: RN4.8 (R1.2), U34.12 (S4A), U37.21 (PF9)
- new net _I2C1_SCL: R10.2, RN6.3 (R2.2), U37.136 (PB6), U39.2 (SCL1)
- new net _I2C1_SDA: R10.2, RN6.4 (R1.2), U37.137 (PB7), U39.3 (SDA1)
- new net _SPI1_MISO: RN1.8 (R1.2), U37.112 (PC11), U46.5 (A4), U47.12 (S4A)
- new net _SPI1_MOSI: RN1.5 (R4.2), U37.113 (PC12), U46.2 (A1), U47.16 (S1A)
- new net _SPI1_NSS: RN1.7 (R2.2), U37.110 (PA15), U46.4 (A3), U47.9 (S3A)
- new net _SPI1_SCK: RN1.6 (R3.2), U37.111 (PC10), U46.3 (A2), U47.3 (S2A)
- new net _UART1_RX: RN2.4 (R1.2), U35.4 (A2Y), U37.37 (PA3)
- new net _UART1_TX: RN2.3 (R2.2), U35.5 (A1), U37.36 (PA2)
- new net nRST: J4.2 (Pin_2), U37.25 (NRST)
- new net nVSYS: R10.2, R10.2, U52.2 (D0), U56.2 (D0), U57.15 (P2_2_WD), U74.20 (P2_3)
- new net nVT3V3: R10.2, U57.18 (P2_0_A3), U73.2 (D0), U74.17 (P2_0)
- new net nVT5V: R10.2, U57.17 (P2_1_A2), U73.3 (D1), U74.18 (P2_1)
- no-connect marks 0 -> 108
Other:
- note added: "Addr: 0100001"
- note added: "Addr: 0100001 1010001"
- note added: "CAN Transceiver"
- note added: "CFG I2C Bridge"
- note added: "Config Expander Options"
- note added: "Debug Header"
- note added: "Decoupling Capacitors"
- note added: "GPIO Transceiver"
- note added: "I2C Transceiver"
- note added: "Indicator LED"
- note added: "Microcontroller"
- note added: "RS485 Transceiver"
- note added: "SPI Transceiver"
- note added: "Subcircuit Power Switches"
- note added: "Transceiver Power"
- note added: "UART Transceiver"
- note added: "USB Port"
- note added: "VDDA: 1u, 100u VDD: 4.7u, 11x100n VREF: 1u, 100u VUSB: 100n"

Commit message: Last tweaks on schematic
Parts:
- added TP1 (x3): TestPoint, TestPoint:TestPoint_Pad_D1.5mm, symbol Connector:TestPoint
- D10: footprint Diode_THT:D_DO-41_SOD81_P10.16mm_Horizontal -> Diode_SMD:D_SOD-323
- U39: footprint (none) -> ESLGSU_Parts_Lib:UQFN8_MICROPAK
- U81: footprint (none) -> ESLGSU_Parts_Lib:UDFN10_ESD
- renumbered Y1 to Y4
Connections:
- net SUB3V3: now also TP1.1
- net SUB5V: now also TP1.1
- net VBUS: now also TP1.1

Commit message: Some PCB work
Connections:
- net GPIO_nEN: now also U74.20 (P2_3); no longer U74.19 (P2_2)
- net RAW_PIN_BUS: now also U74.13 (P1_4)
- net nVSYS: now also U74.19 (P2_2); no longer U74.20 (P2_3)
- net RAW_PIN_BAT: no longer names the net of U74.15 (P1_6)
Changed lines of the file:
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@@
   (no_connect (at 40.64 128.27))
   (no_connect (at 62.23 41.91))
+  (no_connect (at 185.42 104.14))
   (no_connect (at 182.88 81.28))
   (no_connect (at 386.08 171.45))
@@
   (no_connect (at 104.14 156.21))
   (no_connect (at 386.08 173.99))
-  (no_connect (at 185.42 109.22))
   (no_connect (at 40.64 219.71))
   (no_connect (at 40.64 222.25))
@@
     (stroke (width 0) (type default))
   )
-  (wire (pts (xy 185.42 109.22) (xy 182.88 109.22))
-    (stroke (width 0) (type default))
-  )
   (wire (pts (xy 212.09 154.94) (xy 209.55 154.94))
     (stroke (width 0) (type default))
@@
   )
   (wire (pts (xy 350.52 240.03) (xy 365.76 240.03))
+    (stroke (width 0) (type default))
+  )
+  (wire (pts (xy 182.88 109.22) (xy 185.42 109.22))
     (stroke (width 0) (type default))
   )
@@
     (effects (font (size 1.27 1.27)) (justify right bottom))
   )
+  (label "nVSYS" (at 185.42 93.98 0) (fields_autoplaced)
+    (effects (font (size 1.27 1.27)) (justify left bottom))
+  )
   (label "SUB5V" (at 378.46 16.51 0) (fields_autoplaced)
     (effects (font (size 1.27 1.27)) (justify left bottom))
@@
     (effects (font (size 1.27 1.27)) (justify right bottom))
   )
-  (label "nVSYS" (at 185.42 91.44 0) (fields_autoplaced)
-    (effects (font (size 1.27 1.27)) (justify left bottom))
-  )
   (label "VBUS" (at 67.31 54.61 0) (fields_autoplaced)
     (effects (font (size 1.27 1.27)) (justify left bottom))
@@
     (effects (font (size 1.27 1.27)) (justify right bottom))
   )
+  (label "GPIO_nEN" (at 185.42 91.44 0) (fields_autoplaced)
+    (effects (font (size 1.27 1.27)) (justify left bottom))
+  )
   (label "_GPIO_1" (at 60.96 26.67 180) (fields_autoplaced)
     (effects (font (size 1.27 1.27)) (justify right bottom))
@@
     (effects (font (size 1.27 1.27)) (justify left bottom))
   )
-  (label "GPIO_nEN" (at 185.42 93.98 0) (fields_autoplaced)
-    (effects (font (size 1.27 1.27)) (justify left bottom))
-  )
   (label "I2C1_nPEN" (at 392.43 92.71 180) (fields_autoplaced)
     (effects (font (size 1.27 1.27)) (justify right bottom))
@@
     (effects (font (size 1.27 1.27)) (justify left))
   )
+  (hierarchical_label "RAW_PIN_BUS" (shape output) (at 185.42 109.22 0) (fields_autoplaced)
+    (effects (font (size 1.27 1.27)) (justify left))
+  )
   (hierarchical_label "I2C1_SDA" (shape bidirectional) (at 392.43 130.81 0) (fields_autoplaced)
     (effects (font (size 1.27 1.27)) (justify left))
@@
     (effects (font (size 1.27 1.27)) (justify right))
   )
-  (hierarchical_label "RAW_PIN_BAT" (shape output) (at 185.42 104.14 0) (fields_autoplaced)
-    (effects (font (size 1.27 1.27)) (justify left))
-  )
   (hierarchical_label "PISPI_MOSI" (shape input) (at 106.68 120.65 0) (fields_autoplaced)
