File: ESLGSU_EPS_uC.kicad_sch (KiCad schematic)
At the start: 111 parts, among them J4 Conn_01x06_Pin, J7 10118194-0001LF, U29 TCAN1051GVDRBRQ, U30 THVD1450DRBR, U31 TMUX1574RSVR, U32 TMUX1574RSVR, U33 TXU0202DTTR, U34 TMUX1574RSVR, U35 TXU0202DTTR, U37 STM32H743ZITx, U39 FXMA2102L8X, U44 TMUX1574RSVR, U46 TXB0104RUT, U47 TMUX1574RSVR, U52 TPS2115ADRBR, U56 TPS2115ADRBR, U57 CY8C9520A, U73 TPS2115ADRBR, U74 PCAL6524HEAZ, U81 ESD7004MUTAG, Y4 CSTNE8M00G55A

Commit message: Hopefully final full PCB version
Parts:
- removed RN7: 10K, Resistor_SMD:R_Array_Convex_2x0402, symbol Device:R_Pack02
- added R10 (x2): 10K, Resistor_SMD:R_0402_1005Metric, symbol Device:R_Small_US
Connections:
- net I2C1_SCL: now also R10.1
- net I2C1_SDA: now also R10.1
- net VBUS: now also R10.2, R10.2
- net EN_3V3_S1: now reaches U37.124 (PG9)
- net EN_3V3_S2: now reaches U37.125 (PG10)
- net EN_5V_S1: now reaches U37.126 (PG11)
- net EN_5V_S2: now reaches U37.127 (PG12)
- no-connect marks 108 -> 104
Changed lines of the file:
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@@
   (no_connect (at 104.14 105.41))
   (no_connect (at 392.43 115.57))
-  (no_connect (at 40.64 153.67))
   (no_connect (at 104.14 212.09))
   (no_connect (at 368.3 168.91))
@@
   (no_connect (at 62.23 46.99))
   (no_connect (at 40.64 209.55))
-  (no_connect (at 40.64 148.59))
   (no_connect (at 104.14 245.11))
+  (no_connect (at 40.64 148.59))
   (no_connect (at 40.64 163.83))
   (no_connect (at 198.12 234.95))
   (no_connect (at 190.5 257.81))
-  (no_connect (at 40.64 158.75))
-  (no_connect (at 40.64 156.21))
   (no_connect (at 167.64 58.42))
   (no_connect (at 104.14 173.99))
@@
   (no_connect (at 104.14 224.79))
   (no_connect (at 387.35 97.79))
-  (no_connect (at 40.64 151.13))
   (no_connect (at 104.14 151.13))
   (no_connect (at 104.14 199.39))
@@
     (stroke (width 0) (type default))
   )
+  (wire (pts (xy 38.1 151.13) (xy 40.64 151.13))
+    (stroke (width 0) (type default))
+  )
   (wire (pts (xy 336.55 130.81) (xy 339.09 130.81))
     (stroke (width 0) (type default))
@@
     (stroke (width 0) (type default))
   )
+  (wire (pts (xy 38.1 153.67) (xy 40.64 153.67))
+    (stroke (width 0) (type default))
+  )
   (wire (pts (xy 71.12 95.25) (xy 73.66 95.25))
     (stroke (width 0) (type default))
@@
     (stroke (width 0) (type default))
   )
-  (wire (pts (xy 392.43 138.43) (xy 394.97 138.43))
+  (wire (pts (xy 389.89 138.43) (xy 394.97 138.43))
     (stroke (width 0) (type default))
   )
@@
     (stroke (width 0) (type default))
   )
-  (wire (pts (xy 379.73 138.43) (xy 382.27 138.43))
+  (wire (pts (xy 379.73 138.43) (xy 384.81 138.43))
     (stroke (width 0) (type default))
   )
@@
     (stroke (width 0) (type default))
   )
+  (wire (pts (xy 38.1 156.21) (xy 40.64 156.21))
+    (stroke (width 0) (type default))
+  )
   (wire (pts (xy 341.63 186.69) (xy 342.9 186.69))
     (stroke (width 0) (type default))
@@
     (stroke (width 0) (type default))
   )
+  (wire (pts (xy 38.1 158.75) (xy 40.64 158.75))
+    (stroke (width 0) (type default))
+  )
   (wire (pts (xy 82.55 31.75) (xy 80.01 31.75))
     (stroke (width 0) (type default))
@@
     (stroke (width 0) (type default))
   )
-  (wire (pts (xy 392.43 135.89) (xy 394.97 135.89))
+  (wire (pts (xy 389.89 135.89) (xy 394.97 135.89))
     (stroke (width 0) (type default))
   )
@@
     (stroke (width 0) (type default))
   )
-  (wire (pts (xy 377.19 135.89) (xy 382.27 135.89))
+  (wire (pts (xy 377.19 135.89) (xy 384.81 135.89))
     (stroke (width 0) (type default))
   )
@@
     (effects (font (size 1.27 1.27)) (justify right))
   )
+  (hierarchical_label "EN_5V_S2" (shape output) (at 38.1 158.75 180) (fields_autoplaced)
+    (effects (font (size 1.27 1.27)) (justify right))
+  )
   (hierarchical_label "SPI1_NSS" (shape bidirectional) (at 384.81 227.33 0) (fields_autoplaced)
     (effects (font (size 1.27 1.27)) (justify left))
@@
     (effects (font (size 1.27 1.27)) (justify right))
   )
+  (hierarchical_label "EN_5V_S1" (shape output) (at 38.1 156.21 180) (fields_autoplaced)
+    (effects (font (size 1.27 1.27)) (justify right))
+  )
   (hierarchical_label "GPIO_4" (shape bidirectional) (at 82.55 36.83 0) (fields_autoplaced)
     (effects (font (size 1.27 1.27)) (justify left))
@@
     (effects (font (size 1.27 1.27)) (justify right))
   )
+  (hierarchical_label "EN_3V3_S2" (shape output) (at 38.1 153.67 180) (fields_autoplaced)
+    (effects (font (size 1.27 1.27)) (justify right))
+  )
   (hierarchical_label "PISPI_SCK" (shape input) (at 106.68 115.57 0) (fields_autoplaced)
     (effects (font (size 1.27 1.27)) (justify left))
@@
     (effects (font (size 1.27 1.27)) (justify left))
   )
+  (hierarchical_label "EN_3V3_S1" (shape output) (at 38.1 151.13 180) (fields_autoplaced)
+    (effects (font (size 1.27 1.27)) (justify right))
+  )
   (hierarchical_label "CFGI2C_SDA" (shape bidirectional) (at 161.29 55.88 180) (fields_autoplaced)
     (effects (font (size 1.27 1.27)) (justify right))
@@
     )
   )
-  (symbol (lib_id "Device:R_Small_US") (at 355.6 41.91 0) (mirror x) (unit 1)
-    (in_bom yes) (on_board yes) (dnp no)
-    (property "Reference" "R10" (at 349.25 41.91 0)
+  (symbol (lib_id "Device:R_Small_US") (at 387.35 135.89 90) (unit 1)
+    (in_bom no) (on_board yes) (dnp yes)
+    (property "Reference" "R10" (at 386.08 134.62 0)
       (effects (font (size 1.27 1.27)) (justify left))
     )
-    (property "Value" "200K" (at 349.1586 43.6337 0)
+    (property "Value" "10K" (at 388.62 134.62 0)
       (effects (font (size 1.27 1.27)) (justify left))
     )
-    (property "Footprint" "Resistor_SMD:R_0402_1005Metric" (at 355.6 41.91 0)
+    (property "Footprint" "Resistor_SMD:R_0402_1005Metric" (at 387.35 135.89 0)
       (effects (font (size 1.27 1.27)) hide)
     )
-    (property "Datasheet" "~" (at 355.6 41.91 0)
+    (property "Datasheet" "~" (at 387.35 135.89 0)
       (effects (font (size 1.27 1.27)) hide)
     )
-    (property "LCSC Part" "C25764" (at 352.9686 47.4437 0)
+    (property "LCSC Part" "C25744" (at 388.62 134.62 0)
       (effects (font (size 1.27 1.27)) hide)
     )
@@
         )
         (path "/b556fa32-e0cb-409c-ac85-9f2ac606be79/62656839-ead6-4c9d-b4ee-68fd3b49c6dd"
-          (reference "R118") (unit 1)
+          (reference "R12") (unit 1)
         )
         (path "/b556fa32-e0cb-409c-ac85-9f2ac606be79/c41d3519-67b9-43b9-97c4-d20822b3d6ca"
-          (reference "R236") (unit 1)
+          (reference "R279") (unit 1)
         )
       )
     )
   )
-  (symbol (lib_id "Device:R_Pack02") (at 387.35 135.89 90) (unit 1)
+  (symbol (lib_id "Device:R_Small_US") (at 387.35 138.43 90) (unit 1)
     (in_bom no) (on_board yes) (dnp yes)
-    (property "Reference" "RN7" (at 394.97 139.7 90)
-      (effects (font (size 1.27 1.27)))
+    (property "Reference" "R10" (at 386.08 143.51 0)
+      (effects (font (size 1.27 1.27)) (justify left))
     )
-    (property "Value" "10K" (at 394.97 142.24 90)
-      (effects (font (size 1.27 1.27)))
+    (property "Value" "10K" (at 388.62 143.51 0)
+      (effects (font (size 1.27 1.27)) (justify left))
     )
-    (property "Footprint" "Resistor_SMD:R_Array_Convex_2x0402" (at 387.35 131.445 90)
+    (property "Footprint" "Resistor_SMD:R_0402_1005Metric" (at 387.35 138.43 0)
       (effects (font (size 1.27 1.27)) hide)
     )
-    (property "Datasheet" "~" (at 387.35 135.89 0)
+    (property "Datasheet" "~" (at 387.35 138.43 0)
       (effects (font (size 1.27 1.27)) hide)
     )
-    (property "LCSC Part" "C695179" (at 394.97 142.24 90)
+    (property "LCSC Part" "C25744" (at 388.62 137.16 0)
       (effects (font (size 1.27 1.27)) hide)
     )
-    (property "JLCPCB BOM" "0" (at 387.35 135.89 90)
+    (pin "1")
+    (pin "2")
+    (instances
+      (project "ESLGSU"
+        (path "/b556fa32-e0cb-409c-ac85-9f2ac606be79/09a64186-e4de-4db7-b903-c6397ff9a54d"
+          (reference "R10") (unit 1)
+        )
+        (path "/b556fa32-e0cb-409c-ac85-9f2ac606be79/62656839-ead6-4c9d-b4ee-68fd3b49c6dd"
+          (reference "R8") (unit 1)
+        )
+        (path "/b556fa32-e0cb-409c-ac85-9f2ac606be79/c41d3519-67b9-43b9-97c4-d20822b3d6ca"
+          (reference "R280") (unit 1)
+        )
+      )
+    )
+  )
+  (symbol (lib_id "Device:R_Small_US") (at 355.6 41.91 0) (mirror x) (unit 1)
+    (in_bom yes) (on_board yes) (dnp no)
+    (property "Reference" "R10" (at 349.25 41.91 0)
+      (effects (font (size 1.27 1.27)) (justify left))
+    )
+    (property "Value" "200K" (at 349.1586 43.6337 0)
+      (effects (font (size 1.27 1.27)) (justify left))
+    )
+    (property "Footprint" "Resistor_SMD:R_0402_1005Metric" (at 355.6 41.91 0)
+      (effects (font (size 1.27 1.27)) hide)
+    )
+    (property "Datasheet" "~" (at 355.6 41.91 0)
+      (effects (font (size 1.27 1.27)) hide)
+    )
+    (property "LCSC Part" "C25764" (at 352.9686 47.4437 0)
       (effects (font (size 1.27 1.27)) hide)
     )
     (pin "1")
     (pin "2")
-    (pin "3")
-    (pin "4")
     (instances
       (project "ESLGSU"
+        (path "/b556fa32-e0cb-409c-ac85-9f2ac606be79/09a64186-e4de-4db7-b903-c6397ff9a54d"
+          (reference "R10") (unit 1)
+        )
         (path "/b556fa32-e0cb-409c-ac85-9f2ac606be79/62656839-ead6-4c9d-b4ee-68fd3b49c6dd"
-          (reference "RN7") (unit 1)
+          (reference "R118") (unit 1)
         )
         (path "/b556fa32-e0cb-409c-ac85-9f2ac606be79/c41d3519-67b9-43b9-97c4-d20822b3d6ca"
-          (reference "RN25") (unit 1)
+          (reference "R236") (unit 1)
         )
       )

Commit message: Should be done with minimal version
Parts:
- C6, J7, R10, U31, U32, U33, U34, U35, U39, U44, U46, U47, U57, U73, U81: now not fitted; now left out of the parts list
- R10, R6, RN1, RN2, RN3, RN4, RN5, RN6, U74: now fitted; now in the parts list
