File: ESLGSU.kicad_sch (KiCad schematic)
At the start: 4 parts, among them J1 PJ-080BH, U1 TCA9544APWR

Commit message: Last tweaks on schematic
Parts:
- added TP1 (x3): TestPoint, TestPoint:TestPoint_Pad_D1.5mm, symbol Connector:TestPoint
- J1: JLCPCB BOM (none) -> 0; now left out of the parts list
Connections:
- net EPS_I2C_INT: now also TP1.1
- net EPS_I2C_SCL: now also TP1.1
- net EPS_I2C_SDA: now also TP1.1
Other:
- note added: "Nominal 5.5mm outer, 2.5mm inner, positive inner, DC jack. 10A max"
- note added: "To avoid I2C address contention of MP28167A regulators"
- note added: "UART Direct Bridge from Pi to Bus"
- note removed: "UART Direct Bridge"

Commit message: Finished initial revision of PCB
Parts:
- added H1, H2, H3: ~, MountingHole:MountingHole_2.5mm_Pad, symbol Mechanical:MountingHole_Pad
- added TP1 (x2): TestPoint, TestPoint:TestPoint_Pad_D1.5mm, symbol Connector:TestPoint
Connections:
- net CFGI2C_SCL: now also TP1.1
- net CFGI2C_SDA: now also TP1.1
- net GND: now also H1.1, H2.1, H3.1
Changed lines of the file:
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@@
   (junction (at 46.99 124.46) (diameter 0) (color 0 0 0 0)
   )
+  (junction (at 335.28 231.14) (diameter 0) (color 0 0 0 0)
+  )
   (junction (at 46.99 127) (diameter 0) (color 0 0 0 0)
   )
   (junction (at 39.37 93.98) (diameter 0) (color 0 0 0 0)
   )
+  (junction (at 326.39 231.14) (diameter 0) (color 0 0 0 0)
+  )
+  (junction (at 191.77 182.88) (diameter 0) (color 0 0 0 0)
+  )
+  (junction (at 194.31 185.42) (diameter 0) (color 0 0 0 0)
+  )
   (wire (pts (xy 34.29 91.44) (xy 36.83 91.44))
     (stroke (width 0) (type default))
@@
     (stroke (width 0) (type default))
   )
+  (wire (pts (xy 194.31 185.42) (xy 196.85 185.42))
+    (stroke (width 0) (type default))
+  )
   (wire (pts (xy 74.93 177.8) (xy 82.55 177.8))
     (stroke (width 0) (type default))
@@
     (stroke (width 0) (type default))
   )
+  (wire (pts (xy 191.77 182.88) (xy 193.04 182.88))
+    (stroke (width 0) (type default))
+  )
   (wire (pts (xy 270.51 161.29) (xy 274.32 161.29))
     (stroke (width 0) (type default))
@@
     (stroke (width 0) (type default))
   )
+  (wire (pts (xy 326.39 231.14) (xy 335.28 231.14))
+    (stroke (width 0) (type default))
+  )
   (wire (pts (xy 62.23 86.36) (xy 57.15 86.36))
     (stroke (width 0) (type default))
@@
     (stroke (width 0) (type default))
   )
-  (wire (pts (xy 189.23 182.88) (xy 193.04 182.88))
+  (wire (pts (xy 189.23 182.88) (xy 191.77 182.88))
     (stroke (width 0) (type default))
   )
@@
     (stroke (width 0) (type default))
   )
-  (wire (pts (xy 189.23 185.42) (xy 193.04 185.42))
+  (wire (pts (xy 189.23 185.42) (xy 194.31 185.42))
     (stroke (width 0) (type default))
   )
@@
   )
   (wire (pts (xy 222.25 73.66) (xy 226.06 73.66))
+    (stroke (width 0) (type default))
+  )
+  (wire (pts (xy 335.28 231.14) (xy 344.17 231.14))
     (stroke (width 0) (type default))
   )
@@
     (effects (font (size 1.27 1.27)) (justify right bottom))
   )
-  (label "CFGI2C_SCL" (at 193.04 185.42 0) (fields_autoplaced)
+  (label "CFGI2C_SCL" (at 196.85 185.42 0) (fields_autoplaced)
     (effects (font (size 1.27 1.27)) (justify left bottom))
   )
@@
     )
   )
+  (symbol (lib_id "Connector:TestPoint") (at 194.31 185.42 0) (unit 1)
+    (in_bom no) (on_board yes) (dnp no)
+    (property "Reference" "TP1" (at 193.04 187.96 0)
+      (effects (font (size 1.27 1.27)) (justify left))
+    )
+    (property "Value" "TestPoint" (at 193.04 190.5 0)
+      (effects (font (size 1.27 1.27)) (justify left))
+    )
+    (property "Footprint" "TestPoint:TestPoint_Pad_D1.5mm" (at 199.39 185.42 0)
+      (effects (font (size 1.27 1.27)) hide)
+    )
+    (property "Datasheet" "~" (at 199.39 185.42 0)
+      (effects (font (size 1.27 1.27)) hide)
+    )
+    (property "JLCPCB BOM" "0" (at 194.31 185.42 0)
+      (effects (font (size 1.27 1.27)) hide)
+    )
+    (pin "1")
+    (instances
+      (project "ESLGSU"
+        (path "/b556fa32-e0cb-409c-ac85-9f2ac606be79/09a64186-e4de-4db7-b903-c6397ff9a54d"
+          (reference "TP1") (unit 1)
+        )
+        (path "/b556fa32-e0cb-409c-ac85-9f2ac606be79/33c4fea8-f262-455e-abaf-737bb774af6a"
+          (reference "TP13") (unit 1)
+        )
+        (path "/b556fa32-e0cb-409c-ac85-9f2ac606be79"
+          (reference "TP37") (unit 1)
+        )
+      )
+    )
+  )
   (symbol (lib_id "power:GND") (at 68.58 86.36 0) (unit 1)
     (in_bom yes) (on_board yes) (dnp no)
@@
     )
   )
-  (symbol (lib_id "Connector:TestPoint") (at 39.37 93.98 0) (unit 1)
+  (symbol (lib_id "Connector:TestPoint") (at 191.77 182.88 0) (unit 1)
     (in_bom no) (on_board yes) (dnp no)
-    (property "Reference" "TP1" (at 22.86 99.06 0)
-      (effects (font (size 1.27 1.27)) (justify left))
-    )
-    (property "Value" "TestPoint" (at 22.86 101.6 0)
-      (effects (font (size 1.27 1.27)) (justify left))
-    )
-    (property "Footprint" "TestPoint:TestPoint_Pad_D1.5mm" (at 44.45 93.98 0)
-      (effects (font (size 1.27 1.27)) hide)
-    )
-    (property "Datasheet" "~" (at 44.45 93.98 0)
-      (effects (font (size 1.27 1.27)) hide)
-    )
-    (property "JLCPCB BOM" "0" (at 39.37 93.98 0)
+    (property "Reference" "TP1" (at 193.04 176.53 0)
+      (effects (font (size 1.27 1.27)) (justify left))
+    )
+    (property "Value" "TestPoint" (at 193.04 179.07 0)
+      (effects (font (size 1.27 1.27)) (justify left))
+    )
+    (property "Footprint" "TestPoint:TestPoint_Pad_D1.5mm" (at 196.85 182.88 0)
+      (effects (font (size 1.27 1.27)) hide)
+    )
+    (property "Datasheet" "~" (at 196.85 182.88 0)
+      (effects (font (size 1.27 1.27)) hide)
+    )
+    (property "JLCPCB BOM" "0" (at 191.77 182.88 0)
       (effects (font (size 1.27 1.27)) hide)
     )
@@
         )
         (path "/b556fa32-e0cb-409c-ac85-9f2ac606be79"
+          (reference "TP36") (unit 1)
+        )
+      )
+    )
+  )
+  (symbol (lib_id "power:GND") (at 326.39 231.14 0) (unit 1)
+    (in_bom yes) (on_board yes) (dnp no) (fields_autoplaced)
+    (property "Reference" "#PWR0262" (at 326.39 237.49 0)
+      (effects (font (size 1.27 1.27)) hide)
+    )
+    (property "Value" "GND" (at 326.39 236.22 0)
+      (effects (font (size 1.27 1.27)))
+    )
+    (property "Footprint" "" (at 326.39 231.14 0)
+      (effects (font (size 1.27 1.27)) hide)
+    )
+    (property "Datasheet" "" (at 326.39 231.14 0)
+      (effects (font (size 1.27 1.27)) hide)
+    )
+    (pin "1")
+    (instances
+      (project "ESLGSU"
+        (path "/b556fa32-e0cb-409c-ac85-9f2ac606be79"
+          (reference "#PWR0262") (unit 1)
+        )
+      )
+    )
+  )
+  (symbol (lib_id "Mechanical:MountingHole_Pad") (at 335.28 228.6 0) (unit 1)
+    (in_bom yes) (on_board yes) (dnp no) (fields_autoplaced)
+    (property "Reference" "H2" (at 337.82 226.06 0)
+      (effects (font (size 1.27 1.27)) (justify left))
+    )
+    (property "Value" "~" (at 337.82 228.6 0)
+      (effects (font (size 1.27 1.27)) (justify left))
+    )
+    (property "Footprint" "MountingHole:MountingHole_2.5mm_Pad" (at 335.28 228.6 0)
+      (effects (font (size 1.27 1.27)) hide)
+    )
+    (property "Datasheet" "~" (at 335.28 228.6 0)
+      (effects (font (size 1.27 1.27)) hide)
+    )
+    (pin "1")
+    (instances
+      (project "ESLGSU"
+        (path "/b556fa32-e0cb-409c-ac85-9f2ac606be79"
+          (reference "H2") (unit 1)
+        )
+      )
+    )
+  )
+  (symbol (lib_id "Connector:TestPoint") (at 39.37 93.98 0) (unit 1)
+    (in_bom no) (on_board yes) (dnp no)
+    (property "Reference" "TP1" (at 22.86 99.06 0)
+      (effects (font (size 1.27 1.27)) (justify left))
+    )
+    (property "Value" "TestPoint" (at 22.86 101.6 0)
+      (effects (font (size 1.27 1.27)) (justify left))
+    )
+    (property "Footprint" "TestPoint:TestPoint_Pad_D1.5mm" (at 44.45 93.98 0)
+      (effects (font (size 1.27 1.27)) hide)
+    )
+    (property "Datasheet" "~" (at 44.45 93.98 0)
+      (effects (font (size 1.27 1.27)) hide)
+    )
+    (property "JLCPCB BOM" "0" (at 39.37 93.98 0)
+      (effects (font (size 1.27 1.27)) hide)
+    )
+    (pin "1")
+    (instances
+      (project "ESLGSU"
+        (path "/b556fa32-e0cb-409c-ac85-9f2ac606be79/09a64186-e4de-4db7-b903-c6397ff9a54d"
+          (reference "TP1") (unit 1)
+        )
+        (path "/b556fa32-e0cb-409c-ac85-9f2ac606be79/33c4fea8-f262-455e-abaf-737bb774af6a"
+          (reference "TP13") (unit 1)
+        )
+        (path "/b556fa32-e0cb-409c-ac85-9f2ac606be79"
           (reference "TP2") (unit 1)
         )
       )
+    )
+  )
+  (symbol (lib_id "Mechanical:MountingHole_Pad") (at 326.39 228.6 0) (unit 1)
+    (in_bom yes) (on_board yes) (dnp no) (fields_autoplaced)
+    (property "Reference" "H1" (at 328.93 226.06 0)
+      (effects (font (size 1.27 1.27)) (justify left))
+    )
+    (property "Value" "~" (at 328.93 228.6 0)
+      (effects (font (size 1.27 1.27)) (justify left))
+    )
+    (property "Footprint" "MountingHole:MountingHole_2.5mm_Pad" (at 326.39 228.6 0)
+      (effects (font (size 1.27 1.27)) hide)
+    )
+    (property "Datasheet" "~" (at 326.39 228.6 0)
+      (effects (font (size 1.27 1.27)) hide)
+    )
+    (pin "1")
+    (instances
+      (project "ESLGSU"
+        (path "/b556fa32-e0cb-409c-ac85-9f2ac606be79"
+          (reference "H1") (unit 1)
+        )
+      )
+    )
+  )
+  (symbol (lib_id "Mechanical:MountingHole_Pad") (at 344.17 228.6 0) (unit 1)
+    (in_bom yes) (on_board yes) (dnp no) (fields_autoplaced)
+    (property "Reference" "H3" (at 346.71 226.06 0)
+      (effects (font (size 1.27 1.27)) (justify left))
+    )
+    (property "Value" "~" (at 346.71 228.6 0)
+      (effects (font (size 1.27 1.27)) (justify left))
+    )
+    (property "Footprint" "MountingHole:MountingHole_2.5mm_Pad" (at 344.17 228.6 0)
+      (effects (font (size 1.27 1.27)) hide)
+    )
+    (property "Datasheet" "~" (at 344.17 228.6 0)
+      (effects (font (size 1.27 1.27)) hide)
+    )
+    (pin "1")
+    (instances
+      (project "ESLGSU"
+        (path "/b556fa32-e0cb-409c-ac85-9f2ac606be79"
+          (reference "H3") (unit 1)
+        )
+      )

Commit message: Finished for production
Parts:
- H1, H2, H3: now left out of the parts list
- J1: now not fitted
Connections:
- net GND: no longer H1.1, H2.1, H3.1
- new net: H1.1, H2.1, H3.1
Changed lines of the file:
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@@
   (junction (at 39.37 93.98) (diameter 0) (color 0 0 0 0)
-  )
-  (junction (at 326.39 231.14) (diameter 0) (color 0 0 0 0)
   )
   (junction (at 191.77 182.88) (diameter 0) (color 0 0 0 0)
@@
     )
   )
-  (symbol (lib_id "power:GND") (at 326.39 231.14 0) (unit 1)
-    (in_bom yes) (on_board yes) (dnp no) (fields_autoplaced)
-    (property "Reference" "#PWR0262" (at 326.39 237.49 0)
-      (effects (font (size 1.27 1.27)) hide)
-    )
-    (property "Value" "GND" (at 326.39 236.22 0)
-      (effects (font (size 1.27 1.27)))
-    )
-    (property "Footprint" "" (at 326.39 231.14 0)
-      (effects (font (size 1.27 1.27)) hide)
-    )
-    (property "Datasheet" "" (at 326.39 231.14 0)
-      (effects (font (size 1.27 1.27)) hide)
-    )
-    (pin "1")
-    (instances
-      (project "ESLGSU"
-        (path "/b556fa32-e0cb-409c-ac85-9f2ac606be79"
-          (reference "#PWR0262") (unit 1)
-        )
-      )
-    )
-  )
   (symbol (lib_id "Mechanical:MountingHole_Pad") (at 335.28 228.6 0) (unit 1)
-    (in_bom yes) (on_board yes) (dnp no) (fields_autoplaced)
+    (in_bom no) (on_board yes) (dnp no) (fields_autoplaced)
     (property "Reference" "H2" (at 337.82 226.06 0)
       (effects (font (size 1.27 1.27)) (justify left))
@@
   )
   (symbol (lib_id "Mechanical:MountingHole_Pad") (at 326.39 228.6 0) (unit 1)
-    (in_bom yes) (on_board yes) (dnp no) (fields_autoplaced)
+    (in_bom no) (on_board yes) (dnp no) (fields_autoplaced)
     (property "Reference" "H1" (at 328.93 226.06 0)
       (effects (font (size 1.27 1.27)) (justify left))
@@
   )
   (symbol (lib_id "Mechanical:MountingHole_Pad") (at 344.17 228.6 0) (unit 1)
-    (in_bom yes) (on_board yes) (dnp no) (fields_autoplaced)
+    (in_bom no) (on_board yes) (dnp no) (fields_autoplaced)
     (property "Reference" "H3" (at 346.71 226.06 0)
       (effects (font (size 1.27 1.27)) (justify left))
@@
   )
   (symbol (lib_id "Connector:Barrel_Jack_Switch") (at 40.64 34.29 0) (unit 1)
-    (in_bom no) (on_board yes) (dnp no) (fields_autoplaced)
+    (in_bom no) (on_board yes) (dnp yes) (fields_autoplaced)
     (property "Reference" "J1" (at 40.64 25.4 0)
       (effects (font (size 1.27 1.27)))

Commit message: Replaced netwroks with individual resistors
Parts:
- removed RN6: 0R, Resistor_SMD:R_Array_Convex_2x0402, symbol Device:R_Pack02
- added R6 (x2): 0R, Resistor_SMD:R_0402_1005Metric, symbol Device:R_Small_US
Connections:
- net PISER_RX: now also R6.2
- net PISER_TX: now also R6.2
- net UART1_RX: now also R6.1
- net UART1_TX: now also R6.1
Changed lines of the file:
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@@
     (stroke (width 0) (type default))
   )
-  (wire (pts (xy 327.66 193.04) (xy 325.12 193.04))
+  (wire (pts (xy 322.58 193.04) (xy 327.66 193.04))
     (stroke (width 0) (type default))
   )
@@
     (stroke (width 0) (type default))
   )
-  (wire (pts (xy 311.15 195.58) (xy 314.96 195.58))
+  (wire (pts (xy 311.15 195.58) (xy 317.5 195.58))
     (stroke (width 0) (type default))
   )
@@
     (stroke (width 0) (type default))
   )
-  (wire (pts (xy 311.15 193.04) (xy 314.96 193.04))
+  (wire (pts (xy 311.15 193.04) (xy 317.5 193.04))
     (stroke (width 0) (type default))
   )
@@
     (stroke (width 0) (type default))
   )
-  (wire (pts (xy 327.66 195.58) (xy 325.12 195.58))
+  (wire (pts (xy 322.58 195.58) (xy 327.66 195.58))
     (stroke (width 0) (type default))
   )
@@
         (path "/b556fa32-e0cb-409c-ac85-9f2ac606be79"
           (reference "TP1") (unit 1)
+        )
+      )
+    )
+  )
+  (symbol (lib_id "Device:R_Small_US") (at 320.04 195.58 270) (unit 1)
+    (in_bom no) (on_board yes) (dnp yes)
+    (property "Reference" "R6" (at 317.5 198.12 90)
+      (effects (font (size 1.27 1.27)) (justify left))
+    )
+    (property "Value" "0R" (at 323.85 198.12 90)
+      (effects (font (size 1.27 1.27)) (justify left))
+    )
+    (property "Footprint" "Resistor_SMD:R_0402_1005Metric" (at 320.04 195.58 0)
+      (effects (font (size 1.27 1.27)) hide)
+    )
+    (property "Datasheet" "~" (at 320.04 195.58 0)
+      (effects (font (size 1.27 1.27)) hide)
+    )
+    (property "LCSC Part" "C17168" (at 320.04 187.96 0)
+      (effects (font (size 1.27 1.27)) hide)
+    )
+    (property "JLCPCB BOM" "0" (at 320.04 195.58 90)
+      (effects (font (size 1.27 1.27)) hide)
+    )
+    (pin "1")
+    (pin "2")
+    (instances
+      (project "ESLGSU"
+        (path "/b556fa32-e0cb-409c-ac85-9f2ac606be79/09a64186-e4de-4db7-b903-c6397ff9a54d"
+          (reference "R6") (unit 1)
+        )
+        (path "/b556fa32-e0cb-409c-ac85-9f2ac606be79/62656839-ead6-4c9d-b4ee-68fd3b49c6dd"
+          (reference "R191") (unit 1)
+        )
+        (path "/b556fa32-e0cb-409c-ac85-9f2ac606be79/c41d3519-67b9-43b9-97c4-d20822b3d6ca"
+          (reference "R320") (unit 1)
+        )
+        (path "/b556fa32-e0cb-409c-ac85-9f2ac606be79"
+          (reference "R340") (unit 1)
         )
       )
@@
     )
   )
-  (symbol (lib_id "Device:R_Pack02") (at 320.04 193.04 90) (unit 1)
-    (in_bom no) (on_board yes) (dnp yes)
-    (property "Reference" "RN6" (at 327.66 196.85 90)
-      (effects (font (size 1.27 1.27)))
-    )
-    (property "Value" "0R" (at 327.66 199.39 90)
-      (effects (font (size 1.27 1.27)))
-    )
-    (property "Footprint" "Resistor_SMD:R_Array_Convex_2x0402" (at 320.04 188.595 90)
-      (effects (font (size 1.27 1.27)) hide)
-    )
-    (property "Datasheet" "~" (at 320.04 193.04 0)
-      (effects (font (size 1.27 1.27)) hide)
-    )
-    (property "LCSC Part" "C75375" (at 327.66 199.39 90)
-      (effects (font (size 1.27 1.27)) hide)
-    )
-    (property "JLCPCB BOM" "0" (at 320.04 193.04 90)
-      (effects (font (size 1.27 1.27)) hide)
-    )
-    (pin "1")
-    (pin "2")
-    (pin "3")
-    (pin "4")
-    (instances
-      (project "ESLGSU"
-        (path "/b556fa32-e0cb-409c-ac85-9f2ac606be79/62656839-ead6-4c9d-b4ee-68fd3b49c6dd"
-          (reference "RN6") (unit 1)
-        )
-        (path "/b556fa32-e0cb-409c-ac85-9f2ac606be79/c41d3519-67b9-43b9-97c4-d20822b3d6ca"
-          (reference "RN21") (unit 1)
-        )
-        (path "/b556fa32-e0cb-409c-ac85-9f2ac606be79"
-          (reference "RN1") (unit 1)
-        )
-      )
-    )
-  )
   (symbol (lib_id "power:GND") (at 57.15 134.62 0) (unit 1)
     (in_bom yes) (on_board yes) (dnp no) (fields_autoplaced)
@@
         )
       )
+    )
+  )
+  (symbol (lib_id "Device:R_Small_US") (at 320.04 193.04 270) (unit 1)
+    (in_bom no) (on_board yes) (dnp yes)
+    (property "Reference" "R6" (at 317.5 190.5 90)
+      (effects (font (size 1.27 1.27)) (justify left))
+    )
+    (property "Value" "0R" (at 323.85 190.5 90)
+      (effects (font (size 1.27 1.27)) (justify left))
+    )
+    (property "Footprint" "Resistor_SMD:R_0402_1005Metric" (at 320.04 193.04 0)
+      (effects (font (size 1.27 1.27)) hide)
+    )
+    (property "Datasheet" "~" (at 320.04 193.04 0)
+      (effects (font (size 1.27 1.27)) hide)
+    )
+    (property "LCSC Part" "C17168" (at 320.04 185.42 0)
+      (effects (font (size 1.27 1.27)) hide)
+    )
+    (property "JLCPCB BOM" "0" (at 320.04 193.04 90)
+      (effects (font (size 1.27 1.27)) hide)
+    )
+    (pin "1")
+    (pin "2")
+    (instances
+      (project "ESLGSU"
+        (path "/b556fa32-e0cb-409c-ac85-9f2ac606be79/09a64186-e4de-4db7-b903-c6397ff9a54d"
+          (reference "R6") (unit 1)
+        )
+        (path "/b556fa32-e0cb-409c-ac85-9f2ac606be79/62656839-ead6-4c9d-b4ee-68fd3b49c6dd"
+          (reference "R190") (unit 1)
+        )
+        (path "/b556fa32-e0cb-409c-ac85-9f2ac606be79/c41d3519-67b9-43b9-97c4-d20822b3d6ca"
+          (reference "R319") (unit 1)
+        )
+        (path "/b556fa32-e0cb-409c-ac85-9f2ac606be79"
+          (reference "R339") (unit 1)
+        )
+      )
