File: ESLGSU.kicad_sch (KiCad schematic)
At the start: 13 parts, among them J1 PJ-080BH, U1 TCA9544APWR

Commit message: Revert "Replaced netwroks with individual resistors"
This reverts commit e13850981b8de489d340064652a5562029ab4f8c.
Parts:
- removed R6 (x2): 0R, Resistor_SMD:R_0402_1005Metric, symbol Device:R_Small_US
- added RN6: 0R, Resistor_SMD:R_Array_Convex_2x0402, symbol Device:R_Pack02
Connections:
- net PISER_RX: now also RN6.4 (R1.2)
- net PISER_TX: now also RN6.3 (R2.2)
- net UART1_RX: now also RN6.1 (R1.1)
- net UART1_TX: now also RN6.2 (R2.1)
Changed lines of the file:
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@@
     (stroke (width 0) (type default))
   )
-  (wire (pts (xy 322.58 193.04) (xy 327.66 193.04))
+  (wire (pts (xy 327.66 193.04) (xy 325.12 193.04))
     (stroke (width 0) (type default))
   )
@@
     (stroke (width 0) (type default))
   )
-  (wire (pts (xy 311.15 195.58) (xy 317.5 195.58))
+  (wire (pts (xy 311.15 195.58) (xy 314.96 195.58))
     (stroke (width 0) (type default))
   )
@@
     (stroke (width 0) (type default))
   )
-  (wire (pts (xy 311.15 193.04) (xy 317.5 193.04))
+  (wire (pts (xy 311.15 193.04) (xy 314.96 193.04))
     (stroke (width 0) (type default))
   )
@@
     (stroke (width 0) (type default))
   )
-  (wire (pts (xy 322.58 195.58) (xy 327.66 195.58))
+  (wire (pts (xy 327.66 195.58) (xy 325.12 195.58))
     (stroke (width 0) (type default))
   )
@@
         (path "/b556fa32-e0cb-409c-ac85-9f2ac606be79"
           (reference "TP1") (unit 1)
-        )
-      )
-    )
-  )
-  (symbol (lib_id "Device:R_Small_US") (at 320.04 195.58 270) (unit 1)
-    (in_bom no) (on_board yes) (dnp yes)
-    (property "Reference" "R6" (at 317.5 198.12 90)
-      (effects (font (size 1.27 1.27)) (justify left))
-    )
-    (property "Value" "0R" (at 323.85 198.12 90)
-      (effects (font (size 1.27 1.27)) (justify left))
-    )
-    (property "Footprint" "Resistor_SMD:R_0402_1005Metric" (at 320.04 195.58 0)
-      (effects (font (size 1.27 1.27)) hide)
-    )
-    (property "Datasheet" "~" (at 320.04 195.58 0)
-      (effects (font (size 1.27 1.27)) hide)
-    )
-    (property "LCSC Part" "C17168" (at 320.04 187.96 0)
-      (effects (font (size 1.27 1.27)) hide)
-    )
-    (property "JLCPCB BOM" "0" (at 320.04 195.58 90)
-      (effects (font (size 1.27 1.27)) hide)
-    )
-    (pin "1")
-    (pin "2")
-    (instances
-      (project "ESLGSU"
-        (path "/b556fa32-e0cb-409c-ac85-9f2ac606be79/09a64186-e4de-4db7-b903-c6397ff9a54d"
-          (reference "R6") (unit 1)
-        )
-        (path "/b556fa32-e0cb-409c-ac85-9f2ac606be79/62656839-ead6-4c9d-b4ee-68fd3b49c6dd"
-          (reference "R191") (unit 1)
-        )
-        (path "/b556fa32-e0cb-409c-ac85-9f2ac606be79/c41d3519-67b9-43b9-97c4-d20822b3d6ca"
-          (reference "R320") (unit 1)
-        )
-        (path "/b556fa32-e0cb-409c-ac85-9f2ac606be79"
-          (reference "R340") (unit 1)
         )
       )
@@
     )
   )
+  (symbol (lib_id "Device:R_Pack02") (at 320.04 193.04 90) (unit 1)
+    (in_bom no) (on_board yes) (dnp yes)
+    (property "Reference" "RN6" (at 327.66 196.85 90)
+      (effects (font (size 1.27 1.27)))
+    )
+    (property "Value" "0R" (at 327.66 199.39 90)
+      (effects (font (size 1.27 1.27)))
+    )
+    (property "Footprint" "Resistor_SMD:R_Array_Convex_2x0402" (at 320.04 188.595 90)
+      (effects (font (size 1.27 1.27)) hide)
+    )
+    (property "Datasheet" "~" (at 320.04 193.04 0)
+      (effects (font (size 1.27 1.27)) hide)
+    )
+    (property "LCSC Part" "C75375" (at 327.66 199.39 90)
+      (effects (font (size 1.27 1.27)) hide)
+    )
+    (property "JLCPCB BOM" "0" (at 320.04 193.04 90)
+      (effects (font (size 1.27 1.27)) hide)
+    )
+    (pin "1")
+    (pin "2")
+    (pin "3")
+    (pin "4")
+    (instances
+      (project "ESLGSU"
+        (path "/b556fa32-e0cb-409c-ac85-9f2ac606be79/62656839-ead6-4c9d-b4ee-68fd3b49c6dd"
+          (reference "RN6") (unit 1)
+        )
+        (path "/b556fa32-e0cb-409c-ac85-9f2ac606be79/c41d3519-67b9-43b9-97c4-d20822b3d6ca"
+          (reference "RN21") (unit 1)
+        )
+        (path "/b556fa32-e0cb-409c-ac85-9f2ac606be79"
+          (reference "RN1") (unit 1)
+        )
+      )
+    )
+  )
   (symbol (lib_id "power:GND") (at 57.15 134.62 0) (unit 1)
     (in_bom yes) (on_board yes) (dnp no) (fields_autoplaced)
@@
         )
       )
-    )
-  )
-  (symbol (lib_id "Device:R_Small_US") (at 320.04 193.04 270) (unit 1)
-    (in_bom no) (on_board yes) (dnp yes)
-    (property "Reference" "R6" (at 317.5 190.5 90)
-      (effects (font (size 1.27 1.27)) (justify left))
-    )
-    (property "Value" "0R" (at 323.85 190.5 90)
-      (effects (font (size 1.27 1.27)) (justify left))
-    )
-    (property "Footprint" "Resistor_SMD:R_0402_1005Metric" (at 320.04 193.04 0)
-      (effects (font (size 1.27 1.27)) hide)
-    )
-    (property "Datasheet" "~" (at 320.04 193.04 0)
-      (effects (font (size 1.27 1.27)) hide)
-    )
-    (property "LCSC Part" "C17168" (at 320.04 185.42 0)
-      (effects (font (size 1.27 1.27)) hide)
-    )
-    (property "JLCPCB BOM" "0" (at 320.04 193.04 90)
-      (effects (font (size 1.27 1.27)) hide)
-    )
-    (pin "1")
-    (pin "2")
-    (instances
-      (project "ESLGSU"
-        (path "/b556fa32-e0cb-409c-ac85-9f2ac606be79/09a64186-e4de-4db7-b903-c6397ff9a54d"
-          (reference "R6") (unit 1)
-        )
-        (path "/b556fa32-e0cb-409c-ac85-9f2ac606be79/62656839-ead6-4c9d-b4ee-68fd3b49c6dd"
-          (reference "R190") (unit 1)
-        )
-        (path "/b556fa32-e0cb-409c-ac85-9f2ac606be79/c41d3519-67b9-43b9-97c4-d20822b3d6ca"
-          (reference "R319") (unit 1)
-        )
-        (path "/b556fa32-e0cb-409c-ac85-9f2ac606be79"
-          (reference "R339") (unit 1)
-        )
-      )

Commit message: Hopefully final full PCB version
Other:
- added sheet Power_Switches (ESLGSU_Power_Switches.kicad_sch)
- sheet Bus_Umbilical ports: added 3V3_S1, 3V3_S2, 5V_S1, 5V_S2; removed none
- sheet EPS_uC ports: added EN_3V3_S1, EN_3V3_S2, EN_5V_S1, EN_5V_S2; removed none
