File: ESLGSU_Bus_Umbilical.kicad_sch (KiCad schematic)
At the start: 0 parts

Commit message: uC Interface work
Other:
- company: (none) -> Electronic Systems Laboratory
Changed lines of the file:
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@@
 (kicad_sch (version 20230121) (generator eeschema)
   (paper "A4")
+  (title_block
+    (date "2024-01-18")
+    (rev "1")
+    (company "Electronic Systems Laboratory")
+  )
 )

Commit message: Final schematic work, added battery charger, linked everything up
Parts:
- added J6: AMPHENOL_62684-401100ALF, ESLGSU_Parts_Lib:AMPHENOL_62684-401100ALF, symbol Connector_Generic_MountingPin:Conn_01x40_MountingPin
- added J8: 1054301108, ESLGSU_Parts_Lib:MOLEX_1054301108, symbol Connector_Generic_MountingPin:Conn_01x08_MountingPin
Connections:
- new net BUS_3V3: J8.1 (Pin_1)
- new net BUS_5V: J8.2 (Pin_2)
- new net BUS_CH1: J8.7 (Pin_7)
- new net BUS_CH2: J8.8 (Pin_8)
- new net BUS_UNREG: J8.4 (Pin_4), J8.5 (Pin_5)
- new net CAN1_H: J6.03 (Pin_3)
- new net CAN1_L: J6.02 (Pin_2)
- new net CAN2_H: J6.05 (Pin_5)
- new net CAN2_L: J6.04 (Pin_4)
- new net GND: J6.01 (Pin_1), J6.06 (Pin_6), J6.11 (Pin_11), J6.16 (Pin_16), J6.21 (Pin_21), J6.26 (Pin_26), J6.31 (Pin_31), J6.40 (Pin_40), J6.S1 (MountPin), J6.S2 (MountPin), J8.3 (Pin_3), J8.6 (Pin_6), J8.S1 (MountPin), J8.S2 (MountPin)
- new net GPIO_1: J6.32 (Pin_32)
- new net GPIO_2: J6.33 (Pin_33)
- new net GPIO_3: J6.34 (Pin_34)
- new net GPIO_4: J6.35 (Pin_35)
- new net GPIO_5: J6.36 (Pin_36)
- new net GPIO_6: J6.37 (Pin_37)
- new net GPIO_7: J6.38 (Pin_38)
- new net GPIO_8: J6.39 (Pin_39)
- new net I2C1_SCL: J6.17 (Pin_17)
- new net I2C1_SDA: J6.18 (Pin_18)
- new net I2C2_SCL: J6.19 (Pin_19)
- new net I2C2_SDA: J6.20 (Pin_20)
- new net RS4851_A: J6.07 (Pin_7)
- new net RS4851_B: J6.08 (Pin_8)
- new net RS4852_A: J6.09 (Pin_9)
- new net RS4852_B: J6.10 (Pin_10)
- new net SPI1_MISO: J6.22 (Pin_22)
- new net SPI1_MOSI: J6.23 (Pin_23)
- new net SPI1_NSS: J6.25 (Pin_25)
- new net SPI1_SCK: J6.24 (Pin_24)
- new net SPI2_MISO: J6.27 (Pin_27)
- new net SPI2_MOSI: J6.28 (Pin_28)
- new net SPI2_NSS: J6.30 (Pin_30)
- new net SPI2_SCK: J6.29 (Pin_29)
- new net UART1_RX: J6.13 (Pin_13)
- new net UART1_TX: J6.12 (Pin_12)
- new net UART2_RX: J6.15 (Pin_15)
- new net UART2_TX: J6.14 (Pin_14)

Commit message: Last tweaks on schematic
Parts:
- renumbered J8 to J10, J6 to J9
Changed lines of the file:
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@@
   (symbol (lib_id "power:GND") (at 120.65 111.76 0) (unit 1)
     (in_bom yes) (on_board yes) (dnp no) (fields_autoplaced)
-    (property "Reference" "#PWR0226" (at 120.65 118.11 0)
+    (property "Reference" "#PWR0257" (at 120.65 118.11 0)
       (effects (font (size 1.27 1.27)) hide)
     )
@@
       (project "ESLGSU"
         (path "/b556fa32-e0cb-409c-ac85-9f2ac606be79/feac87e8-d04c-4646-81d1-6a4c94f01f41"
-          (reference "#PWR0226") (unit 1)
+          (reference "#PWR0257") (unit 1)
         )
       )
@@
   (symbol (lib_id "power:GND") (at 60.96 116.84 270) (unit 1)
     (in_bom yes) (on_board yes) (dnp no) (fields_autoplaced)
-    (property "Reference" "#PWR0220" (at 54.61 116.84 0)
+    (property "Reference" "#PWR0258" (at 54.61 116.84 0)
       (effects (font (size 1.27 1.27)) hide)
     )
@@
       (project "ESLGSU"
         (path "/b556fa32-e0cb-409c-ac85-9f2ac606be79/feac87e8-d04c-4646-81d1-6a4c94f01f41"
-          (reference "#PWR0220") (unit 1)
+          (reference "#PWR0258") (unit 1)
         )
       )
@@
   (symbol (lib_id "power:GND") (at 60.96 91.44 270) (unit 1)
     (in_bom yes) (on_board yes) (dnp no) (fields_autoplaced)
-    (property "Reference" "#PWR0219" (at 54.61 91.44 0)
+    (property "Reference" "#PWR0253" (at 54.61 91.44 0)
       (effects (font (size 1.27 1.27)) hide)
     )
@@
       (project "ESLGSU"
         (path "/b556fa32-e0cb-409c-ac85-9f2ac606be79/feac87e8-d04c-4646-81d1-6a4c94f01f41"
-          (reference "#PWR0219") (unit 1)
+          (reference "#PWR0253") (unit 1)
         )
       )
@@
   (symbol (lib_id "power:GND") (at 60.96 104.14 270) (unit 1)
     (in_bom yes) (on_board yes) (dnp no) (fields_autoplaced)
-    (property "Reference" "#PWR0223" (at 54.61 104.14 0)
+    (property "Reference" "#PWR0256" (at 54.61 104.14 0)
       (effects (font (size 1.27 1.27)) hide)
     )
@@
       (project "ESLGSU"
         (path "/b556fa32-e0cb-409c-ac85-9f2ac606be79/feac87e8-d04c-4646-81d1-6a4c94f01f41"
-          (reference "#PWR0223") (unit 1)
+          (reference "#PWR0256") (unit 1)
         )
       )
@@
   (symbol (lib_id "power:GND") (at 60.96 139.7 270) (unit 1)
     (in_bom yes) (on_board yes) (dnp no) (fields_autoplaced)
-    (property "Reference" "#PWR0221" (at 54.61 139.7 0)
+    (property "Reference" "#PWR0259" (at 54.61 139.7 0)
       (effects (font (size 1.27 1.27)) hide)
     )
@@
       (project "ESLGSU"
         (path "/b556fa32-e0cb-409c-ac85-9f2ac606be79/feac87e8-d04c-4646-81d1-6a4c94f01f41"
-          (reference "#PWR0221") (unit 1)
+          (reference "#PWR0259") (unit 1)
         )
       )
@@
   (symbol (lib_id "power:GND") (at 111.76 101.6 270) (unit 1)
     (in_bom yes) (on_board yes) (dnp no) (fields_autoplaced)
-    (property "Reference" "#PWR0246" (at 105.41 101.6 0)
+    (property "Reference" "#PWR0255" (at 105.41 101.6 0)
       (effects (font (size 1.27 1.27)) hide)
     )
@@
       (project "ESLGSU"
         (path "/b556fa32-e0cb-409c-ac85-9f2ac606be79/feac87e8-d04c-4646-81d1-6a4c94f01f41"
-          (reference "#PWR0246") (unit 1)
+          (reference "#PWR0255") (unit 1)
         )
       )
@@
   (symbol (lib_id "power:GND") (at 60.96 40.64 270) (unit 1)
     (in_bom yes) (on_board yes) (dnp no) (fields_autoplaced)
-    (property "Reference" "#PWR0222" (at 54.61 40.64 0)
+    (property "Reference" "#PWR0249" (at 54.61 40.64 0)
       (effects (font (size 1.27 1.27)) hide)
     )
@@
       (project "ESLGSU"
         (path "/b556fa32-e0cb-409c-ac85-9f2ac606be79/feac87e8-d04c-4646-81d1-6a4c94f01f41"
-          (reference "#PWR0222") (unit 1)
+          (reference "#PWR0249") (unit 1)
         )
       )
@@
   (symbol (lib_id "Connector_Generic_MountingPin:Conn_01x08_MountingPin") (at 120.65 96.52 0) (unit 1)
     (in_bom yes) (on_board yes) (dnp no) (fields_autoplaced)
-    (property "Reference" "J8" (at 123.19 96.8756 0)
+    (property "Reference" "J10" (at 123.19 96.8756 0)
       (effects (font (size 1.27 1.27)) (justify left))
     )
@@
       (effects (font (size 1.27 1.27)) hide)
     )
-    (pin "4")
-    (pin "S1")
-    (pin "5")
+    (pin "S2")
+    (pin "1")
     (pin "2")
     (pin "3")
+    (pin "4")
+    (pin "5")
     (pin "6")
-    (pin "S2")
+    (pin "7")
     (pin "8")
-    (pin "7")
-    (pin "1")
-    (instances
-      (project "ESLGSU"
-        (path "/b556fa32-e0cb-409c-ac85-9f2ac606be79/feac87e8-d04c-4646-81d1-6a4c94f01f41"
-          (reference "J8") (unit 1)
+    (pin "S1")
+    (instances
+      (project "ESLGSU"
+        (path "/b556fa32-e0cb-409c-ac85-9f2ac606be79/feac87e8-d04c-4646-81d1-6a4c94f01f41"
+          (reference "J10") (unit 1)
         )
       )
@@
   (symbol (lib_id "Connector_Generic_MountingPin:Conn_01x40_MountingPin") (at 69.85 88.9 0) (unit 1)
     (in_bom yes) (on_board yes) (dnp no)
-    (property "Reference" "J6" (at 55.88 156.21 0)
+    (property "Reference" "J9" (at 55.88 156.21 0)
       (effects (font (size 1.27 1.27)) (justify left))
     )
@@
       (effects (font (size 1.27 1.27)) hide)
     )
+    (pin "01")
+    (pin "02")
+    (pin "03")
+    (pin "04")
+    (pin "05")
+    (pin "06")
+    (pin "07")
+    (pin "08")
+    (pin "09")
+    (pin "10")
+    (pin "11")
     (pin "12")
+    (pin "13")
+    (pin "14")
+    (pin "15")
+    (pin "16")
+    (pin "17")
+    (pin "18")
+    (pin "19")
+    (pin "20")
+    (pin "21")
+    (pin "22")
+    (pin "23")
+    (pin "24")
+    (pin "25")
+    (pin "26")
+    (pin "27")
+    (pin "28")
+    (pin "29")
+    (pin "30")
+    (pin "31")
+    (pin "32")
+    (pin "33")
+    (pin "34")
     (pin "35")
-    (pin "25")
+    (pin "36")
     (pin "37")
-    (pin "26")
-    (pin "10")
-    (pin "22")
-    (pin "19")
-    (pin "30")
     (pin "38")
     (pin "39")
-    (pin "04")
-    (pin "03")
-    (pin "34")
-    (pin "05")
-    (pin "16")
-    (pin "23")
-    (pin "28")
-    (pin "08")
-    (pin "17")
-    (pin "32")
-    (pin "20")
-    (pin "27")
-    (pin "36")
+    (pin "40")
+    (pin "S1")
     (pin "S2")
-    (pin "18")
-    (pin "02")
-    (pin "06")
-    (pin "33")
-    (pin "09")
-    (pin "13")
-    (pin "07")
-    (pin "01")
-    (pin "11")
-    (pin "14")
-    (pin "15")
-    (pin "24")
-    (pin "21")
-    (pin "31")
-    (pin "40")
-    (pin "29")
-    (pin "S1")
-    (instances
-      (project "ESLGSU"
-        (path "/b556fa32-e0cb-409c-ac85-9f2ac606be79/feac87e8-d04c-4646-81d1-6a4c94f01f41"
-          (reference "J6") (unit 1)
+    (instances
+      (project "ESLGSU"
+        (path "/b556fa32-e0cb-409c-ac85-9f2ac606be79/feac87e8-d04c-4646-81d1-6a4c94f01f41"
+          (reference "J9") (unit 1)
         )
       )
@@
   (symbol (lib_id "power:GND") (at 111.76 93.98 270) (unit 1)
     (in_bom yes) (on_board yes) (dnp no) (fields_autoplaced)
-    (property "Reference" "#PWR0227" (at 105.41 93.98 0)
+    (property "Reference" "#PWR0254" (at 105.41 93.98 0)
       (effects (font (size 1.27 1.27)) hide)
     )
@@
       (project "ESLGSU"
         (path "/b556fa32-e0cb-409c-ac85-9f2ac606be79/feac87e8-d04c-4646-81d1-6a4c94f01f41"
-          (reference "#PWR0227") (unit 1)
+          (reference "#PWR0254") (unit 1)
         )
       )
@@
   (symbol (lib_id "power:GND") (at 69.85 144.78 0) (unit 1)
     (in_bom yes) (on_board yes) (dnp no) (fields_autoplaced)
-    (property "Reference" "#PWR0215" (at 69.85 151.13 0)
+    (property "Reference" "#PWR0260" (at 69.85 151.13 0)
       (effects (font (size 1.27 1.27)) hide)
     )
@@
       (project "ESLGSU"
         (path "/b556fa32-e0cb-409c-ac85-9f2ac606be79/feac87e8-d04c-4646-81d1-6a4c94f01f41"
-          (reference "#PWR0215") (unit 1)
+          (reference "#PWR0260") (unit 1)
         )
       )
@@
   (symbol (lib_id "power:GND") (at 60.96 53.34 270) (unit 1)
     (in_bom yes) (on_board yes) (dnp no) (fields_autoplaced)
-    (property "Reference" "#PWR0216" (at 54.61 53.34 0)
+    (property "Reference" "#PWR0250" (at 54.61 53.34 0)
       (effects (font (size 1.27 1.27)) hide)
     )
@@
       (project "ESLGSU"
         (path "/b556fa32-e0cb-409c-ac85-9f2ac606be79/feac87e8-d04c-4646-81d1-6a4c94f01f41"
-          (reference "#PWR0216") (unit 1)
+          (reference "#PWR0250") (unit 1)
         )
       )
@@
   (symbol (lib_id "power:GND") (at 60.96 66.04 270) (unit 1)
     (in_bom yes) (on_board yes) (dnp no) (fields_autoplaced)
-    (property "Reference" "#PWR0217" (at 54.61 66.04 0)
+    (property "Reference" "#PWR0251" (at 54.61 66.04 0)
       (effects (font (size 1.27 1.27)) hide)
     )
@@
       (project "ESLGSU"
         (path "/b556fa32-e0cb-409c-ac85-9f2ac606be79/feac87e8-d04c-4646-81d1-6a4c94f01f41"
-          (reference "#PWR0217") (unit 1)
+          (reference "#PWR0251") (unit 1)
         )
       )
@@
   (symbol (lib_id "power:GND") (at 60.96 78.74 270) (unit 1)
     (in_bom yes) (on_board yes) (dnp no) (fields_autoplaced)
-    (property "Reference" "#PWR0218" (at 54.61 78.74 0)
+    (property "Reference" "#PWR0252" (at 54.61 78.74 0)
       (effects (font (size 1.27 1.27)) hide)
     )
@@
       (project "ESLGSU"
         (path "/b556fa32-e0cb-409c-ac85-9f2ac606be79/feac87e8-d04c-4646-81d1-6a4c94f01f41"
-          (reference "#PWR0218") (unit 1)
-        )
-      )
+          (reference "#PWR0252") (unit 1)
+        )
+      )

Commit message: Finished for production
Parts:
- J9: LCDC Part C2904111 -> (none); LCSC Part (none) -> C2904111
Changed lines of the file:
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@@
       (effects (font (size 1.27 1.27)) hide)
     )
-    (property "LCDC Part" "C2904111" (at 69.85 88.9 0)
+    (property "LCSC Part" "C2904111" (at 69.85 88.9 0)
       (effects (font (size 1.27 1.27)) hide)
     )

Commit message: Hopefully final full PCB version
Connections:
- net GND: no longer J9.01 (Pin_1), J9.11 (Pin_11), J9.21 (Pin_21), J9.31 (Pin_31)
- new net 3V3_S1: J9.01 (Pin_1)
- new net 3V3_S2: J9.11 (Pin_11)
- new net 5V_S1: J9.21 (Pin_21)
- new net 5V_S2: J9.31 (Pin_31)
Changed lines of the file:
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@@
+    (stroke (width 0) (type default))
+  )
+  (wire (pts (xy 60.96 101.6) (xy 64.77 101.6))
+    (stroke (width 0) (type default))
+  )
+  (wire (pts (xy 60.96 53.34) (xy 64.77 53.34))
+    (stroke (width 0) (type default))
+  )
+  (wire (pts (xy 60.96 88.9) (xy 64.77 88.9))
+    (stroke (width 0) (type default))
+  )
+  (wire (pts (xy 60.96 134.62) (xy 64.77 134.62))
+    (stroke (width 0) (type default))
+  )
+  (wire (pts (xy 111.76 88.9) (xy 115.57 88.9))
+    (stroke (width 0) (type default))
+  )
+  (wire (pts (xy 60.96 86.36) (xy 64.77 86.36))
+    (stroke (width 0) (type default))
+  )
+  (wire (pts (xy 60.96 119.38) (xy 64.77 119.38))
+    (stroke (width 0) (type default))
+  )
+  (wire (pts (xy 60.96 91.44) (xy 64.77 91.44))
+    (stroke (width 0) (type default))
+  )
+  (wire (pts (xy 60.96 43.18) (xy 64.77 43.18))
+    (stroke (width 0) (type default))
+  )
+  (wire (pts (xy 60.96 99.06) (xy 64.77 99.06))
+    (stroke (width 0) (type default))
+  )
+  (wire (pts (xy 60.96 129.54) (xy 64.77 129.54))
+    (stroke (width 0) (type default))
+  )
+  (wire (pts (xy 60.96 96.52) (xy 64.77 96.52))
     (stroke (width 0) (type default))
   )
@@
     (stroke (width 0) (type default))
   )
-  (wire (pts (xy 60.96 101.6) (xy 64.77 101.6))
-    (stroke (width 0) (type default))
-  )
-  (wire (pts (xy 60.96 53.34) (xy 64.77 53.34))
-    (stroke (width 0) (type default))
-  )
-  (wire (pts (xy 60.96 88.9) (xy 64.77 88.9))
-    (stroke (width 0) (type default))
-  )
-  (wire (pts (xy 60.96 134.62) (xy 64.77 134.62))
-    (stroke (width 0) (type default))
-  )
-  (wire (pts (xy 111.76 88.9) (xy 115.57 88.9))
-    (stroke (width 0) (type default))
-  )
-  (wire (pts (xy 60.96 86.36) (xy 64.77 86.36))
-    (stroke (width 0) (type default))
-  )
-  (wire (pts (xy 60.96 119.38) (xy 64.77 119.38))
-    (stroke (width 0) (type default))
-  )
-  (wire (pts (xy 60.96 91.44) (xy 64.77 91.44))
-    (stroke (width 0) (type default))
-  )
-  (wire (pts (xy 60.96 43.18) (xy 64.77 43.18))
-    (stroke (width 0) (type default))
-  )
-  (wire (pts (xy 60.96 99.06) (xy 64.77 99.06))
-    (stroke (width 0) (type default))
-  )
-  (wire (pts (xy 60.96 129.54) (xy 64.77 129.54))
-    (stroke (width 0) (type default))
-  )
-  (wire (pts (xy 60.96 96.52) (xy 64.77 96.52))
-    (stroke (width 0) (type default))
-  )
   (wire (pts (xy 60.96 81.28) (xy 64.77 81.28))
     (stroke (width 0) (type default))
@@
     (effects (font (size 1.27 1.27)) (justify right))
   )
+  (hierarchical_label "5V_S1" (shape input) (at 60.96 91.44 180) (fields_autoplaced)
+    (effects (font (size 1.27 1.27)) (justify right))
+  )
   (hierarchical_label "CAN2_L" (shape bidirectional) (at 60.96 48.26 180) (fields_autoplaced)
     (effects (font (size 1.27 1.27)) (justify right))
@@
     (effects (font (size 1.27 1.27)) (justify right))
   )
+  (hierarchical_label "3V3_S2" (shape input) (at 60.96 66.04 180) (fields_autoplaced)
+    (effects (font (size 1.27 1.27)) (justify right))
+  )
   (hierarchical_label "UART1_TX" (shape bidirectional) (at 60.96 68.58 180) (fields_autoplaced)
     (effects (font (size 1.27 1.27)) (justify right))
@@
     (effects (font (size 1.27 1.27)) (justify right))
   )
+  (hierarchical_label "5V_S2" (shape input) (at 60.96 116.84 180) (fields_autoplaced)
+    (effects (font (size 1.27 1.27)) (justify right))
+  )
   (hierarchical_label "RS4851_B" (shape bidirectional) (at 60.96 58.42 180) (fields_autoplaced)
     (effects (font (size 1.27 1.27)) (justify right))
   )
   (hierarchical_label "SPI1_MOSI" (shape bidirectional) (at 60.96 96.52 180) (fields_autoplaced)
+    (effects (font (size 1.27 1.27)) (justify right))
+  )
+  (hierarchical_label "3V3_S1" (shape input) (at 60.96 40.64 180) (fields_autoplaced)
     (effects (font (size 1.27 1.27)) (justify right))
   )
@@
     )
   )
-  (symbol (lib_id "power:GND") (at 60.96 116.84 270) (unit 1)
-    (in_bom yes) (on_board yes) (dnp no) (fields_autoplaced)
-    (property "Reference" "#PWR0258" (at 54.61 116.84 0)
-      (effects (font (size 1.27 1.27)) hide)
-    )
-    (property "Value" "GND" (at 57.15 116.84 90)
-      (effects (font (size 1.27 1.27)) (justify right))
-    )
-    (property "Footprint" "" (at 60.96 116.84 0)
-      (effects (font (size 1.27 1.27)) hide)
-    )
-    (property "Datasheet" "" (at 60.96 116.84 0)
-      (effects (font (size 1.27 1.27)) hide)
-    )
-    (pin "1")
-    (instances
-      (project "ESLGSU"
-        (path "/b556fa32-e0cb-409c-ac85-9f2ac606be79/feac87e8-d04c-4646-81d1-6a4c94f01f41"
-          (reference "#PWR0258") (unit 1)
-        )
-      )
-    )
-  )
-  (symbol (lib_id "power:GND") (at 60.96 91.44 270) (unit 1)
-    (in_bom yes) (on_board yes) (dnp no) (fields_autoplaced)
-    (property "Reference" "#PWR0253" (at 54.61 91.44 0)
-      (effects (font (size 1.27 1.27)) hide)
-    )
-    (property "Value" "GND" (at 57.15 91.44 90)
-      (effects (font (size 1.27 1.27)) (justify right))
-    )
-    (property "Footprint" "" (at 60.96 91.44 0)
-      (effects (font (size 1.27 1.27)) hide)
-    )
-    (property "Datasheet" "" (at 60.96 91.44 0)
-      (effects (font (size 1.27 1.27)) hide)
-    )
-    (pin "1")
-    (instances
-      (project "ESLGSU"
-        (path "/b556fa32-e0cb-409c-ac85-9f2ac606be79/feac87e8-d04c-4646-81d1-6a4c94f01f41"
-          (reference "#PWR0253") (unit 1)
-        )
-      )
-    )
-  )
   (symbol (lib_id "power:GND") (at 60.96 104.14 270) (unit 1)
     (in_bom yes) (on_board yes) (dnp no) (fields_autoplaced)
@@
         (path "/b556fa32-e0cb-409c-ac85-9f2ac606be79/feac87e8-d04c-4646-81d1-6a4c94f01f41"
           (reference "#PWR0255") (unit 1)
-        )
-      )
-    )
-  )
-  (symbol (lib_id "power:GND") (at 60.96 40.64 270) (unit 1)
-    (in_bom yes) (on_board yes) (dnp no) (fields_autoplaced)
-    (property "Reference" "#PWR0249" (at 54.61 40.64 0)
-      (effects (font (size 1.27 1.27)) hide)
-    )
-    (property "Value" "GND" (at 57.15 40.64 90)
-      (effects (font (size 1.27 1.27)) (justify right))
-    )
-    (property "Footprint" "" (at 60.96 40.64 0)
-      (effects (font (size 1.27 1.27)) hide)
-    )
-    (property "Datasheet" "" (at 60.96 40.64 0)
-      (effects (font (size 1.27 1.27)) hide)
-    )
-    (pin "1")
-    (instances
-      (project "ESLGSU"
-        (path "/b556fa32-e0cb-409c-ac85-9f2ac606be79/feac87e8-d04c-4646-81d1-6a4c94f01f41"
-          (reference "#PWR0249") (unit 1)
         )
       )
@@
         )
       )
-    )
-  )
-  (symbol (lib_id "power:GND") (at 60.96 66.04 270) (unit 1)
-    (in_bom yes) (on_board yes) (dnp no) (fields_autoplaced)
-    (property "Reference" "#PWR0251" (at 54.61 66.04 0)
-      (effects (font (size 1.27 1.27)) hide)
-    )
-    (property "Value" "GND" (at 57.15 66.04 90)
-      (effects (font (size 1.27 1.27)) (justify right))
-    )
-    (property "Footprint" "" (at 60.96 66.04 0)
-      (effects (font (size 1.27 1.27)) hide)
-    )
-    (property "Datasheet" "" (at 60.96 66.04 0)
-      (effects (font (size 1.27 1.27)) hide)
-    )
-    (pin "1")
-    (instances
-      (project "ESLGSU"
-        (path "/b556fa32-e0cb-409c-ac85-9f2ac606be79/feac87e8-d04c-4646-81d1-6a4c94f01f41"
-          (reference "#PWR0251") (unit 1)
-        )
-      )
