File: ESLGSU_Power_Switches.kicad_sch (KiCad schematic)
At the start: 12 parts, among them U94 TPS2553DRVR, U95 TPS2553DRVR, U96 TPS2553DRVR, U97 TPS2553DRVR

Commit message: Should be done with minimal version
Parts:
- C12, R285, R286, R287, R288, U94, U95, U96, U97: now not fitted; now left out of the parts list
Changed lines of the file:
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@@
   )
   (symbol (lib_id "ESLGSU_Parts_Lib:TPS2553DRVR") (at 90.17 49.53 0) (unit 1)
-    (in_bom yes) (on_board yes) (dnp no) (fields_autoplaced)
+    (in_bom no) (on_board yes) (dnp yes) (fields_autoplaced)
     (property "Reference" "U94" (at 90.17 30.48 0)
       (effects (font (size 1.27 1.27)))
@@
   )
   (symbol (lib_id "ESLGSU_Parts_Lib:TPS2553DRVR") (at 90.17 146.05 0) (unit 1)
-    (in_bom yes) (on_board yes) (dnp no) (fields_autoplaced)
+    (in_bom no) (on_board yes) (dnp yes) (fields_autoplaced)
     (property "Reference" "U97" (at 90.17 127 0)
       (effects (font (size 1.27 1.27)))
@@
   )
   (symbol (lib_id "Device:C_Small") (at 60.96 41.91 0) (unit 1)
-    (in_bom yes) (on_board yes) (dnp no)
+    (in_bom no) (on_board yes) (dnp yes)
     (property "Reference" "C12" (at 63.5 41.91 0)
       (effects (font (size 1.27 1.27)) (justify left))
@@
   )
   (symbol (lib_id "Device:C_Small") (at 60.96 138.43 0) (unit 1)
-    (in_bom yes) (on_board yes) (dnp no)
+    (in_bom no) (on_board yes) (dnp yes)
     (property "Reference" "C12" (at 63.5 138.43 0)
       (effects (font (size 1.27 1.27)) (justify left))
@@
   )
   (symbol (lib_id "Device:R_Small_US") (at 97.79 111.76 0) (unit 1)
-    (in_bom yes) (on_board yes) (dnp no) (fields_autoplaced)
+    (in_bom no) (on_board yes) (dnp yes) (fields_autoplaced)
     (property "Reference" "R287" (at 100.33 110.49 0)
       (effects (font (size 1.27 1.27)) (justify left))
@@
   )
   (symbol (lib_id "Device:C_Small") (at 60.96 106.68 0) (unit 1)
-    (in_bom yes) (on_board yes) (dnp no)
+    (in_bom no) (on_board yes) (dnp yes)
     (property "Reference" "C12" (at 63.5 106.68 0)
       (effects (font (size 1.27 1.27)) (justify left))
@@
   )
   (symbol (lib_id "Device:C_Small") (at 60.96 74.93 0) (unit 1)
-    (in_bom yes) (on_board yes) (dnp no)
+    (in_bom no) (on_board yes) (dnp yes)
     (property "Reference" "C12" (at 63.5 74.93 0)
       (effects (font (size 1.27 1.27)) (justify left))
@@
   )
   (symbol (lib_id "Device:R_Small_US") (at 97.79 80.01 0) (unit 1)
-    (in_bom yes) (on_board yes) (dnp no) (fields_autoplaced)
+    (in_bom no) (on_board yes) (dnp yes) (fields_autoplaced)
     (property "Reference" "R286" (at 100.33 78.74 0)
       (effects (font (size 1.27 1.27)) (justify left))
@@
   )
   (symbol (lib_id "ESLGSU_Parts_Lib:TPS2553DRVR") (at 90.17 82.55 0) (unit 1)
-    (in_bom yes) (on_board yes) (dnp no) (fields_autoplaced)
+    (in_bom no) (on_board yes) (dnp yes) (fields_autoplaced)
     (property "Reference" "U95" (at 90.17 63.5 0)
       (effects (font (size 1.27 1.27)))
@@
   )
   (symbol (lib_id "ESLGSU_Parts_Lib:TPS2553DRVR") (at 90.17 114.3 0) (unit 1)
-    (in_bom yes) (on_board yes) (dnp no) (fields_autoplaced)
+    (in_bom no) (on_board yes) (dnp yes) (fields_autoplaced)
     (property "Reference" "U96" (at 90.17 95.25 0)
       (effects (font (size 1.27 1.27)))
@@
   )
   (symbol (lib_id "Device:R_Small_US") (at 97.79 46.99 0) (unit 1)
-    (in_bom yes) (on_board yes) (dnp no) (fields_autoplaced)
+    (in_bom no) (on_board yes) (dnp yes) (fields_autoplaced)
     (property "Reference" "R285" (at 100.33 45.72 0)
       (effects (font (size 1.27 1.27)) (justify left))
@@
   )
   (symbol (lib_id "Device:R_Small_US") (at 97.79 143.51 0) (unit 1)
-    (in_bom yes) (on_board yes) (dnp no) (fields_autoplaced)
+    (in_bom no) (on_board yes) (dnp yes) (fields_autoplaced)
     (property "Reference" "R288" (at 100.33 142.24 0)
       (effects (font (size 1.27 1.27)) (justify left))
