File: ESLGSU_Pi_Zero.kicad_sch (KiCad schematic)
At the start: 3 parts, among them U72 FH-00339

Commit message: Final V1 board with notes
Parts:
- U72: LCSC Part C2685112 -> C2685115
Changed lines of the file:
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@@
       (effects (font (size 1.27 1.27)) hide)
     )
-    (property "LCSC Part" "C2685112" (at 128.27 80.01 0)
+    (property "LCSC Part" "C2685115" (at 128.27 80.01 0)
       (effects (font (size 1.27 1.27)) hide)
     )
